Commit message: [organization] Keep files as in original repos: talos-data and hyq-description

File: hyq_description/robots/hyq_no_sensors.urdf (robot description, URDF)
Before this commit: robot hyq, 19 links, 18 joints
Links:
- link lf_hipassembly: geometry collision mesh filename=package://hyq_description/meshes/leg/hipassembly.dae scale=1 1 1; visual mesh filename=package://hyq_description/meshes/leg/hipassembly.dae scale=1 1 1
- link lf_lowerleg: geometry collision cylinder length=0.346 radius=0.02; visual mesh filename=package://hyq_description/meshes/leg/lowerleg.dae scale=1 1 1
- link lf_upperleg: geometry collision mesh filename=package://hyq_description/meshes/leg/upperleg.dae scale=1 1 1; visual mesh filename=package://hyq_description/meshes/leg/upperleg.dae scale=1 1 1
- link lh_hipassembly: geometry collision mesh filename=package://hyq_description/meshes/leg/hipassembly.dae scale=1 1 1; visual mesh filename=package://hyq_description/meshes/leg/hipassembly.dae scale=1 1 1
- link lh_lowerleg: geometry collision cylinder length=0.346 radius=0.02; visual mesh filename=package://hyq_description/meshes/leg/lowerleg.dae scale=1 1 1
- link lh_upperleg: geometry collision mesh filename=package://hyq_description/meshes/leg/upperleg.dae scale=1 1 1; visual mesh filename=package://hyq_description/meshes/leg/upperleg.dae scale=1 1 1
- link rf_hipassembly: geometry collision mesh filename=package://hyq_description/meshes/leg/hipassembly.dae scale=1 1 1; visual mesh filename=package://hyq_description/meshes/leg/hipassembly.dae scale=1 1 1
- link rf_lowerleg: geometry collision cylinder length=0.346 radius=0.02; visual mesh filename=package://hyq_description/meshes/leg/lowerleg.dae scale=1 1 1
- link rf_upperleg: geometry collision mesh filename=package://hyq_description/meshes/leg/upperleg.dae scale=1 1 1; visual mesh filename=package://hyq_description/meshes/leg/upperleg.dae scale=1 1 1
- link rh_hipassembly: geometry collision mesh filename=package://hyq_description/meshes/leg/hipassembly.dae scale=1 1 1; visual mesh filename=package://hyq_description/meshes/leg/hipassembly.dae scale=1 1 1
- link rh_lowerleg: geometry collision cylinder length=0.346 radius=0.02; visual mesh filename=package://hyq_description/meshes/leg/lowerleg.dae scale=1 1 1
- link rh_upperleg: geometry collision mesh filename=package://hyq_description/meshes/leg/upperleg.dae scale=1 1 1; visual mesh filename=package://hyq_description/meshes/leg/upperleg.dae scale=1 1 1
- link trunk: geometry collision mesh filename=package://hyq_description/meshes/trunk/trunk.dae scale=1 1 1; visual mesh filename=package://hyq_description/meshes/trunk/trunk.dae scale=1 1 1

File: talos_data/robots/talos_left_arm.urdf (robot description, URDF)
Before this commit: robot talos, 17 links, 16 joints
Links:
- link arm_left_1_link: geometry collision mesh filename=package://talos_data/meshes/arm/arm_1_collision.STL scale=1 1 1; visual mesh filename=package://talos_data/meshes/arm/arm_1_collision.STL scale=1 1 1
- link arm_left_2_link: geometry collision mesh filename=package://talos_data/meshes/arm/arm_2_collision.STL scale=1 1 1; visual mesh filename=package://talos_data/meshes/arm/arm_2_collision.STL scale=1 1 1
- link arm_left_3_link: geometry collision mesh filename=package://talos_data/meshes/arm/arm_3_collision.STL scale=1 1 1; visual mesh filename=package://talos_data/meshes/arm/arm_3_collision.STL scale=1 1 1
- link arm_left_4_link: geometry collision mesh filename=package://talos_data/meshes/arm/arm_4_collision.STL scale=1 1 1; visual mesh filename=package://talos_data/meshes/arm/arm_4_collision.STL scale=1 1 1
- link arm_left_5_link: geometry collision mesh filename=package://talos_data/meshes/arm/arm_5_collision.STL scale=1 1 1; visual mesh filename=package://talos_data/meshes/arm/arm_5_collision.STL scale=1 1 1
- link arm_left_6_link: geometry collision mesh filename=package://talos_data/meshes/arm/arm_6_collision.STL scale=1 1 1; visual mesh filename=package://talos_data/meshes/arm/arm_6_collision.STL scale=1 1 1
- link arm_left_7_link: geometry collision mesh filename=package://talos_data/meshes/arm/arm_7_collision.STL scale=1 1 1; visual mesh filename=package://talos_data/meshes/arm/arm_7.STL scale=1 1 1
- link gripper_left_base_link: geometry collision mesh filename=package://talos_data/meshes/gripper/base_link_collision.STL scale=1 1 1; visual mesh filename=package://talos_data/meshes/gripper/base_link.STL scale=1 1 1
- link gripper_left_fingertip_1_link: geometry collision mesh filename=package://talos_data/meshes/gripper/fingertip_collision.STL scale=1 1 1; visual mesh filename=package://talos_data/meshes/gripper/fingertip.STL scale=1 1 1
- link gripper_left_fingertip_2_link: geometry collision mesh filename=package://talos_data/meshes/gripper/fingertip_collision.STL scale=1 1 1; visual mesh filename=package://talos_data/meshes/gripper/fingertip.STL scale=1 1 1
- link gripper_left_fingertip_3_link: geometry collision mesh filename=package://talos_data/meshes/gripper/fingertip_collision.STL scale=1 1 1; visual mesh filename=package://talos_data/meshes/gripper/fingertip.STL scale=1 1 1
- link gripper_left_inner_double_link: geometry collision mesh filename=package://talos_data/meshes/gripper/inner_double_collision.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 scale=1 1 1; visual mesh filename=package://talos_data/meshes/gripper/inner_double.STL scale=1 1 1
- link gripper_left_inner_single_link: geometry collision mesh filename=package://talos_data/meshes/gripper/inner_single_collision.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 scale=1 1 1; visual mesh filename=package://talos_data/meshes/gripper/inner_single.STL scale=1 1 1
- link gripper_left_motor_double_link: geometry collision mesh filename=package://talos_data/meshes/gripper/gripper_motor_double_co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 scale=1 1 1; visual mesh filename=package://talos_data/meshes/gripper/gripper_motor_double.STL scale=1 1 1
- link gripper_left_motor_single_link: geometry collision mesh filename=package://talos_data/meshes/gripper/gripper_motor_single_co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 scale=1 1 1; visual mesh filename=package://talos_data/meshes/gripper/gripper_motor_single.STL scale=1 1 1

File: talos_data/robots/talos_reduced.urdf (robot description, URDF)
Before this commit: robot talos, 60 links, 59 joints
Links:
- link arm_left_1_link: geometry collision mesh filename=package://talos_data/meshes/arm/arm_1_collision.STL scale=1 1 1; visual mesh filename=package://talos_data/meshes/arm/arm_1_collision.STL scale=1 1 1
- link arm_left_2_link: geometry collision mesh filename=package://talos_data/meshes/arm/arm_2_collision.STL scale=1 1 1; visual mesh filename=package://talos_data/meshes/arm/arm_2_collision.STL scale=1 1 1
- link arm_left_3_link: geometry collision mesh filename=package://talos_data/meshes/arm/arm_3_collision.STL scale=1 1 1; visual mesh filename=package://talos_data/meshes/arm/arm_3_collision.STL scale=1 1 1
- link arm_left_4_link: geometry collision mesh filename=package://talos_data/meshes/arm/arm_4_collision.STL scale=1 1 1; visual mesh filename=package://talos_data/meshes/arm/arm_4_collision.STL scale=1 1 1
- link arm_left_5_link: geometry collision mesh filename=package://talos_data/meshes/arm/arm_5_collision.STL scale=1 1 1; visual mesh filename=package://talos_data/meshes/arm/arm_5_collision.STL scale=1 1 1
- link arm_left_6_link: geometry collision mesh filename=package://talos_data/meshes/arm/arm_6_collision.STL scale=1 1 1; visual mesh filename=package://talos_data/meshes/arm/arm_6_collision.STL scale=1 1 1
- link arm_left_7_link: geometry collision mesh filename=package://talos_data/meshes/arm/arm_7_collision.STL scale=1 1 1; visual mesh filename=package://talos_data/meshes/arm/arm_7.STL scale=1 1 1
- link arm_right_1_link: geometry collision mesh filename=package://talos_data/meshes/arm/arm_1_collision.STL scale=1 -1 1; visual mesh filename=package://talos_data/meshes/arm/arm_1_collision.STL scale=1 -1 1
- link arm_right_2_link: geometry collision mesh filename=package://talos_data/meshes/arm/arm_2_collision.STL scale=1 -1 1; visual mesh filename=package://talos_data/meshes/arm/arm_2_collision.STL scale=1 -1 1
- link arm_right_3_link: geometry collision mesh filename=package://talos_data/meshes/arm/arm_3_collision.STL scale=1 -1 1; visual mesh filename=package://talos_data/meshes/arm/arm_3_collision.STL scale=1 -1 1
- link arm_right_4_link: geometry collision mesh filename=package://talos_data/meshes/arm/arm_4_collision.STL scale=1 -1 1; visual mesh filename=package://talos_data/meshes/arm/arm_4_collision.STL scale=1 -1 1
- link arm_right_5_link: geometry collision mesh filename=package://talos_data/meshes/arm/arm_5_collision.STL scale=1 -1 1; visual mesh filename=package://talos_data/meshes/arm/arm_5_collision.STL scale=1 -1 1
- link arm_right_6_link: geometry collision mesh filename=package://talos_data/meshes/arm/arm_6_collision.STL scale=1 -1 1; visual mesh filename=package://talos_data/meshes/arm/arm_6_collision.STL scale=1 -1 1
- link arm_right_7_link: geometry collision mesh filename=package://talos_data/meshes/arm/arm_7_collision.STL scale=1 -1 1; visual mesh filename=package://talos_data/meshes/arm/arm_7_collision.STL scale=1 -1 1
- link base_link: geometry collision mesh filename=package://talos_data/meshes/torso/base_link_collision.STL scale=1 1 1; visual mesh filename=package://talos_data/meshes/torso/base_link.STL scale=1 1 1
- link gripper_left_base_link: geometry collision mesh filename=package://talos_data/meshes/gripper/base_link_collision.STL scale=1 1 1; visual mesh filename=package://talos_data/meshes/gripper/base_link.STL scale=1 1 1
- link gripper_left_fingertip_1_link: geometry collision mesh filename=package://talos_data/meshes/gripper/fingertip_collision.STL scale=1 1 1; visual mesh filename=package://talos_data/meshes/gripper/fingertip.STL scale=1 1 1
- link gripper_left_fingertip_2_link: geometry collision mesh filename=package://talos_data/meshes/gripper/fingertip_collision.STL scale=1 1 1; visual mesh filename=package://talos_data/meshes/gripper/fingertip.STL scale=1 1 1
- link gripper_left_fingertip_3_link: geometry collision mesh filename=package://talos_data/meshes/gripper/fingertip_collision.STL scale=1 1 1; visual mesh filename=package://talos_data/meshes/gripper/fingertip.STL scale=1 1 1
- link gripper_left_inner_double_link: geometry collision mesh filename=package://talos_data/meshes/gripper/inner_double_collision.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 scale=1 1 1; visual mesh filename=package://talos_data/meshes/gripper/inner_double.STL scale=1 1 1
- link gripper_left_inner_single_link: geometry collision mesh filename=package://talos_data/meshes/gripper/inner_single_collision.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 scale=1 1 1; visual mesh filename=package://talos_data/meshes/gripper/inner_single.STL scale=1 1 1
- link gripper_left_motor_double_link: geometry collision mesh filename=package://talos_data/meshes/gripper/gripper_motor_double_co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 scale=1 1 1; visual mesh filename=package://talos_data/meshes/gripper/gripper_motor_double.STL scale=1 1 1
- link gripper_left_motor_single_link: geometry collision mesh filename=package://talos_data/meshes/gripper/gripper_motor_single_co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 scale=1 1 1; visual mesh filename=package://talos_data/meshes/gripper/gripper_motor_single.STL scale=1 1 1
- link gripper_right_base_link: geometry collision mesh filename=package://talos_data/meshes/gripper/base_link_collision.STL scale=1 1 1; visual mesh filename=package://talos_data/meshes/gripper/base_link.STL scale=1 1 1
- link gripper_right_fingertip_1_link: geometry collision mesh filename=package://talos_data/meshes/gripper/fingertip_collision.STL scale=1 1 1; visual mesh filename=package://talos_data/meshes/gripper/fingertip.STL scale=1 1 1
- link gripper_right_fingertip_2_link: geometry collision mesh filename=package://talos_data/meshes/gripper/fingertip_collision.STL scale=1 1 1; visual mesh filename=package://talos_data/meshes/gripper/fingertip.STL scale=1 1 1
- link gripper_right_fingertip_3_link: geometry collision mesh filename=package://talos_data/meshes/gripper/fingertip_collision.STL scale=1 1 1; visual mesh filename=package://talos_data/meshes/gripper/fingertip.STL scale=1 1 1
- link gripper_right_inner_double_link: geometry collision mesh filename=package://talos_data/meshes/gripper/inner_double_collision.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 scale=1 1 1; visual mesh filename=package://talos_data/meshes/gripper/inner_double.STL scale=1 1 1
- link gripper_right_inner_single_link: geometry collision mesh filename=package://talos_data/meshes/gripper/inner_single_collision.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 scale=1 1 1; visual mesh filename=package://talos_data/meshes/gripper/inner_single.STL scale=1 1 1
- link gripper_right_motor_double_link: geometry collision mesh filename=package://talos_data/meshes/gripper/gripper_motor_double_co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 scale=1 1 1; visual mesh filename=package://talos_data/meshes/gripper/gripper_motor_double.STL scale=1 1 1
- link gripper_right_motor_single_link: geometry collision mesh filename=package://talos_data/meshes/gripper/gripper_motor_single_co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 scale=1 1 1; visual mesh filename=package://talos_data/meshes/gripper/gripper_motor_single.STL scale=1 1 1
- link head_1_link: geometry collision mesh filename=package://talos_data/meshes/head/head_1_collision.stl scale=1 1 1; visual mesh filename=package://talos_data/meshes/head/head_1.stl scale=1 1 1
- link head_2_link: geometry collision mesh filename=package://talos_data/meshes/head/head_2_collision.stl scale=1 1 1; visual mesh filename=package://talos_data/meshes/head/head_2.stl scale=1 1 1
- link leg_left_1_link: geometry collision mesh filename=package://talos_data/meshes/v2/hip_z_collision.stl scale=1 1.0 1; visual mesh filename=package://talos_data/meshes/v2/hip_z_lo_res.stl scale=1 1.0 1
- link leg_left_2_link: geometry collision mesh filename=package://talos_data/meshes/v2/hip_x_collision.stl scale=1 1.0 1; visual mesh filename=package://talos_data/meshes/v2/hip_x_lo_res.stl scale=1 1.0 1
- link leg_left_3_link: geometry collision mesh filename=package://talos_data/meshes/v2/hip_y_collision.stl scale=1 1.0 1; visual mesh filename=package://talos_data/meshes/v2/hip_y_lo_res.stl scale=1 1.0 1
- link leg_left_4_link: geometry collision mesh filename=package://talos_data/meshes/v2/knee_collision.stl scale=1 1.0 1; visual mesh filename=package://talos_data/meshes/v2/knee_lo_res.stl scale=1 1.0 1
- link leg_left_5_link: geometry collision mesh filename=package://talos_data/meshes/v2/ankle_Y_collision.stl scale=1 1.0 1; visual mesh filename=package://talos_data/meshes/v2/ankle_Y_lo_res.stl scale=1 1.0 1
- link leg_left_6_link: geometry collision box size=0.21 0.13 0.02; visual mesh filename=package://talos_data/meshes/v2/ankle_X_lo_res.stl scale=1 1.0 1
- link leg_right_1_link: geometry collision mesh filename=package://talos_data/meshes/v2/hip_z_collision.stl scale=1 -1.0 1; visual mesh filename=package://talos_data/meshes/v2/hip_z_lo_res.stl scale=1 -1.0 1
- link leg_right_2_link: geometry collision mesh filename=package://talos_data/meshes/v2/hip_x_collision.stl scale=1 -1.0 1; visual mesh filename=package://talos_data/meshes/v2/hip_x_lo_res.stl scale=1 -1.0 1
- link leg_right_3_link: geometry collision mesh filename=package://talos_data/meshes/v2/hip_y_collision.stl scale=1 -1.0 1; visual mesh filename=package://talos_data/meshes/v2/hip_y_lo_res.stl scale=1 -1.0 1
- link leg_right_4_link: geometry collision mesh filename=package://talos_data/meshes/v2/knee_collision.stl scale=1 -1.0 1; visual mesh filename=package://talos_data/meshes/v2/knee_lo_res.stl scale=1 -1.0 1
- link leg_right_5_link: geometry collision mesh filename=package://talos_data/meshes/v2/ankle_Y_collision.stl scale=1 -1.0 1; visual mesh filename=package://talos_data/meshes/v2/ankle_Y_lo_res.stl scale=1 -1.0 1
- link leg_right_6_link: geometry collision box size=0.21 0.13 0.02; visual mesh filename=package://talos_data/meshes/v2/ankle_X_lo_res.stl scale=1 -1.0 1
- link torso_1_link: geometry collision mesh filename=package://talos_data/meshes/torso/torso_1.STL scale=1 1 1; visual mesh filename=package://talos_data/meshes/torso/torso_1.STL scale=1 1 1
- link torso_2_link: geometry collision mesh filename=package://talos_data/meshes/torso/torso_2_collision.STL scale=1 1 1; visual mesh filename=package://talos_data/meshes/torso/torso_2.STL scale=1 1 1
