Commit message: [icub] Added some mass for massless links, this is for numerical reasons

File: icub_description/robots/icub.urdf (robot description, URDF)
Before this commit: robot iCub, 56 links, 55 joints
Links:
- link l_wrist_1: mass 0 -> 0.1
- link neck_1: mass 0 -> 0.1
- link neck_2: mass 0 -> 0.1
- link r_wrist_1: mass 0 -> 0.1
- link torso: mass 0 -> 0.1
- link torso_1: mass 0 -> 0.1
- link torso_2: mass 0 -> 0.1
