Commit message: [bugfix] Fixed bug with the mesh path + used .stl instead of .STL

File: double_pendulum_description/urdf/double_pendulum.urdf (robot description, URDF)
Before this commit: robot 2dof_planar, 3 links, 2 joints
Links:
- link base_link: geometry collision mesh filename=package://double_pendulum_description/meshes/base_link.stl; visual mesh filename=package://double_pendulum_description/meshes/base_link.stl
- link link1: geometry collision mesh filename=package://double_pendulum_description/meshes/link1.stl; visual mesh filename=package://double_pendulum_description/meshes/link1.stl
- link link2: geometry collision mesh filename=package://double_pendulum_description/meshes/link2.stl; visual mesh filename=package://double_pendulum_description/meshes/link2.stl
