Commit message: [talos_data] Update paths - cf. #19

File: robots/talos_data/robots/talos_left_arm.urdf (robot description, URDF)
Before this commit: robot talos, 17 links, 16 joints
Links:
- link arm_left_1_link: geometry collision mesh filename=package://example-robot-data/robots/talos_data/meshes/arm/a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 scale=1 1 1; visual mesh filename=package://example-robot-data/robots/talos_data/meshes/arm/a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 scale=1 1 1
- link arm_left_2_link: geometry collision mesh filename=package://example-robot-data/robots/talos_data/meshes/arm/a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 scale=1 1 1; visual mesh filename=package://example-robot-data/robots/talos_data/meshes/arm/a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 scale=1 1 1
- link arm_left_3_link: geometry collision mesh filename=package://example-robot-data/robots/talos_data/meshes/arm/a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 scale=1 1 1; visual mesh filename=package://example-robot-data/robots/talos_data/meshes/arm/a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 scale=1 1 1
- link arm_left_4_link: geometry collision mesh filename=package://example-robot-data/robots/talos_data/meshes/arm/a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 scale=1 1 1; visual mesh filename=package://example-robot-data/robots/talos_data/meshes/arm/a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 scale=1 1 1
- link arm_left_5_link: geometry collision mesh filename=package://example-robot-data/robots/talos_data/meshes/arm/a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 scale=1 1 1; visual mesh filename=package://example-robot-data/robots/talos_data/meshes/arm/a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 scale=1 1 1
- link arm_left_6_link: geometry collision mesh filename=package://example-robot-data/robots/talos_data/meshes/arm/a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 scale=1 1 1; visual mesh filename=package://example-robot-data/robots/talos_data/meshes/arm/a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 scale=1 1 1
- link arm_left_7_link: geometry collision mesh filename=package://example-robot-data/robots/talos_data/meshes/arm/a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 scale=1 1 1; visual mesh filename=package://example-robot-data/robots/talos_data/meshes/arm/a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 scale=1 1 1
- link gripper_left_base_link: geometry collision mesh filename=package://example-robot-data/robots/talos_data/meshes/gripp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 scale=1 1 1; visual mesh filename=package://example-robot-data/robots/talos_data/meshes/gripp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 scale=1 1 1
- link gripper_left_fingertip_1_link: geometry collision mesh filename=package://example-robot-data/robots/talos_data/meshes/gripp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 scale=1 1 1; visual mesh filename=package://example-robot-data/robots/talos_data/meshes/gripp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 scale=1 1 1
- link gripper_left_fingertip_2_link: geometry collision mesh filename=package://example-robot-data/robots/talos_data/meshes/gripp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 scale=1 1 1; visual mesh filename=package://example-robot-data/robots/talos_data/meshes/gripp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 scale=1 1 1
- link gripper_left_fingertip_3_link: geometry collision mesh filename=package://example-robot-data/robots/talos_data/meshes/gripp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 scale=1 1 1; visual mesh filename=package://example-robot-data/robots/talos_data/meshes/gripp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 scale=1 1 1
- link gripper_left_inner_double_link: geometry collision mesh filename=package://example-robot-data/robots/talos_data/meshes/gripp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 scale=1 1 1; visual mesh filename=package://example-robot-data/robots/talos_data/meshes/gripp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 scale=1 1 1
- link gripper_left_inner_single_link: geometry collision mesh filename=package://example-robot-data/robots/talos_data/meshes/gripp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 scale=1 1 1; visual mesh filename=package://example-robot-data/robots/talos_data/meshes/gripp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 scale=1 1 1
- link gripper_left_motor_double_link: geometry collision mesh filename=package://example-robot-data/robots/talos_data/meshes/gripp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 scale=1 1 1; visual mesh filename=package://example-robot-data/robots/talos_data/meshes/gripp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 scale=1 1 1
- link gripper_left_motor_single_link: geometry collision mesh filename=package://example-robot-data/robots/talos_data/meshes/gripp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 scale=1 1 1; visual mesh filename=package://example-robot-data/robots/talos_data/meshes/gripp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 scale=1 1 1

File: robots/talos_data/robots/talos_reduced.urdf (robot description, URDF)
Before this commit: robot talos, 60 links, 59 joints
Links:
- link arm_left_1_link: geometry collision mesh filename=package://example-robot-data/robots/talos_data/meshes/arm/a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 scale=1 1 1; visual mesh filename=package://example-robot-data/robots/talos_data/meshes/arm/a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 scale=1 1 1
- link arm_left_2_link: geometry collision mesh filename=package://example-robot-data/robots/talos_data/meshes/arm/a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 scale=1 1 1; visual mesh filename=package://example-robot-data/robots/talos_data/meshes/arm/a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 scale=1 1 1
- link arm_left_3_link: geometry collision mesh filename=package://example-robot-data/robots/talos_data/meshes/arm/a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 scale=1 1 1; visual mesh filename=package://example-robot-data/robots/talos_data/meshes/arm/a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 scale=1 1 1
- link arm_left_4_link: geometry collision mesh filename=package://example-robot-data/robots/talos_data/meshes/arm/a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 scale=1 1 1; visual mesh filename=package://example-robot-data/robots/talos_data/meshes/arm/a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 scale=1 1 1
- link arm_left_5_link: geometry collision mesh filename=package://example-robot-data/robots/talos_data/meshes/arm/a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 scale=1 1 1; visual mesh filename=package://example-robot-data/robots/talos_data/meshes/arm/a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 scale=1 1 1
- link arm_left_6_link: geometry collision mesh filename=package://example-robot-data/robots/talos_data/meshes/arm/a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 scale=1 1 1; visual mesh filename=package://example-robot-data/robots/talos_data/meshes/arm/a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 scale=1 1 1
- link arm_left_7_link: geometry collision mesh filename=package://example-robot-data/robots/talos_data/meshes/arm/a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 scale=1 1 1; visual mesh filename=package://example-robot-data/robots/talos_data/meshes/arm/a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 scale=1 1 1
- link arm_right_1_link: geometry collision mesh filename=package://example-robot-data/robots/talos_data/meshes/arm/a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 scale=1 -1 1; visual mesh filename=package://example-robot-data/robots/talos_data/meshes/arm/a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 scale=1 -1 1
- link arm_right_2_link: geometry collision mesh filename=package://example-robot-data/robots/talos_data/meshes/arm/a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 scale=1 -1 1; visual mesh filename=package://example-robot-data/robots/talos_data/meshes/arm/a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 scale=1 -1 1
- link arm_right_3_link: geometry collision mesh filename=package://example-robot-data/robots/talos_data/meshes/arm/a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 scale=1 -1 1; visual mesh filename=package://example-robot-data/robots/talos_data/meshes/arm/a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 scale=1 -1 1
- link arm_right_4_link: geometry collision mesh filename=package://example-robot-data/robots/talos_data/meshes/arm/a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 scale=1 -1 1; visual mesh filename=package://example-robot-data/robots/talos_data/meshes/arm/a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 scale=1 -1 1
- link arm_right_5_link: geometry collision mesh filename=package://example-robot-data/robots/talos_data/meshes/arm/a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 scale=1 -1 1; visual mesh filename=package://example-robot-data/robots/talos_data/meshes/arm/a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 scale=1 -1 1
- link arm_right_6_link: geometry collision mesh filename=package://example-robot-data/robots/talos_data/meshes/arm/a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 scale=1 -1 1; visual mesh filename=package://example-robot-data/robots/talos_data/meshes/arm/a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 scale=1 -1 1
- link arm_right_7_link: geometry collision mesh filename=package://example-robot-data/robots/talos_data/meshes/arm/a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 scale=1 -1 1; visual mesh filename=package://example-robot-data/robots/talos_data/meshes/arm/a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 scale=1 -1 1
- link base_link: geometry collision mesh filename=package://example-robot-data/robots/talos_data/meshes/torso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 scale=1 1 1; visual mesh filename=package://example-robot-data/robots/talos_data/meshes/torso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 scale=1 1 1
- link gripper_left_base_link: geometry collision mesh filename=package://example-robot-data/robots/talos_data/meshes/gripp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 scale=1 1 1; visual mesh filename=package://example-robot-data/robots/talos_data/meshes/gripp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 scale=1 1 1
- link gripper_left_fingertip_1_link: geometry collision mesh filename=package://example-robot-data/robots/talos_data/meshes/gripp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 scale=1 1 1; visual mesh filename=package://example-robot-data/robots/talos_data/meshes/gripp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 scale=1 1 1
- link gripper_left_fingertip_2_link: geometry collision mesh filename=package://example-robot-data/robots/talos_data/meshes/gripp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 scale=1 1 1; visual mesh filename=package://example-robot-data/robots/talos_data/meshes/gripp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 scale=1 1 1
- link gripper_left_fingertip_3_link: geometry collision mesh filename=package://example-robot-data/robots/talos_data/meshes/gripp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 scale=1 1 1; visual mesh filename=package://example-robot-data/robots/talos_data/meshes/gripp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 scale=1 1 1
- link gripper_left_inner_double_link: geometry collision mesh filename=package://example-robot-data/robots/talos_data/meshes/gripp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 scale=1 1 1; visual mesh filename=package://example-robot-data/robots/talos_data/meshes/gripp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 scale=1 1 1
- link gripper_left_inner_single_link: geometry collision mesh filename=package://example-robot-data/robots/talos_data/meshes/gripp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 scale=1 1 1; visual mesh filename=package://example-robot-data/robots/talos_data/meshes/gripp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 scale=1 1 1
- link gripper_left_motor_double_link: geometry collision mesh filename=package://example-robot-data/robots/talos_data/meshes/gripp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 scale=1 1 1; visual mesh filename=package://example-robot-data/robots/talos_data/meshes/gripp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 scale=1 1 1
- link gripper_left_motor_single_link: geometry collision mesh filename=package://example-robot-data/robots/talos_data/meshes/gripp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 scale=1 1 1; visual mesh filename=package://example-robot-data/robots/talos_data/meshes/gripp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 scale=1 1 1
- link gripper_right_base_link: geometry collision mesh filename=package://example-robot-data/robots/talos_data/meshes/gripp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 scale=1 1 1; visual mesh filename=package://example-robot-data/robots/talos_data/meshes/gripp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 scale=1 1 1
- link gripper_right_fingertip_1_link: geometry collision mesh filename=package://example-robot-data/robots/talos_data/meshes/gripp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 scale=1 1 1; visual mesh filename=package://example-robot-data/robots/talos_data/meshes/gripp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 scale=1 1 1
- link gripper_right_fingertip_2_link: geometry collision mesh filename=package://example-robot-data/robots/talos_data/meshes/gripp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 scale=1 1 1; visual mesh filename=package://example-robot-data/robots/talos_data/meshes/gripp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 scale=1 1 1
- link gripper_right_fingertip_3_link: geometry collision mesh filename=package://example-robot-data/robots/talos_data/meshes/gripp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 scale=1 1 1; visual mesh filename=package://example-robot-data/robots/talos_data/meshes/gripp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 scale=1 1 1
- link gripper_right_inner_double_link: geometry collision mesh filename=package://example-robot-data/robots/talos_data/meshes/gripp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 scale=1 1 1; visual mesh filename=package://example-robot-data/robots/talos_data/meshes/gripp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 scale=1 1 1
- link gripper_right_inner_single_link: geometry collision mesh filename=package://example-robot-data/robots/talos_data/meshes/gripp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 scale=1 1 1; visual mesh filename=package://example-robot-data/robots/talos_data/meshes/gripp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 scale=1 1 1
- link gripper_right_motor_double_link: geometry collision mesh filename=package://example-robot-data/robots/talos_data/meshes/gripp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 scale=1 1 1; visual mesh filename=package://example-robot-data/robots/talos_data/meshes/gripp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 scale=1 1 1
- link gripper_right_motor_single_link: geometry collision mesh filename=package://example-robot-data/robots/talos_data/meshes/gripp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 scale=1 1 1; visual mesh filename=package://example-robot-data/robots/talos_data/meshes/gripp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 scale=1 1 1
- link head_1_link: geometry collision mesh filename=package://example-robot-data/robots/talos_data/meshes/head/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 scale=1 1 1; visual mesh filename=package://example-robot-data/robots/talos_data/meshes/head/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 scale=1 1 1
- link head_2_link: geometry collision mesh filename=package://example-robot-data/robots/talos_data/meshes/head/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 scale=1 1 1; visual mesh filename=package://example-robot-data/robots/talos_data/meshes/head/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 scale=1 1 1
- link leg_left_1_link: geometry collision mesh filename=package://example-robot-data/robots/talos_data/meshes/v2/hi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 scale=1 1.0 1; visual mesh filename=package://example-robot-data/robots/talos_data/meshes/v2/hi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 scale=1 1.0 1
- link leg_left_2_link: geometry collision mesh filename=package://example-robot-data/robots/talos_data/meshes/v2/hi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 scale=1 1.0 1; visual mesh filename=package://example-robot-data/robots/talos_data/meshes/v2/hi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 scale=1 1.0 1
- link leg_left_3_link: geometry collision mesh filename=package://example-robot-data/robots/talos_data/meshes/v2/hi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 scale=1 1.0 1; visual mesh filename=package://example-robot-data/robots/talos_data/meshes/v2/hi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 scale=1 1.0 1
- link leg_left_4_link: geometry collision mesh filename=package://example-robot-data/robots/talos_data/meshes/v2/kn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 scale=1 1.0 1; visual mesh filename=package://example-robot-data/robots/talos_data/meshes/v2/kn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 scale=1 1.0 1
- link leg_left_5_link: geometry collision mesh filename=package://example-robot-data/robots/talos_data/meshes/v2/an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 scale=1 1.0 1; visual mesh filename=package://example-robot-data/robots/talos_data/meshes/v2/an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 scale=1 1.0 1
- link leg_left_6_link: geometry collision box size=0.21 0.13 0.02; visual mesh filename=package://example-robot-data/robots/talos_data/meshes/v2/an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 scale=1 1.0 1
- link leg_right_1_link: geometry collision mesh filename=package://example-robot-data/robots/talos_data/meshes/v2/hi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 scale=1 -1.0 1; visual mesh filename=package://example-robot-data/robots/talos_data/meshes/v2/hi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 scale=1 -1.0 1
- link leg_right_2_link: geometry collision mesh filename=package://example-robot-data/robots/talos_data/meshes/v2/hi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 scale=1 -1.0 1; visual mesh filename=package://example-robot-data/robots/talos_data/meshes/v2/hi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 scale=1 -1.0 1
- link leg_right_3_link: geometry collision mesh filename=package://example-robot-data/robots/talos_data/meshes/v2/hi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 scale=1 -1.0 1; visual mesh filename=package://example-robot-data/robots/talos_data/meshes/v2/hi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 scale=1 -1.0 1
- link leg_right_4_link: geometry collision mesh filename=package://example-robot-data/robots/talos_data/meshes/v2/kn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 scale=1 -1.0 1; visual mesh filename=package://example-robot-data/robots/talos_data/meshes/v2/kn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 scale=1 -1.0 1
- link leg_right_5_link: geometry collision mesh filename=package://example-robot-data/robots/talos_data/meshes/v2/an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 scale=1 -1.0 1; visual mesh filename=package://example-robot-data/robots/talos_data/meshes/v2/an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 scale=1 -1.0 1
- link leg_right_6_link: geometry collision box size=0.21 0.13 0.02; visual mesh filename=package://example-robot-data/robots/talos_data/meshes/v2/an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 scale=1 -1.0 1
- link torso_1_link: geometry collision mesh filename=package://example-robot-data/robots/talos_data/meshes/torso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 scale=1 1 1; visual mesh filename=package://example-robot-data/robots/talos_data/meshes/torso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 scale=1 1 1
- link torso_2_link: geometry collision mesh filename=package://example-robot-data/robots/talos_data/meshes/torso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 scale=1 1 1; visual mesh filename=package://example-robot-data/robots/talos_data/meshes/torso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 scale=1 1 1
