Commit message: [talos_reduced] Fix inertia and mass to zero for optical links. Letting this unfix is adding 1kg for each link in pybullet.

File: robots/talos_data/robots/talos_reduced.urdf (robot description, URDF)
Before this commit: robot talos, 60 links, 59 joints
Links:
- link rgbd_depth_frame: mass None -> 0.0
- link rgbd_depth_optical_frame: mass None -> 0.0
- link rgbd_rgb_frame: mass None -> 0.0
- link rgbd_rgb_optical_frame: mass None -> 0.0
