Commit message: talos_box & talos_full_box: set default link mass to 0

File: robots/talos_data/robots/talos_full_v2.urdf (robot description, URDF)
Before this commit: robot talos, 60 links, 59 joints
Links:
- link rgbd_depth_frame: mass 0.0 -> 0
- link rgbd_depth_optical_frame: mass 0.0 -> 0
- link rgbd_rgb_frame: mass 0.0 -> 0
- link rgbd_rgb_optical_frame: mass 0.0 -> 0

File: robots/talos_data/robots/talos_full_v2_box.urdf (robot description, URDF)
Before this commit: robot talos, 60 links, 59 joints
Links:
- link rgbd_depth_frame: mass None -> 0
- link rgbd_depth_optical_frame: mass None -> 0
- link rgbd_rgb_frame: mass None -> 0
- link rgbd_rgb_optical_frame: mass None -> 0

File: robots/talos_data/robots/talos_reduced_box.urdf (robot description, URDF)
Before this commit: robot talos, 60 links, 59 joints
Links:
- link rgbd_depth_frame: mass None -> 0
- link rgbd_depth_optical_frame: mass None -> 0
- link rgbd_rgb_frame: mass None -> 0
- link rgbd_rgb_optical_frame: mass None -> 0
