Commit message: [iris_description] Update paths - cf. #19

File: robots/iris_description/robots/iris.urdf (robot description, URDF)
Before this commit: robot iris, 6 links, 5 joints
Links:
- link iris__base_link: geometry collision box size=0.47 0.47 0.11; visual mesh filename=package://example-robot-data/robots/iris_description/meshes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 scale=1 1 1
- link iris__rotor_0: geometry collision cylinder length=0.005 radius=0.128; visual mesh filename=package://example-robot-data/robots/iris_description/meshes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 scale=1 1 1
- link iris__rotor_1: geometry collision cylinder length=0.005 radius=0.128; visual mesh filename=package://example-robot-data/robots/iris_description/meshes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 scale=1 1 1
- link iris__rotor_2: geometry collision cylinder length=0.005 radius=0.128; visual mesh filename=package://example-robot-data/robots/iris_description/meshes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 scale=1 1 1
- link iris__rotor_3: geometry collision cylinder length=0.005 radius=0.128; visual mesh filename=package://example-robot-data/robots/iris_description/meshes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 scale=1 1 1

File: robots/iris_description/robots/iris_simple.urdf (robot description, URDF)
Before this commit: robot iris, 6 links, 5 joints
Links:
- link iris__base_link: geometry collision box size=0.47 0.47 0.11; visual mesh filename=package://example-robot-data/robots/iris_description/meshes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 scale=1 1 1
- link iris__rotor_0: geometry collision cylinder length=0.005 radius=0.128; visual mesh filename=package://example-robot-data/robots/iris_description/meshes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 scale=1 1 1
- link iris__rotor_1: geometry collision cylinder length=0.005 radius=0.128; visual mesh filename=package://example-robot-data/robots/iris_description/meshes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 scale=1 1 1
- link iris__rotor_2: geometry collision cylinder length=0.005 radius=0.128; visual mesh filename=package://example-robot-data/robots/iris_description/meshes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 scale=1 1 1
- link iris__rotor_3: geometry collision cylinder length=0.005 radius=0.128; visual mesh filename=package://example-robot-data/robots/iris_description/meshes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 scale=1 1 1
