Commit message: hyq_description: Add inertia information for simulator

File: robots/hyq_description/robots/hyq_no_sensors.urdf (robot description, URDF)
Before this commit: robot hyq, 19 links, 18 joints
Links:
- link base_link: mass None -> 1e-6
- link lf_foot: mass None -> 1e-6
- link lh_foot: mass None -> 1e-6
- link rf_foot: mass None -> 1e-6
- link rh_foot: mass None -> 1e-6

Commit message: [hyq_description] Update paths - cf. #19

File: robots/hyq_description/robots/hyq_no_sensors.urdf (robot description, URDF)
Before this commit: robot hyq, 19 links, 18 joints
Links:
- link lf_hipassembly: geometry collision mesh filename=package://example-robot-data/robots/hyq_description/meshes/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 scale=1 1 1; visual mesh filename=package://example-robot-data/robots/hyq_description/meshes/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 scale=1 1 1
- link lf_lowerleg: geometry collision cylinder length=0.346 radius=0.02; visual mesh filename=package://example-robot-data/robots/hyq_description/meshes/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 scale=1 1 1
- link lf_upperleg: geometry collision mesh filename=package://example-robot-data/robots/hyq_description/meshes/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 scale=1 1 1; visual mesh filename=package://example-robot-data/robots/hyq_description/meshes/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 scale=1 1 1
- link lh_hipassembly: geometry collision mesh filename=package://example-robot-data/robots/hyq_description/meshes/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 scale=1 1 1; visual mesh filename=package://example-robot-data/robots/hyq_description/meshes/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 scale=1 1 1
- link lh_lowerleg: geometry collision cylinder length=0.346 radius=0.02; visual mesh filename=package://example-robot-data/robots/hyq_description/meshes/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 scale=1 1 1
- link lh_upperleg: geometry collision mesh filename=package://example-robot-data/robots/hyq_description/meshes/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 scale=1 1 1; visual mesh filename=package://example-robot-data/robots/hyq_description/meshes/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 scale=1 1 1
- link rf_hipassembly: geometry collision mesh filename=package://example-robot-data/robots/hyq_description/meshes/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 scale=1 1 1; visual mesh filename=package://example-robot-data/robots/hyq_description/meshes/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 scale=1 1 1
- link rf_lowerleg: geometry collision cylinder length=0.346 radius=0.02; visual mesh filename=package://example-robot-data/robots/hyq_description/meshes/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 scale=1 1 1
- link rf_upperleg: geometry collision mesh filename=package://example-robot-data/robots/hyq_description/meshes/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 scale=1 1 1; visual mesh filename=package://example-robot-data/robots/hyq_description/meshes/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 scale=1 1 1
- link rh_hipassembly: geometry collision mesh filename=package://example-robot-data/robots/hyq_description/meshes/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 scale=1 1 1; visual mesh filename=package://example-robot-data/robots/hyq_description/meshes/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 scale=1 1 1
- link rh_lowerleg: geometry collision cylinder length=0.346 radius=0.02; visual mesh filename=package://example-robot-data/robots/hyq_description/meshes/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 scale=1 1 1
- link rh_upperleg: geometry collision mesh filename=package://example-robot-data/robots/hyq_description/meshes/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 scale=1 1 1; visual mesh filename=package://example-robot-data/robots/hyq_description/meshes/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 scale=1 1 1
- link trunk: geometry collision mesh filename=package://example-robot-data/robots/hyq_description/meshes/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 scale=1 1 1; visual mesh filename=package://example-robot-data/robots/hyq_description/meshes/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 scale=1 1 1
