Commit message: [hector_description] Update paths - cf. #19

File: robots/hector_description/robots/quadrotor_base.urdf (robot description, URDF)
Before this commit: robot hector, 1 links, 0 joints
Links:
- link base_link: geometry collision mesh filename=package://example-robot-data/robots/hector_description/mesh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; visual mesh filename=package://example-robot-data/robots/hector_description/mesh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

File: robots/hector_description/robots/quadrotor_base.urdf.xacro (robot description, xacro)
@@ -13,5 +13,5 @@
         <origin xyz="0 0 0" rpy="0 0 0" />
         <geometry>
-          <mesh filename="package://hector-description/meshes/quadrotor/quadrotor_base.dae"/>
+          <mesh filename="package://example-robot-data/robots/hector_description/meshes/quadrotor/quadrotor_base.dae"/>
         </geometry>
       </visual>
@@ -19,5 +19,5 @@
         <origin xyz="0 0 0" rpy="0 0 0" />
         <geometry>
-          <mesh filename="package://hector-description/meshes/quadrotor/quadrotor_base.stl"/>
+          <mesh filename="package://example-robot-data/robots/hector_description/meshes/quadrotor/quadrotor_base.stl"/>
         </geometry>
       </collision>

File: robots/hector_description/robots/quadrotor_base.xacro (robot description, xacro)
@@ -1,5 +1,5 @@
 <?xml version="1.0" ?>
 <robot name="hector" xmlns:xacro="http://www.ros.org/wiki/xacro">
-  <xacro:include filename="package://hector-description/urdf/quadrotor_base.urdf.xacro"/>
+  <xacro:include filename="package://example-robot-data/robots/hector_description/urdf/quadrotor_base.urdf.xacro"/>
   <xacro:quadrotor_base_macro/>
 </robot>
