Commit message: WIP: ANYmal-Kinova Change joint type from continuous to revolute To not trigger Pinocchio's SO(2) representation

File: robots/anymal_b_simple_description/robots/anymal-kinova.urdf (robot description, URDF)
Before this commit: robot anymal, 37 links, 36 joints
Joints:
- joint j2s6s200_joint_1: type continuous -> revolute
- joint j2s6s200_joint_4: type continuous -> revolute
- joint j2s6s200_joint_6: type continuous -> revolute

Commit message: anymal_b_simple_description: Add missing inertia, fix for simulator

File: robots/anymal_b_simple_description/robots/anymal-kinova.urdf (robot description, URDF)
Before this commit: robot anymal, 37 links, 36 joints
Links:
- removed link base_inertia
- link LF_FOOT: mass None -> 0.001
- link LH_FOOT: mass None -> 0.001
- link RF_FOOT: mass None -> 0.001
- link RH_FOOT: mass None -> 0.001
- link base: mass None -> 16.793507758
- link j2s6s200_end_effector: mass None -> 0.001
- link jaco_front_hatch_support_v2: mass None -> 0.205; geometry collision sphere radius=0.031; visual mesh filename=package://kinova_description/meshes/jaco_front_hatch_suppor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
- link jaco_mounting_block: mass None -> 0.1741; geometry collision sphere radius=0.031; visual mesh filename=package://kinova_description/meshes/jaco_mounting_block.dae
Joints:
- removed joint base_to_base_inertia

File: robots/anymal_b_simple_description/robots/anymal.urdf (robot description, URDF)
Before this commit: robot anymal, 23 links, 22 joints
Links:
- removed link base_inertia
- link LF_FOOT: mass None -> 0.001
- link LH_FOOT: mass None -> 0.001
- link RF_FOOT: mass None -> 0.001
- link RH_FOOT: mass None -> 0.001
- link base: mass None -> 16.793507758
Joints:
- removed joint base_to_base_inertia

Commit message: [anymal_b_simple_description] Update paths - cf. #19

File: robots/anymal_b_simple_description/robots/anymal-kinova.urdf (robot description, URDF)
Before this commit: robot anymal, 36 links, 35 joints
Links:
- link LF_ADAPTER: geometry collision cylinder length=0.32125 radius=0.015; visual mesh filename=package://example-robot-data/robots/anymal_b_simple_descrip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 scale=1 1 1
- link LF_HIP: geometry collision cylinder length=0.03 radius=0.045; collision cylinder length=0.1 radius=0.08
- link LF_SHANK: geometry collision box size=0.08 0.07 0.13; visual mesh filename=package://example-robot-data/robots/anymal_b_simple_descrip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 scale=1 1 1
- link LF_THIGH: geometry collision box size=0.08 0.04 0.25; collision cylinder length=0.12 radius=0.06
- link LH_ADAPTER: geometry collision cylinder length=0.32125 radius=0.015; visual mesh filename=package://example-robot-data/robots/anymal_b_simple_descrip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 scale=1 1 1
- link LH_HIP: geometry collision cylinder length=0.03 radius=0.045; collision cylinder length=0.1 radius=0.08
- link LH_SHANK: geometry collision box size=0.08 0.07 0.13; visual mesh filename=package://example-robot-data/robots/anymal_b_simple_descrip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 scale=1 1 1
- link LH_THIGH: geometry collision box size=0.08 0.04 0.25; collision cylinder length=0.12 radius=0.06
- link RF_ADAPTER: geometry collision cylinder length=0.32125 radius=0.015; visual mesh filename=package://example-robot-data/robots/anymal_b_simple_descrip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 scale=1 1 1
- link RF_HIP: geometry collision cylinder length=0.03 radius=0.045; collision cylinder length=0.1 radius=0.08
- link RF_SHANK: geometry collision box size=0.08 0.07 0.13; visual mesh filename=package://example-robot-data/robots/anymal_b_simple_descrip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 scale=1 1 1
- link RF_THIGH: geometry collision box size=0.08 0.04 0.25; collision cylinder length=0.12 radius=0.06
- link RH_ADAPTER: geometry collision cylinder length=0.32125 radius=0.015; visual mesh filename=package://example-robot-data/robots/anymal_b_simple_descrip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 scale=1 1 1
- link RH_HIP: geometry collision cylinder length=0.03 radius=0.045; collision cylinder length=0.1 radius=0.08
- link RH_SHANK: geometry collision box size=0.08 0.07 0.13; visual mesh filename=package://example-robot-data/robots/anymal_b_simple_descrip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 scale=1 1 1
- link RH_THIGH: geometry collision box size=0.08 0.04 0.25; collision cylinder length=0.12 radius=0.06
- link base: geometry collision box size=0.1 0.1 0.07; collision box size=0.1 0.1 0.07
- link j2s6s200_link_1: geometry collision mesh filename=package://example-robot-data/robots/kinova_description/mesh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; visual mesh filename=package://example-robot-data/robots/kinova_description/mesh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
- link j2s6s200_link_2: geometry collision mesh filename=package://example-robot-data/robots/kinova_description/mesh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; visual mesh filename=package://example-robot-data/robots/kinova_description/mesh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
- link j2s6s200_link_3: geometry collision mesh filename=package://example-robot-data/robots/kinova_description/mesh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; visual mesh filename=package://example-robot-data/robots/kinova_description/mesh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
- link j2s6s200_link_4: geometry collision mesh filename=package://example-robot-data/robots/kinova_description/mesh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; visual mesh filename=package://example-robot-data/robots/kinova_description/mesh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
- link j2s6s200_link_5: geometry collision mesh filename=package://example-robot-data/robots/kinova_description/mesh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; visual mesh filename=package://example-robot-data/robots/kinova_description/mesh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
- link j2s6s200_link_6: geometry collision mesh filename=package://example-robot-data/robots/kinova_description/mesh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; visual mesh filename=package://example-robot-data/robots/kinova_description/mesh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
- link j2s6s200_link_base: geometry collision mesh filename=package://example-robot-data/robots/kinova_description/mesh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; visual mesh filename=package://example-robot-data/robots/kinova_description/mesh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
- link j2s6s200_link_finger_1: geometry collision mesh filename=package://example-robot-data/robots/kinova_description/mesh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; visual mesh filename=package://example-robot-data/robots/kinova_description/mesh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
- link j2s6s200_link_finger_2: geometry collision mesh filename=package://example-robot-data/robots/kinova_description/mesh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; visual mesh filename=package://example-robot-data/robots/kinova_description/mesh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
- link j2s6s200_link_finger_tip_1: geometry collision mesh filename=package://example-robot-data/robots/kinova_description/mesh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; visual mesh filename=package://example-robot-data/robots/kinova_description/mesh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
- link j2s6s200_link_finger_tip_2: geometry collision mesh filename=package://example-robot-data/robots/kinova_description/mesh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; visual mesh filename=package://example-robot-data/robots/kinova_description/mesh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
- link jaco_front_hatch_support_v2: geometry collision sphere radius=0.031; visual mesh filename=package://example-robot-data/robots/kinova_description/mesh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
- link jaco_mounting_block: geometry collision sphere radius=0.031; visual mesh filename=package://example-robot-data/robots/kinova_description/mesh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

File: robots/anymal_b_simple_description/robots/anymal.urdf (robot description, URDF)
Before this commit: robot anymal, 22 links, 21 joints
Links:
- link LF_ADAPTER: geometry collision cylinder length=0.32125 radius=0.015; visual mesh filename=package://example-robot-data/robots/anymal_b_simple_descrip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 scale=1 1 1
- link LF_HIP: geometry collision cylinder length=0.03 radius=0.045; collision cylinder length=0.1 radius=0.08
- link LF_SHANK: geometry collision box size=0.08 0.07 0.13; visual mesh filename=package://example-robot-data/robots/anymal_b_simple_descrip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 scale=1 1 1
- link LF_THIGH: geometry collision box size=0.08 0.04 0.25; collision cylinder length=0.12 radius=0.06
- link LH_ADAPTER: geometry collision cylinder length=0.32125 radius=0.015; visual mesh filename=package://example-robot-data/robots/anymal_b_simple_descrip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 scale=1 1 1
- link LH_HIP: geometry collision cylinder length=0.03 radius=0.045; collision cylinder length=0.1 radius=0.08
- link LH_SHANK: geometry collision box size=0.08 0.07 0.13; visual mesh filename=package://example-robot-data/robots/anymal_b_simple_descrip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 scale=1 1 1
- link LH_THIGH: geometry collision box size=0.08 0.04 0.25; collision cylinder length=0.12 radius=0.06
- link RF_ADAPTER: geometry collision cylinder length=0.32125 radius=0.015; visual mesh filename=package://example-robot-data/robots/anymal_b_simple_descrip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 scale=1 1 1
- link RF_HIP: geometry collision cylinder length=0.03 radius=0.045; collision cylinder length=0.1 radius=0.08
- link RF_SHANK: geometry collision box size=0.08 0.07 0.13; visual mesh filename=package://example-robot-data/robots/anymal_b_simple_descrip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 scale=1 1 1
- link RF_THIGH: geometry collision box size=0.08 0.04 0.25; collision cylinder length=0.12 radius=0.06
- link RH_ADAPTER: geometry collision cylinder length=0.32125 radius=0.015; visual mesh filename=package://example-robot-data/robots/anymal_b_simple_descrip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 scale=1 1 1
- link RH_HIP: geometry collision cylinder length=0.03 radius=0.045; collision cylinder length=0.1 radius=0.08
- link RH_SHANK: geometry collision box size=0.08 0.07 0.13; visual mesh filename=package://example-robot-data/robots/anymal_b_simple_descrip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 scale=1 1 1
- link RH_THIGH: geometry collision box size=0.08 0.04 0.25; collision cylinder length=0.12 radius=0.06
- link base: geometry collision box size=0.1 0.1 0.07; collision box size=0.1 0.1 0.07
