Commit message: [anymal] Reverted inertial modification + defined base with tiny inertia

File: robots/anymal_b_simple_description/robots/anymal.urdf (robot description, URDF)
Before this commit: robot anymal, 22 links, 21 joints
Links:
- added link base_inertia, mass 16.793507758
- link base: mass 16.793507758 -> 1e-6
Joints:
- added joint base_to_base_inertia: type fixed, parent base, child base_inertia, origin xyz=0 0 0 rpy=0 0 0
