Commit message: solo_description: Update paths, ref #19

File: robots/solo_description/robots/solo.urdf (robot description, URDF)
Before this commit: robot solo, 13 links, 12 joints
Links:
- link FL_FOOT: geometry collision mesh filename=package://example-robot-data/robots/solo_description/meshes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; visual mesh filename=package://example-robot-data/robots/solo_description/meshes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
- link FL_LOWER_LEG: geometry collision mesh filename=package://example-robot-data/robots/solo_description/meshes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; visual mesh filename=package://example-robot-data/robots/solo_description/meshes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
- link FL_UPPER_LEG: geometry collision mesh filename=package://example-robot-data/robots/solo_description/meshes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; visual mesh filename=package://example-robot-data/robots/solo_description/meshes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
- link FR_FOOT: geometry collision mesh filename=package://example-robot-data/robots/solo_description/meshes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; visual mesh filename=package://example-robot-data/robots/solo_description/meshes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
- link FR_LOWER_LEG: geometry collision mesh filename=package://example-robot-data/robots/solo_description/meshes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; visual mesh filename=package://example-robot-data/robots/solo_description/meshes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
- link FR_UPPER_LEG: geometry collision mesh filename=package://example-robot-data/robots/solo_description/meshes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; visual mesh filename=package://example-robot-data/robots/solo_description/meshes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
- link HL_FOOT: geometry collision mesh filename=package://example-robot-data/robots/solo_description/meshes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; visual mesh filename=package://example-robot-data/robots/solo_description/meshes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
- link HL_LOWER_LEG: geometry collision mesh filename=package://example-robot-data/robots/solo_description/meshes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; visual mesh filename=package://example-robot-data/robots/solo_description/meshes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
- link HL_UPPER_LEG: geometry collision mesh filename=package://example-robot-data/robots/solo_description/meshes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; visual mesh filename=package://example-robot-data/robots/solo_description/meshes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
- link HR_FOOT: geometry collision mesh filename=package://example-robot-data/robots/solo_description/meshes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; visual mesh filename=package://example-robot-data/robots/solo_description/meshes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
- link HR_LOWER_LEG: geometry collision mesh filename=package://example-robot-data/robots/solo_description/meshes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; visual mesh filename=package://example-robot-data/robots/solo_description/meshes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
- link HR_UPPER_LEG: geometry collision mesh filename=package://example-robot-data/robots/solo_description/meshes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; visual mesh filename=package://example-robot-data/robots/solo_description/meshes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
- link base_link: geometry collision mesh filename=package://example-robot-data/robots/solo_description/meshes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; visual mesh filename=package://example-robot-data/robots/solo_description/meshes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

File: robots/solo_description/robots/solo12.urdf (robot description, URDF)
Before this commit: robot solo, 17 links, 16 joints
Links:
- link FL_FOOT: geometry collision mesh filename=package://example-robot-data/robots/solo_description/meshes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; visual mesh filename=package://example-robot-data/robots/solo_description/meshes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
- link FL_LOWER_LEG: geometry collision mesh filename=package://example-robot-data/robots/solo_description/meshes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; visual mesh filename=package://example-robot-data/robots/solo_description/meshes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
- link FL_SHOULDER: geometry collision mesh filename=package://example-robot-data/robots/solo_description/meshes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; visual mesh filename=package://example-robot-data/robots/solo_description/meshes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
- link FL_UPPER_LEG: geometry collision mesh filename=package://example-robot-data/robots/solo_description/meshes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; visual mesh filename=package://example-robot-data/robots/solo_description/meshes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
- link FR_FOOT: geometry collision mesh filename=package://example-robot-data/robots/solo_description/meshes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; visual mesh filename=package://example-robot-data/robots/solo_description/meshes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
- link FR_LOWER_LEG: geometry collision mesh filename=package://example-robot-data/robots/solo_description/meshes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; visual mesh filename=package://example-robot-data/robots/solo_description/meshes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
- link FR_SHOULDER: geometry collision mesh filename=package://example-robot-data/robots/solo_description/meshes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; visual mesh filename=package://example-robot-data/robots/solo_description/meshes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
- link FR_UPPER_LEG: geometry collision mesh filename=package://example-robot-data/robots/solo_description/meshes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; visual mesh filename=package://example-robot-data/robots/solo_description/meshes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
- link HL_FOOT: geometry collision mesh filename=package://example-robot-data/robots/solo_description/meshes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; visual mesh filename=package://example-robot-data/robots/solo_description/meshes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
- link HL_LOWER_LEG: geometry collision mesh filename=package://example-robot-data/robots/solo_description/meshes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; visual mesh filename=package://example-robot-data/robots/solo_description/meshes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
- link HL_SHOULDER: geometry collision mesh filename=package://example-robot-data/robots/solo_description/meshes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; visual mesh filename=package://example-robot-data/robots/solo_description/meshes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
- link HL_UPPER_LEG: geometry collision mesh filename=package://example-robot-data/robots/solo_description/meshes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; visual mesh filename=package://example-robot-data/robots/solo_description/meshes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
- link HR_FOOT: geometry collision mesh filename=package://example-robot-data/robots/solo_description/meshes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; visual mesh filename=package://example-robot-data/robots/solo_description/meshes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
- link HR_LOWER_LEG: geometry collision mesh filename=package://example-robot-data/robots/solo_description/meshes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; visual mesh filename=package://example-robot-data/robots/solo_description/meshes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
- link HR_SHOULDER: geometry collision mesh filename=package://example-robot-data/robots/solo_description/meshes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; visual mesh filename=package://example-robot-data/robots/solo_description/meshes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
- link HR_UPPER_LEG: geometry collision mesh filename=package://example-robot-data/robots/solo_description/meshes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; visual mesh filename=package://example-robot-data/robots/solo_description/meshes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
- link base_link: geometry collision mesh filename=package://example-robot-data/robots/solo_description/meshes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; visual mesh filename=package://example-robot-data/robots/solo_description/meshes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
