Commit message: solo_description: update solo12.urdf

File: robots/solo_description/robots/solo12.urdf (robot description, URDF)
Before this commit: robot solo, 17 links, 16 joints
Links:
- link FL_FOOT: geometry collision mesh filename=package://solo_description/meshes/stl/with_foot/solo_foot.s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; visual mesh filename=package://solo_description/meshes/stl/with_foot/solo_foot.s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
- link FL_LOWER_LEG: geometry collision mesh filename=package://solo_description/meshes/stl/with_foot/solo_lower_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; visual mesh filename=package://solo_description/meshes/stl/with_foot/solo_lower_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
- link FL_SHOULDER: mass 0.150 -> 0.14853845; geometry collision mesh filename=package://solo_description/meshes/stl/solo12/solo12_hip_fe_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; visual mesh filename=package://solo_description/meshes/stl/solo12/solo12_hip_fe_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
- link FL_UPPER_LEG: geometry collision mesh filename=package://solo_description/meshes/stl/with_foot/solo_upper_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; visual mesh filename=package://solo_description/meshes/stl/with_foot/solo_upper_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
- link FR_FOOT: geometry collision mesh filename=package://solo_description/meshes/stl/with_foot/solo_foot.s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; visual mesh filename=package://solo_description/meshes/stl/with_foot/solo_foot.s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
- link FR_LOWER_LEG: geometry collision mesh filename=package://solo_description/meshes/stl/with_foot/solo_lower_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; visual mesh filename=package://solo_description/meshes/stl/with_foot/solo_lower_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
- link FR_SHOULDER: mass 0.150 -> 0.14853845; geometry collision mesh filename=package://solo_description/meshes/stl/solo12/solo12_hip_fe_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; visual mesh filename=package://solo_description/meshes/stl/solo12/solo12_hip_fe_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
- link FR_UPPER_LEG: geometry collision mesh filename=package://solo_description/meshes/stl/with_foot/solo_upper_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; visual mesh filename=package://solo_description/meshes/stl/with_foot/solo_upper_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
- link HL_FOOT: geometry collision mesh filename=package://solo_description/meshes/stl/with_foot/solo_foot.s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; visual mesh filename=package://solo_description/meshes/stl/with_foot/solo_foot.s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
- link HL_LOWER_LEG: geometry collision mesh filename=package://solo_description/meshes/stl/with_foot/solo_lower_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; visual mesh filename=package://solo_description/meshes/stl/with_foot/solo_lower_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
- link HL_SHOULDER: mass 0.150 -> 0.14853845; geometry collision mesh filename=package://solo_description/meshes/stl/solo12/solo12_hip_fe_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; visual mesh filename=package://solo_description/meshes/stl/solo12/solo12_hip_fe_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
- link HL_UPPER_LEG: geometry collision mesh filename=package://solo_description/meshes/stl/with_foot/solo_upper_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; visual mesh filename=package://solo_description/meshes/stl/with_foot/solo_upper_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
- link HR_FOOT: geometry collision mesh filename=package://solo_description/meshes/stl/with_foot/solo_foot.s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; visual mesh filename=package://solo_description/meshes/stl/with_foot/solo_foot.s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
- link HR_LOWER_LEG: geometry collision mesh filename=package://solo_description/meshes/stl/with_foot/solo_lower_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; visual mesh filename=package://solo_description/meshes/stl/with_foot/solo_lower_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
- link HR_SHOULDER: mass 0.150 -> 0.14853845; geometry collision mesh filename=package://solo_description/meshes/stl/solo12/solo12_hip_fe_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; visual mesh filename=package://solo_description/meshes/stl/solo12/solo12_hip_fe_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
- link HR_UPPER_LEG: geometry collision mesh filename=package://solo_description/meshes/stl/with_foot/solo_upper_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; visual mesh filename=package://solo_description/meshes/stl/with_foot/solo_upper_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
- link base_link: mass 1.63315091 -> 1.16115091; geometry collision mesh filename=package://solo_description/meshes/stl/solo12/solo_12_base.s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; visual mesh filename=package://solo_description/meshes/stl/solo12/solo_12_base.s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
Joints:
- joint FL_HAA: origin xyz=0.19 0.1046 0 rpy=0 0 0 -> xyz=0.1946 0.0875 0 rpy=0 0 0
- joint FL_HFE: origin xyz=0 0 0 rpy=0 0 0 -> xyz=0 0.014 0 rpy=0 0 0
- joint FR_HAA: origin xyz=0.19 -0.1046 0 rpy=0 0 0 -> xyz=0.1946 -0.0875 0 rpy=0 0 0
- joint FR_HFE: origin xyz=0 0 0 rpy=0 0 0 -> xyz=0 -0.014 0 rpy=0 0 0
- joint HL_HAA: origin xyz=-0.19 0.1046 0 rpy=0 0 0 -> xyz=-0.1946 0.0875 0 rpy=0 0 0
- joint HL_HFE: origin xyz=0 0 0 rpy=0 0 0 -> xyz=0 0.014 0 rpy=0 0 0
- joint HR_HAA: origin xyz=-0.19 -0.1046 0 rpy=0 0 0 -> xyz=-0.1946 -0.0875 0 rpy=0 0 0
- joint HR_HFE: origin xyz=0 0 0 rpy=0 0 0 -> xyz=0 -0.014 0 rpy=0 0 0
