Commit message: [icub_description] Update paths - cf. #19

File: robots/icub_description/robots/icub.urdf (robot description, URDF)
Before this commit: robot iCub, 56 links, 55 joints
Links:
- link chest: geometry collision mesh filename=package://example-robot-data/robots/icub_description/meshes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 scale=1 1 1; visual mesh filename=package://example-robot-data/robots/icub_description/meshes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 scale=1 1 1
- link head: geometry collision mesh filename=package://example-robot-data/robots/icub_description/meshes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 scale=1 1 1; visual mesh filename=package://example-robot-data/robots/icub_description/meshes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 scale=1 1 1
- link l_ankle_1: geometry collision mesh filename=package://example-robot-data/robots/icub_description/meshes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 scale=1 1 1; visual mesh filename=package://example-robot-data/robots/icub_description/meshes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 scale=1 1 1
- link l_foot: geometry collision mesh filename=package://example-robot-data/robots/icub_description/meshes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 scale=1 1 1; visual mesh filename=package://example-robot-data/robots/icub_description/meshes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 scale=1 1 1
- link l_forearm: geometry collision mesh filename=package://example-robot-data/robots/icub_description/meshes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 scale=1 1 1; visual mesh filename=package://example-robot-data/robots/icub_description/meshes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 scale=1 1 1
- link l_hand: geometry collision mesh filename=package://example-robot-data/robots/icub_description/meshes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 scale=1 1 1; visual mesh filename=package://example-robot-data/robots/icub_description/meshes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 scale=1 1 1
- link l_hip_1: geometry collision mesh filename=package://example-robot-data/robots/icub_description/meshes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 scale=1 1 1; visual mesh filename=package://example-robot-data/robots/icub_description/meshes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 scale=1 1 1
- link l_hip_2: geometry collision mesh filename=package://example-robot-data/robots/icub_description/meshes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 scale=1 1 1; visual mesh filename=package://example-robot-data/robots/icub_description/meshes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 scale=1 1 1
- link l_lower_leg: geometry collision mesh filename=package://example-robot-data/robots/icub_description/meshes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 scale=1 1 1; visual mesh filename=package://example-robot-data/robots/icub_description/meshes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 scale=1 1 1
- link l_shoulder_1: geometry collision mesh filename=package://example-robot-data/robots/icub_description/meshes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 scale=1 1 1; visual mesh filename=package://example-robot-data/robots/icub_description/meshes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 scale=1 1 1
- link l_shoulder_2: geometry collision mesh filename=package://example-robot-data/robots/icub_description/meshes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 scale=1 1 1; visual mesh filename=package://example-robot-data/robots/icub_description/meshes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 scale=1 1 1
- link l_upper_arm: geometry collision mesh filename=package://example-robot-data/robots/icub_description/meshes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 scale=1 1 1; visual mesh filename=package://example-robot-data/robots/icub_description/meshes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 scale=1 1 1
- link l_upper_leg: geometry collision mesh filename=package://example-robot-data/robots/icub_description/meshes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 scale=1 1 1; visual mesh filename=package://example-robot-data/robots/icub_description/meshes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 scale=1 1 1
- link neck_1: geometry collision mesh filename=package://example-robot-data/robots/icub_description/meshes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 scale=1 1 1; visual mesh filename=package://example-robot-data/robots/icub_description/meshes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 scale=1 1 1
- link neck_2: geometry collision mesh filename=package://example-robot-data/robots/icub_description/meshes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 scale=1 1 1; visual mesh filename=package://example-robot-data/robots/icub_description/meshes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 scale=1 1 1
- link r_ankle_1: geometry collision mesh filename=package://example-robot-data/robots/icub_description/meshes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 scale=1 1 1; visual mesh filename=package://example-robot-data/robots/icub_description/meshes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 scale=1 1 1
- link r_foot: geometry collision mesh filename=package://example-robot-data/robots/icub_description/meshes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 scale=1 1 1; visual mesh filename=package://example-robot-data/robots/icub_description/meshes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 scale=1 1 1
- link r_forearm: geometry collision mesh filename=package://example-robot-data/robots/icub_description/meshes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 scale=1 1 1; visual mesh filename=package://example-robot-data/robots/icub_description/meshes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 scale=1 1 1
- link r_hand: geometry collision mesh filename=package://example-robot-data/robots/icub_description/meshes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 scale=1 1 1; visual mesh filename=package://example-robot-data/robots/icub_description/meshes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 scale=1 1 1
- link r_hip_1: geometry collision mesh filename=package://example-robot-data/robots/icub_description/meshes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 scale=1 1 1; visual mesh filename=package://example-robot-data/robots/icub_description/meshes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 scale=1 1 1
- link r_hip_2: geometry collision mesh filename=package://example-robot-data/robots/icub_description/meshes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 scale=1 1 1; visual mesh filename=package://example-robot-data/robots/icub_description/meshes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 scale=1 1 1
- link r_lower_leg: geometry collision mesh filename=package://example-robot-data/robots/icub_description/meshes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 scale=1 1 1; visual mesh filename=package://example-robot-data/robots/icub_description/meshes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 scale=1 1 1
- link r_shoulder_1: geometry collision mesh filename=package://example-robot-data/robots/icub_description/meshes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 scale=1 1 1; visual mesh filename=package://example-robot-data/robots/icub_description/meshes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 scale=1 1 1
- link r_shoulder_2: geometry collision mesh filename=package://example-robot-data/robots/icub_description/meshes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 scale=1 1 1; visual mesh filename=package://example-robot-data/robots/icub_description/meshes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 scale=1 1 1
- link r_upper_arm: geometry collision mesh filename=package://example-robot-data/robots/icub_description/meshes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 scale=1 1 1; visual mesh filename=package://example-robot-data/robots/icub_description/meshes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 scale=1 1 1
- link r_upper_leg: geometry collision mesh filename=package://example-robot-data/robots/icub_description/meshes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 scale=1 1 1; visual mesh filename=package://example-robot-data/robots/icub_description/meshes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 scale=1 1 1
- link root_link: geometry collision mesh filename=package://example-robot-data/robots/icub_description/meshes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 scale=1 1 1; visual mesh filename=package://example-robot-data/robots/icub_description/meshes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 scale=1 1 1
- link torso_1: geometry collision mesh filename=package://example-robot-data/robots/icub_description/meshes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 scale=1 1 1; visual mesh filename=package://example-robot-data/robots/icub_description/meshes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 scale=1 1 1

File: robots/icub_description/robots/icub_reduced.urdf (robot description, URDF)
Before this commit: robot iCub, 56 links, 55 joints
Links:
- link chest: geometry collision mesh filename=package://example-robot-data/robots/icub_description/meshes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 scale=1 1 1; visual mesh filename=package://example-robot-data/robots/icub_description/meshes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 scale=1 1 1
- link head: geometry collision mesh filename=package://example-robot-data/robots/icub_description/meshes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 scale=1 1 1; visual mesh filename=package://example-robot-data/robots/icub_description/meshes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 scale=1 1 1
- link l_ankle_1: geometry collision mesh filename=package://example-robot-data/robots/icub_description/meshes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 scale=1 1 1; visual mesh filename=package://example-robot-data/robots/icub_description/meshes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 scale=1 1 1
- link l_foot: geometry collision mesh filename=package://example-robot-data/robots/icub_description/meshes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 scale=1 1 1; visual mesh filename=package://example-robot-data/robots/icub_description/meshes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 scale=1 1 1
- link l_forearm: geometry collision mesh filename=package://example-robot-data/robots/icub_description/meshes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 scale=1 1 1; visual mesh filename=package://example-robot-data/robots/icub_description/meshes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 scale=1 1 1
- link l_hand: geometry collision mesh filename=package://example-robot-data/robots/icub_description/meshes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 scale=1 1 1; visual mesh filename=package://example-robot-data/robots/icub_description/meshes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 scale=1 1 1
- link l_hip_1: geometry collision mesh filename=package://example-robot-data/robots/icub_description/meshes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 scale=1 1 1; visual mesh filename=package://example-robot-data/robots/icub_description/meshes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 scale=1 1 1
- link l_hip_2: geometry collision mesh filename=package://example-robot-data/robots/icub_description/meshes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 scale=1 1 1; visual mesh filename=package://example-robot-data/robots/icub_description/meshes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 scale=1 1 1
- link l_lower_leg: geometry collision mesh filename=package://example-robot-data/robots/icub_description/meshes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 scale=1 1 1; visual mesh filename=package://example-robot-data/robots/icub_description/meshes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 scale=1 1 1
- link l_shoulder_1: geometry collision mesh filename=package://example-robot-data/robots/icub_description/meshes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 scale=1 1 1; visual mesh filename=package://example-robot-data/robots/icub_description/meshes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 scale=1 1 1
- link l_shoulder_2: geometry collision mesh filename=package://example-robot-data/robots/icub_description/meshes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 scale=1 1 1; visual mesh filename=package://example-robot-data/robots/icub_description/meshes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 scale=1 1 1
- link l_upper_arm: geometry collision mesh filename=package://example-robot-data/robots/icub_description/meshes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 scale=1 1 1; visual mesh filename=package://example-robot-data/robots/icub_description/meshes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 scale=1 1 1
- link l_upper_leg: geometry collision mesh filename=package://example-robot-data/robots/icub_description/meshes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 scale=1 1 1; visual mesh filename=package://example-robot-data/robots/icub_description/meshes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 scale=1 1 1
- link neck_1: geometry collision mesh filename=package://example-robot-data/robots/icub_description/meshes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 scale=1 1 1; visual mesh filename=package://example-robot-data/robots/icub_description/meshes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 scale=1 1 1
- link neck_2: geometry collision mesh filename=package://example-robot-data/robots/icub_description/meshes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 scale=1 1 1; visual mesh filename=package://example-robot-data/robots/icub_description/meshes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 scale=1 1 1
- link r_ankle_1: geometry collision mesh filename=package://example-robot-data/robots/icub_description/meshes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 scale=1 1 1; visual mesh filename=package://example-robot-data/robots/icub_description/meshes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 scale=1 1 1
- link r_foot: geometry collision mesh filename=package://example-robot-data/robots/icub_description/meshes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 scale=1 1 1; visual mesh filename=package://example-robot-data/robots/icub_description/meshes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 scale=1 1 1
- link r_forearm: geometry collision mesh filename=package://example-robot-data/robots/icub_description/meshes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 scale=1 1 1; visual mesh filename=package://example-robot-data/robots/icub_description/meshes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 scale=1 1 1
- link r_hand: geometry collision mesh filename=package://example-robot-data/robots/icub_description/meshes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 scale=1 1 1; visual mesh filename=package://example-robot-data/robots/icub_description/meshes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 scale=1 1 1
- link r_hip_1: geometry collision mesh filename=package://example-robot-data/robots/icub_description/meshes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 scale=1 1 1; visual mesh filename=package://example-robot-data/robots/icub_description/meshes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 scale=1 1 1
- link r_hip_2: geometry collision mesh filename=package://example-robot-data/robots/icub_description/meshes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 scale=1 1 1; visual mesh filename=package://example-robot-data/robots/icub_description/meshes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 scale=1 1 1
- link r_lower_leg: geometry collision mesh filename=package://example-robot-data/robots/icub_description/meshes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 scale=1 1 1; visual mesh filename=package://example-robot-data/robots/icub_description/meshes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 scale=1 1 1
- link r_shoulder_1: geometry collision mesh filename=package://example-robot-data/robots/icub_description/meshes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 scale=1 1 1; visual mesh filename=package://example-robot-data/robots/icub_description/meshes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 scale=1 1 1
- link r_shoulder_2: geometry collision mesh filename=package://example-robot-data/robots/icub_description/meshes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 scale=1 1 1; visual mesh filename=package://example-robot-data/robots/icub_description/meshes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 scale=1 1 1
- link r_upper_arm: geometry collision mesh filename=package://example-robot-data/robots/icub_description/meshes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 scale=1 1 1; visual mesh filename=package://example-robot-data/robots/icub_description/meshes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 scale=1 1 1
- link r_upper_leg: geometry collision mesh filename=package://example-robot-data/robots/icub_description/meshes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 scale=1 1 1; visual mesh filename=package://example-robot-data/robots/icub_description/meshes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 scale=1 1 1
- link root_link: geometry collision mesh filename=package://example-robot-data/robots/icub_description/meshes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 scale=1 1 1; visual mesh filename=package://example-robot-data/robots/icub_description/meshes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 scale=1 1 1
- link torso_1: geometry collision mesh filename=package://example-robot-data/robots/icub_description/meshes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 scale=1 1 1; visual mesh filename=package://example-robot-data/robots/icub_description/meshes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 scale=1 1 1

Commit message: [icub] Include tiny inertia for ICub robot

File: robots/icub_description/robots/icub.urdf (robot description, URDF)
Before this commit: robot iCub, 56 links, 55 joints
Links:
- link base_link: mass None -> 1e-6

File: robots/icub_description/robots/icub_reduced.urdf (robot description, URDF)
Before this commit: robot iCub, 56 links, 55 joints
Links:
- link base_link: mass None -> 1e-6
