Commit message: [kinova_description] Update paths - cf. #19

File: robots/kinova_description/robots/kinova.urdf (robot description, URDF)
Before this commit: robot kinova, 15 links, 14 joints
Links:
- link j2s6s200_link_1: geometry collision mesh filename=package://example-robot-data/robots/kinova_description/mesh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; visual mesh filename=package://example-robot-data/robots/kinova_description/mesh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
- link j2s6s200_link_2: geometry collision mesh filename=package://example-robot-data/robots/kinova_description/mesh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; visual mesh filename=package://example-robot-data/robots/kinova_description/mesh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
- link j2s6s200_link_3: geometry collision mesh filename=package://example-robot-data/robots/kinova_description/mesh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; visual mesh filename=package://example-robot-data/robots/kinova_description/mesh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
- link j2s6s200_link_4: geometry collision mesh filename=package://example-robot-data/robots/kinova_description/mesh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; visual mesh filename=package://example-robot-data/robots/kinova_description/mesh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
- link j2s6s200_link_5: geometry collision mesh filename=package://example-robot-data/robots/kinova_description/mesh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; visual mesh filename=package://example-robot-data/robots/kinova_description/mesh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
- link j2s6s200_link_6: geometry collision mesh filename=package://example-robot-data/robots/kinova_description/mesh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; visual mesh filename=package://example-robot-data/robots/kinova_description/mesh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
- link j2s6s200_link_base: geometry collision mesh filename=package://example-robot-data/robots/kinova_description/mesh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; visual mesh filename=package://example-robot-data/robots/kinova_description/mesh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
- link j2s6s200_link_finger_1: geometry collision mesh filename=package://example-robot-data/robots/kinova_description/mesh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; visual mesh filename=package://example-robot-data/robots/kinova_description/mesh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
- link j2s6s200_link_finger_2: geometry collision mesh filename=package://example-robot-data/robots/kinova_description/mesh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; visual mesh filename=package://example-robot-data/robots/kinova_description/mesh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
- link j2s6s200_link_finger_tip_1: geometry collision mesh filename=package://example-robot-data/robots/kinova_description/mesh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; visual mesh filename=package://example-robot-data/robots/kinova_description/mesh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
- link j2s6s200_link_finger_tip_2: geometry collision mesh filename=package://example-robot-data/robots/kinova_description/mesh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; visual mesh filename=package://example-robot-data/robots/kinova_description/mesh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
- link jaco_front_hatch_support_v2: geometry visual mesh filename=package://example-robot-data/robots/kinova_description/mesh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
- link jaco_mounting_block: geometry visual mesh filename=package://example-robot-data/robots/kinova_description/mesh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

Commit message: Fix Kinova robot

File: robots/kinova_description/robots/kinova.urdf (robot description, URDF)
Before this commit: robot kinova, 15 links, 14 joints
Links:
- link base: mass None -> 0.0
- link j2s6s200_end_effector: mass None -> 0.0
- link jaco_front_hatch_support_v2: mass None -> 0.0
- link jaco_mounting_block: mass None -> 0.0
