Commit message: [romeo_description] Use meshes provided by example-robot-data.

File: robots/romeo_description/urdf/romeo.urdf (robot description, URDF)
Before this commit: robot romeo, 82 links, 81 joints
Links:
- link HeadRollLink: geometry collision mesh filename=package://example-robot-data/robots/romeo_description/meshe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 scale=1 1 1; visual mesh filename=package://example-robot-data/robots/romeo_description/meshe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 scale=1 1 1
- link LElbowYawLink: geometry collision mesh filename=package://example-robot-data/robots/romeo_description/meshe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 scale=1 1 1; visual mesh filename=package://example-robot-data/robots/romeo_description/meshe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 scale=1 1 1
- link LFinger11Link: geometry collision mesh filename=package://example-robot-data/robots/romeo_description/meshe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; visual mesh filename=package://example-robot-data/robots/romeo_description/meshe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
- link LFinger12Link: geometry collision mesh filename=package://example-robot-data/robots/romeo_description/meshe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; visual mesh filename=package://example-robot-data/robots/romeo_description/meshe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
- link LFinger13Link: geometry collision mesh filename=package://example-robot-data/robots/romeo_description/meshe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; visual mesh filename=package://example-robot-data/robots/romeo_description/meshe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
- link LFinger21Link: geometry collision mesh filename=package://example-robot-data/robots/romeo_description/meshe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; visual mesh filename=package://example-robot-data/robots/romeo_description/meshe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
- link LFinger22Link: geometry collision mesh filename=package://example-robot-data/robots/romeo_description/meshe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; visual mesh filename=package://example-robot-data/robots/romeo_description/meshe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
- link LFinger23Link: geometry collision mesh filename=package://example-robot-data/robots/romeo_description/meshe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; visual mesh filename=package://example-robot-data/robots/romeo_description/meshe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
- link LFinger31Link: geometry collision mesh filename=package://example-robot-data/robots/romeo_description/meshe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; visual mesh filename=package://example-robot-data/robots/romeo_description/meshe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
- link LFinger32Link: geometry collision mesh filename=package://example-robot-data/robots/romeo_description/meshe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; visual mesh filename=package://example-robot-data/robots/romeo_description/meshe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
- link LFinger33Link: geometry collision mesh filename=package://example-robot-data/robots/romeo_description/meshe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; visual mesh filename=package://example-robot-data/robots/romeo_description/meshe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
- link LHipPitchLink: geometry collision mesh filename=package://example-robot-data/robots/romeo_description/meshe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 scale=1 1 1; visual mesh filename=package://example-robot-data/robots/romeo_description/meshe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 scale=1 1 1
- link LKneePitchLink: geometry collision mesh filename=package://example-robot-data/robots/romeo_description/meshe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 scale=1 1 1; visual mesh filename=package://example-robot-data/robots/romeo_description/meshe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 scale=1 1 1
- link LShoulderYawLink: geometry collision mesh filename=package://example-robot-data/robots/romeo_description/meshe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 scale=1 1 1; visual mesh filename=package://example-robot-data/robots/romeo_description/meshe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 scale=1 1 1
- link LThumb1Link: geometry collision mesh filename=package://example-robot-data/robots/romeo_description/meshe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; visual mesh filename=package://example-robot-data/robots/romeo_description/meshe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
- link LThumb2Link: geometry collision mesh filename=package://example-robot-data/robots/romeo_description/meshe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; visual mesh filename=package://example-robot-data/robots/romeo_description/meshe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
- link LThumb3Link: geometry collision mesh filename=package://example-robot-data/robots/romeo_description/meshe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; visual mesh filename=package://example-robot-data/robots/romeo_description/meshe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
- link LWristRollLink: geometry collision mesh filename=package://example-robot-data/robots/romeo_description/meshe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 scale=1 1 1; visual mesh filename=package://example-robot-data/robots/romeo_description/meshe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 scale=1 1 1
- link LWristYawLink: geometry collision mesh filename=package://example-robot-data/robots/romeo_description/meshe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 scale=1 1 1; visual mesh filename=package://example-robot-data/robots/romeo_description/meshe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 scale=1 1 1
- link NeckPitchLink: geometry collision mesh filename=package://example-robot-data/robots/romeo_description/meshe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 scale=1 1 1; visual mesh filename=package://example-robot-data/robots/romeo_description/meshe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 scale=1 1 1
- link RElbowYawLink: geometry collision mesh filename=package://example-robot-data/robots/romeo_description/meshe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 scale=1 1 1; visual mesh filename=package://example-robot-data/robots/romeo_description/meshe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 scale=1 1 1
- link RFinger11Link: geometry collision mesh filename=package://example-robot-data/robots/romeo_description/meshe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; visual mesh filename=package://example-robot-data/robots/romeo_description/meshe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
- link RFinger12Link: geometry collision mesh filename=package://example-robot-data/robots/romeo_description/meshe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; visual mesh filename=package://example-robot-data/robots/romeo_description/meshe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
- link RFinger13Link: geometry collision mesh filename=package://example-robot-data/robots/romeo_description/meshe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; visual mesh filename=package://example-robot-data/robots/romeo_description/meshe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
- link RFinger21Link: geometry collision mesh filename=package://example-robot-data/robots/romeo_description/meshe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; visual mesh filename=package://example-robot-data/robots/romeo_description/meshe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
- link RFinger22Link: geometry collision mesh filename=package://example-robot-data/robots/romeo_description/meshe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; visual mesh filename=package://example-robot-data/robots/romeo_description/meshe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
- link RFinger23Link: geometry collision mesh filename=package://example-robot-data/robots/romeo_description/meshe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; visual mesh filename=package://example-robot-data/robots/romeo_description/meshe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
- link RFinger31Link: geometry collision mesh filename=package://example-robot-data/robots/romeo_description/meshe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; visual mesh filename=package://example-robot-data/robots/romeo_description/meshe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
- link RFinger32Link: geometry collision mesh filename=package://example-robot-data/robots/romeo_description/meshe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; visual mesh filename=package://example-robot-data/robots/romeo_description/meshe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
- link RFinger33Link: geometry collision mesh filename=package://example-robot-data/robots/romeo_description/meshe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; visual mesh filename=package://example-robot-data/robots/romeo_description/meshe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
- link RHipPitchLink: geometry collision mesh filename=package://example-robot-data/robots/romeo_description/meshe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 scale=1 1 1; visual mesh filename=package://example-robot-data/robots/romeo_description/meshe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 scale=1 1 1
- link RKneePitchLink: geometry collision mesh filename=package://example-robot-data/robots/romeo_description/meshe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 scale=1 1 1; visual mesh filename=package://example-robot-data/robots/romeo_description/meshe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 scale=1 1 1
- link RShoulderYawLink: geometry collision mesh filename=package://example-robot-data/robots/romeo_description/meshe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 scale=1 1 1; visual mesh filename=package://example-robot-data/robots/romeo_description/meshe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 scale=1 1 1
- link RThumb1Link: geometry collision mesh filename=package://example-robot-data/robots/romeo_description/meshe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; visual mesh filename=package://example-robot-data/robots/romeo_description/meshe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
- link RThumb2Link: geometry collision mesh filename=package://example-robot-data/robots/romeo_description/meshe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; visual mesh filename=package://example-robot-data/robots/romeo_description/meshe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
- link RThumb3Link: geometry collision mesh filename=package://example-robot-data/robots/romeo_description/meshe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; visual mesh filename=package://example-robot-data/robots/romeo_description/meshe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
- link RWristRollLink: geometry collision mesh filename=package://example-robot-data/robots/romeo_description/meshe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 scale=1 1 1; visual mesh filename=package://example-robot-data/robots/romeo_description/meshe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 scale=1 1 1
- link RWristYawLink: geometry collision mesh filename=package://example-robot-data/robots/romeo_description/meshe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 scale=1 1 1; visual mesh filename=package://example-robot-data/robots/romeo_description/meshe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 scale=1 1 1
- link body: geometry collision mesh filename=package://example-robot-data/robots/romeo_description/meshe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 scale=1 1 1; visual mesh filename=package://example-robot-data/robots/romeo_description/meshe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 scale=1 1 1
- link l_ankle: geometry collision mesh filename=package://example-robot-data/robots/romeo_description/meshe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 scale=1 1 1; visual mesh filename=package://example-robot-data/robots/romeo_description/meshe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 scale=1 1 1
- link l_wrist: geometry collision mesh filename=package://example-robot-data/robots/romeo_description/meshe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 scale=1 1 1; visual mesh filename=package://example-robot-data/robots/romeo_description/meshe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 scale=1 1 1
- link r_ankle: geometry collision mesh filename=package://example-robot-data/robots/romeo_description/meshe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 scale=1 1 1; visual mesh filename=package://example-robot-data/robots/romeo_description/meshe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 scale=1 1 1
- link r_wrist: geometry collision mesh filename=package://example-robot-data/robots/romeo_description/meshe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 scale=1 1 1; visual mesh filename=package://example-robot-data/robots/romeo_description/meshe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 scale=1 1 1
- link torso: geometry collision mesh filename=package://example-robot-data/robots/romeo_description/meshe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 scale=1 1 1; visual mesh filename=package://example-robot-data/robots/romeo_description/meshe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 scale=1 1 1

File: robots/romeo_description/urdf/romeo_small.urdf (robot description, URDF)
Before this commit: robot romeo, 58 links, 57 joints
Links:
- link HeadRollLink: geometry collision mesh filename=package://example-robot-data/robots/romeo_description/meshe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 scale=1 1 1; visual mesh filename=package://example-robot-data/robots/romeo_description/meshe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 scale=1 1 1
- link LElbowYawLink: geometry collision mesh filename=package://example-robot-data/robots/romeo_description/meshe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 scale=1 1 1; visual mesh filename=package://example-robot-data/robots/romeo_description/meshe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 scale=1 1 1
- link LHipPitchLink: geometry collision mesh filename=package://example-robot-data/robots/romeo_description/meshe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 scale=1 1 1; visual mesh filename=package://example-robot-data/robots/romeo_description/meshe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 scale=1 1 1
- link LKneePitchLink: geometry collision mesh filename=package://example-robot-data/robots/romeo_description/meshe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 scale=1 1 1; visual mesh filename=package://example-robot-data/robots/romeo_description/meshe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 scale=1 1 1
- link LShoulderYawLink: geometry collision mesh filename=package://example-robot-data/robots/romeo_description/meshe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 scale=1 1 1; visual mesh filename=package://example-robot-data/robots/romeo_description/meshe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 scale=1 1 1
- link LWristRollLink: geometry collision mesh filename=package://example-robot-data/robots/romeo_description/meshe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 scale=1 1 1; visual mesh filename=package://example-robot-data/robots/romeo_description/meshe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 scale=1 1 1
- link LWristYawLink: geometry collision mesh filename=package://example-robot-data/robots/romeo_description/meshe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 scale=1 1 1; visual mesh filename=package://example-robot-data/robots/romeo_description/meshe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 scale=1 1 1
- link NeckPitchLink: geometry collision mesh filename=package://example-robot-data/robots/romeo_description/meshe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 scale=1 1 1; visual mesh filename=package://example-robot-data/robots/romeo_description/meshe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 scale=1 1 1
- link RElbowYawLink: geometry collision mesh filename=package://example-robot-data/robots/romeo_description/meshe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 scale=1 1 1; visual mesh filename=package://example-robot-data/robots/romeo_description/meshe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 scale=1 1 1
- link RHipPitchLink: geometry collision mesh filename=package://example-robot-data/robots/romeo_description/meshe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 scale=1 1 1; visual mesh filename=package://example-robot-data/robots/romeo_description/meshe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 scale=1 1 1
- link RKneePitchLink: geometry collision mesh filename=package://example-robot-data/robots/romeo_description/meshe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 scale=1 1 1; visual mesh filename=package://example-robot-data/robots/romeo_description/meshe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 scale=1 1 1
- link RShoulderYawLink: geometry collision mesh filename=package://example-robot-data/robots/romeo_description/meshe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 scale=1 1 1; visual mesh filename=package://example-robot-data/robots/romeo_description/meshe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 scale=1 1 1
- link RWristRollLink: geometry collision mesh filename=package://example-robot-data/robots/romeo_description/meshe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 scale=1 1 1; visual mesh filename=package://example-robot-data/robots/romeo_description/meshe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 scale=1 1 1
- link RWristYawLink: geometry collision mesh filename=package://example-robot-data/robots/romeo_description/meshe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 scale=1 1 1; visual mesh filename=package://example-robot-data/robots/romeo_description/meshe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 scale=1 1 1
- link body: geometry collision mesh filename=package://example-robot-data/robots/romeo_description/meshe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 scale=1 1 1; visual mesh filename=package://example-robot-data/robots/romeo_description/meshe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 scale=1 1 1
- link l_ankle: geometry collision mesh filename=package://example-robot-data/robots/romeo_description/meshe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 scale=1 1 1; visual mesh filename=package://example-robot-data/robots/romeo_description/meshe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 scale=1 1 1
- link l_wrist: geometry collision mesh filename=package://example-robot-data/robots/romeo_description/meshe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 scale=1 1 1; visual mesh filename=package://example-robot-data/robots/romeo_description/meshe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 scale=1 1 1
- link r_ankle: geometry collision mesh filename=package://example-robot-data/robots/romeo_description/meshe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 scale=1 1 1; visual mesh filename=package://example-robot-data/robots/romeo_description/meshe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 scale=1 1 1
- link r_wrist: geometry collision mesh filename=package://example-robot-data/robots/romeo_description/meshe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 scale=1 1 1; visual mesh filename=package://example-robot-data/robots/romeo_description/meshe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 scale=1 1 1
- link torso: geometry collision mesh filename=package://example-robot-data/robots/romeo_description/meshe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 scale=1 1 1; visual mesh filename=package://example-robot-data/robots/romeo_description/meshe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 scale=1 1 1

Commit message: Fix romeo robot

File: robots/romeo_description/urdf/romeo.urdf (robot description, URDF)
Before this commit: robot romeo, 82 links, 81 joints
Links:
- link CameraDepth_frame: mass None -> 0.0
- link CameraLeftEye_frame: mass None -> 0.0
- link CameraLeft_frame: mass None -> 0.0
- link CameraRightEye_frame: mass None -> 0.0
- link CameraRight_frame: mass None -> 0.0
- link HeadTouchFront_frame: mass None -> 0.0
- link HeadTouchMiddle_frame: mass None -> 0.0
- link HeadTouchRear_frame: mass None -> 0.0
- link ImuHeadAccelerometer_frame: mass None -> 0.0
- link ImuHeadGyrometer_frame: mass None -> 0.0
- link ImuTorsoAccelerometer_frame: mass None -> 0.0
- link ImuTorsoGyrometer_frame: mass None -> 0.0
- link LFsrCenter_frame: mass None -> 0.0
- link LFsrFL_frame: mass None -> 0.0
- link LFsrFR_frame: mass None -> 0.0
- link LFsrRCenter_frame: mass None -> 0.0
- link RFsrCenter_frame: mass None -> 0.0
- link RFsrFL_frame: mass None -> 0.0
- link RFsrFR_frame: mass None -> 0.0
- link RFsrRCenter_frame: mass None -> 0.0
- link base_link: mass None -> 0.0
- link gaze: mass None -> 0.0
- link l_gripper: mass None -> 0.0
- link l_sole: mass None -> 0.0
- link r_gripper: mass None -> 0.0
- link r_sole: mass None -> 0.0
