Commit message: Universal Robot.

File: robots/ur_description/urdf/ur3_joint_limited_robot.urdf (robot description, URDF)
Before this commit: robot ur3, 11 links, 10 joints
Links:
- link base: mass None -> 0.0
- link ee_link: mass None -> 0.0
- link tool0: mass None -> 0.0

File: robots/ur_description/urdf/ur3_robot.urdf (robot description, URDF)
Before this commit: robot ur3, 11 links, 10 joints
Links:
- link base: mass None -> 0.0
- link ee_link: mass None -> 0.0
- link tool0: mass None -> 0.0

File: robots/ur_description/urdf/ur5_joint_limited_robot.urdf (robot description, URDF)
Before this commit: robot ur5, 11 links, 10 joints
Links:
- link base: mass None -> 0.0
- link ee_link: mass None -> 0.0
- link tool0: mass None -> 0.0
