Commit message: ur5 &_ur5_gripper: set default link mass to 0

File: robots/ur_description/urdf/ur5_gripper.urdf (robot description, URDF)
Before this commit: robot ur5, 11 links, 10 joints
Links:
- link base: mass None -> 0
- link ee_link: mass None -> 0
- link tool0: mass None -> 0

File: robots/ur_description/urdf/ur5_robot.urdf (robot description, URDF)
Before this commit: robot ur5, 11 links, 10 joints
Links:
- link base: mass None -> 0
- link ee_link: mass None -> 0
- link tool0: mass None -> 0
