Commit message: [ur_description] Use meshes from example-robot-data.

File: robots/ur_description/urdf/ur10_joint_limited_robot.urdf (robot description, URDF)
Before this commit: robot ur10, 11 links, 10 joints
Links:
- link base_link: geometry collision mesh filename=package://example-robot-data/robots/ur_description/meshes/u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; visual mesh filename=package://example-robot-data/robots/ur_description/meshes/u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
- link forearm_link: geometry collision mesh filename=package://example-robot-data/robots/ur_description/meshes/u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; visual mesh filename=package://example-robot-data/robots/ur_description/meshes/u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
- link shoulder_link: geometry collision mesh filename=package://example-robot-data/robots/ur_description/meshes/u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; visual mesh filename=package://example-robot-data/robots/ur_description/meshes/u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
- link upper_arm_link: geometry collision mesh filename=package://example-robot-data/robots/ur_description/meshes/u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; visual mesh filename=package://example-robot-data/robots/ur_description/meshes/u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
- link wrist_1_link: geometry collision mesh filename=package://example-robot-data/robots/ur_description/meshes/u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; visual mesh filename=package://example-robot-data/robots/ur_description/meshes/u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
- link wrist_2_link: geometry collision mesh filename=package://example-robot-data/robots/ur_description/meshes/u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; visual mesh filename=package://example-robot-data/robots/ur_description/meshes/u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
- link wrist_3_link: geometry collision mesh filename=package://example-robot-data/robots/ur_description/meshes/u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; visual mesh filename=package://example-robot-data/robots/ur_description/meshes/u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

File: robots/ur_description/urdf/ur10_robot.urdf (robot description, URDF)
Before this commit: robot ur10, 11 links, 10 joints
Links:
- link base_link: geometry collision mesh filename=package://example-robot-data/robots/ur_description/meshes/u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; visual mesh filename=package://example-robot-data/robots/ur_description/meshes/u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
- link forearm_link: geometry collision mesh filename=package://example-robot-data/robots/ur_description/meshes/u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; visual mesh filename=package://example-robot-data/robots/ur_description/meshes/u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
- link shoulder_link: geometry collision mesh filename=package://example-robot-data/robots/ur_description/meshes/u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; visual mesh filename=package://example-robot-data/robots/ur_description/meshes/u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
- link upper_arm_link: geometry collision mesh filename=package://example-robot-data/robots/ur_description/meshes/u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; visual mesh filename=package://example-robot-data/robots/ur_description/meshes/u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
- link wrist_1_link: geometry collision mesh filename=package://example-robot-data/robots/ur_description/meshes/u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; visual mesh filename=package://example-robot-data/robots/ur_description/meshes/u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
- link wrist_2_link: geometry collision mesh filename=package://example-robot-data/robots/ur_description/meshes/u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; visual mesh filename=package://example-robot-data/robots/ur_description/meshes/u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
- link wrist_3_link: geometry collision mesh filename=package://example-robot-data/robots/ur_description/meshes/u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; visual mesh filename=package://example-robot-data/robots/ur_description/meshes/u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

File: robots/ur_description/urdf/ur3_gripper.urdf (robot description, URDF)
Before this commit: robot ur3, 11 links, 10 joints
Links:
- link base_link: geometry collision mesh filename=package://example-robot-data/robots/ur_description/meshes/u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; visual mesh filename=package://example-robot-data/robots/ur_description/meshes/u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
- link forearm_link: geometry collision mesh filename=package://example-robot-data/robots/ur_description/meshes/u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; visual mesh filename=package://example-robot-data/robots/ur_description/meshes/u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
- link shoulder_link: geometry collision mesh filename=package://example-robot-data/robots/ur_description/meshes/u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; visual mesh filename=package://example-robot-data/robots/ur_description/meshes/u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
- link upper_arm_link: geometry collision mesh filename=package://example-robot-data/robots/ur_description/meshes/u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; visual mesh filename=package://example-robot-data/robots/ur_description/meshes/u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
- link wrist_1_link: geometry collision mesh filename=package://example-robot-data/robots/ur_description/meshes/u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; visual mesh filename=package://example-robot-data/robots/ur_description/meshes/u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
- link wrist_2_link: geometry collision mesh filename=package://example-robot-data/robots/ur_description/meshes/u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; visual mesh filename=package://example-robot-data/robots/ur_description/meshes/u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
- link wrist_3_link: geometry collision mesh filename=package://example-robot-data/robots/ur_description/meshes/u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; visual mesh filename=package://example-robot-data/robots/ur_description/meshes/u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

File: robots/ur_description/urdf/ur3_joint_limited_robot.urdf (robot description, URDF)
Before this commit: robot ur3, 11 links, 10 joints
Links:
- link base_link: geometry collision mesh filename=package://example-robot-data/robots/ur_description/meshes/u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; visual mesh filename=package://example-robot-data/robots/ur_description/meshes/u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
- link forearm_link: geometry collision mesh filename=package://example-robot-data/robots/ur_description/meshes/u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; visual mesh filename=package://example-robot-data/robots/ur_description/meshes/u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
- link shoulder_link: geometry collision mesh filename=package://example-robot-data/robots/ur_description/meshes/u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; visual mesh filename=package://example-robot-data/robots/ur_description/meshes/u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
- link upper_arm_link: geometry collision mesh filename=package://example-robot-data/robots/ur_description/meshes/u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; visual mesh filename=package://example-robot-data/robots/ur_description/meshes/u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
- link wrist_1_link: geometry collision mesh filename=package://example-robot-data/robots/ur_description/meshes/u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; visual mesh filename=package://example-robot-data/robots/ur_description/meshes/u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
- link wrist_2_link: geometry collision mesh filename=package://example-robot-data/robots/ur_description/meshes/u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; visual mesh filename=package://example-robot-data/robots/ur_description/meshes/u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
- link wrist_3_link: geometry collision mesh filename=package://example-robot-data/robots/ur_description/meshes/u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; visual mesh filename=package://example-robot-data/robots/ur_description/meshes/u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

File: robots/ur_description/urdf/ur3_robot.urdf (robot description, URDF)
Before this commit: robot ur3, 11 links, 10 joints
Links:
- link base_link: geometry collision mesh filename=package://example-robot-data/robots/ur_description/meshes/u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; visual mesh filename=package://example-robot-data/robots/ur_description/meshes/u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
- link forearm_link: geometry collision mesh filename=package://example-robot-data/robots/ur_description/meshes/u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; visual mesh filename=package://example-robot-data/robots/ur_description/meshes/u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
- link shoulder_link: geometry collision mesh filename=package://example-robot-data/robots/ur_description/meshes/u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; visual mesh filename=package://example-robot-data/robots/ur_description/meshes/u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
- link upper_arm_link: geometry collision mesh filename=package://example-robot-data/robots/ur_description/meshes/u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; visual mesh filename=package://example-robot-data/robots/ur_description/meshes/u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
- link wrist_1_link: geometry collision mesh filename=package://example-robot-data/robots/ur_description/meshes/u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; visual mesh filename=package://example-robot-data/robots/ur_description/meshes/u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
- link wrist_2_link: geometry collision mesh filename=package://example-robot-data/robots/ur_description/meshes/u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; visual mesh filename=package://example-robot-data/robots/ur_description/meshes/u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
- link wrist_3_link: geometry collision mesh filename=package://example-robot-data/robots/ur_description/meshes/u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; visual mesh filename=package://example-robot-data/robots/ur_description/meshes/u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

File: robots/ur_description/urdf/ur5_gripper.urdf (robot description, URDF)
Before this commit: robot ur5, 11 links, 10 joints
Links:
- link base_link: geometry collision mesh filename=package://example-robot-data/robots/ur_description/meshes/u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; visual mesh filename=package://example-robot-data/robots/ur_description/meshes/u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
- link forearm_link: geometry collision mesh filename=package://example-robot-data/robots/ur_description/meshes/u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; visual mesh filename=package://example-robot-data/robots/ur_description/meshes/u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
- link shoulder_link: geometry collision mesh filename=package://example-robot-data/robots/ur_description/meshes/u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; visual mesh filename=package://example-robot-data/robots/ur_description/meshes/u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
- link upper_arm_link: geometry collision mesh filename=package://example-robot-data/robots/ur_description/meshes/u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; visual mesh filename=package://example-robot-data/robots/ur_description/meshes/u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
- link wrist_1_link: geometry collision mesh filename=package://example-robot-data/robots/ur_description/meshes/u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; visual mesh filename=package://example-robot-data/robots/ur_description/meshes/u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
- link wrist_2_link: geometry collision mesh filename=package://example-robot-data/robots/ur_description/meshes/u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; visual mesh filename=package://example-robot-data/robots/ur_description/meshes/u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
- link wrist_3_link: geometry collision mesh filename=package://example-robot-data/robots/ur_description/meshes/u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; visual mesh filename=package://example-robot-data/robots/ur_description/meshes/u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

File: robots/ur_description/urdf/ur5_joint_limited_robot.urdf (robot description, URDF)
Before this commit: robot ur5, 11 links, 10 joints
Links:
- link base_link: geometry collision mesh filename=package://example-robot-data/robots/ur_description/meshes/u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; visual mesh filename=package://example-robot-data/robots/ur_description/meshes/u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
- link forearm_link: geometry collision mesh filename=package://example-robot-data/robots/ur_description/meshes/u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; visual mesh filename=package://example-robot-data/robots/ur_description/meshes/u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
- link shoulder_link: geometry collision mesh filename=package://example-robot-data/robots/ur_description/meshes/u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; visual mesh filename=package://example-robot-data/robots/ur_description/meshes/u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
- link upper_arm_link: geometry collision mesh filename=package://example-robot-data/robots/ur_description/meshes/u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; visual mesh filename=package://example-robot-data/robots/ur_description/meshes/u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
- link wrist_1_link: geometry collision mesh filename=package://example-robot-data/robots/ur_description/meshes/u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; visual mesh filename=package://example-robot-data/robots/ur_description/meshes/u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
- link wrist_2_link: geometry collision mesh filename=package://example-robot-data/robots/ur_description/meshes/u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; visual mesh filename=package://example-robot-data/robots/ur_description/meshes/u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
- link wrist_3_link: geometry collision mesh filename=package://example-robot-data/robots/ur_description/meshes/u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; visual mesh filename=package://example-robot-data/robots/ur_description/meshes/u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

File: robots/ur_description/urdf/ur5_robot.urdf (robot description, URDF)
Before this commit: robot ur5, 11 links, 10 joints
Links:
- link base_link: geometry collision mesh filename=package://example-robot-data/robots/ur_description/meshes/u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; visual mesh filename=package://example-robot-data/robots/ur_description/meshes/u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
- link forearm_link: geometry collision mesh filename=package://example-robot-data/robots/ur_description/meshes/u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; visual mesh filename=package://example-robot-data/robots/ur_description/meshes/u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
- link shoulder_link: geometry collision mesh filename=package://example-robot-data/robots/ur_description/meshes/u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; visual mesh filename=package://example-robot-data/robots/ur_description/meshes/u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
- link upper_arm_link: geometry collision mesh filename=package://example-robot-data/robots/ur_description/meshes/u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; visual mesh filename=package://example-robot-data/robots/ur_description/meshes/u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
- link wrist_1_link: geometry collision mesh filename=package://example-robot-data/robots/ur_description/meshes/u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; visual mesh filename=package://example-robot-data/robots/ur_description/meshes/u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
- link wrist_2_link: geometry collision mesh filename=package://example-robot-data/robots/ur_description/meshes/u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; visual mesh filename=package://example-robot-data/robots/ur_description/meshes/u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
- link wrist_3_link: geometry collision mesh filename=package://example-robot-data/robots/ur_description/meshes/u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; visual mesh filename=package://example-robot-data/robots/ur_description/meshes/u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
