Commit message: Revert "[ur_description] Use meshes from example-robot-data."
This reverts commit 2545adcf0bbecd43ed40d6be03820cb53f3a16d7.

File: robots/ur_description/urdf/ur10_joint_limited_robot.urdf (robot description, URDF)
Before this commit: robot ur10, 11 links, 10 joints
Links:
- link base_link: geometry collision mesh filename=package://ur_description/meshes/ur10/collision/base.stl; visual mesh filename=package://ur_description/meshes/ur10/visual/base.dae
- link forearm_link: geometry collision mesh filename=package://ur_description/meshes/ur10/collision/forearm.stl; visual mesh filename=package://ur_description/meshes/ur10/visual/forearm.dae
- link shoulder_link: geometry collision mesh filename=package://ur_description/meshes/ur10/collision/shoulder.stl; visual mesh filename=package://ur_description/meshes/ur10/visual/shoulder.dae
- link upper_arm_link: geometry collision mesh filename=package://ur_description/meshes/ur10/collision/upperarm.stl; visual mesh filename=package://ur_description/meshes/ur10/visual/upperarm.dae
- link wrist_1_link: geometry collision mesh filename=package://ur_description/meshes/ur10/collision/wrist1.stl; visual mesh filename=package://ur_description/meshes/ur10/visual/wrist1.dae
- link wrist_2_link: geometry collision mesh filename=package://ur_description/meshes/ur10/collision/wrist2.stl; visual mesh filename=package://ur_description/meshes/ur10/visual/wrist2.dae
- link wrist_3_link: geometry collision mesh filename=package://ur_description/meshes/ur10/collision/wrist3.stl; visual mesh filename=package://ur_description/meshes/ur10/visual/wrist3.dae

File: robots/ur_description/urdf/ur10_robot.urdf (robot description, URDF)
Before this commit: robot ur10, 11 links, 10 joints
Links:
- link base_link: geometry collision mesh filename=package://ur_description/meshes/ur10/collision/base.stl; visual mesh filename=package://ur_description/meshes/ur10/visual/base.dae
- link forearm_link: geometry collision mesh filename=package://ur_description/meshes/ur10/collision/forearm.stl; visual mesh filename=package://ur_description/meshes/ur10/visual/forearm.dae
- link shoulder_link: geometry collision mesh filename=package://ur_description/meshes/ur10/collision/shoulder.stl; visual mesh filename=package://ur_description/meshes/ur10/visual/shoulder.dae
- link upper_arm_link: geometry collision mesh filename=package://ur_description/meshes/ur10/collision/upperarm.stl; visual mesh filename=package://ur_description/meshes/ur10/visual/upperarm.dae
- link wrist_1_link: geometry collision mesh filename=package://ur_description/meshes/ur10/collision/wrist1.stl; visual mesh filename=package://ur_description/meshes/ur10/visual/wrist1.dae
- link wrist_2_link: geometry collision mesh filename=package://ur_description/meshes/ur10/collision/wrist2.stl; visual mesh filename=package://ur_description/meshes/ur10/visual/wrist2.dae
- link wrist_3_link: geometry collision mesh filename=package://ur_description/meshes/ur10/collision/wrist3.stl; visual mesh filename=package://ur_description/meshes/ur10/visual/wrist3.dae

File: robots/ur_description/urdf/ur3_gripper.urdf (robot description, URDF)
Before this commit: robot ur3, 11 links, 10 joints
Links:
- link base_link: geometry collision mesh filename=package://ur_description/meshes/ur3/collision/base.stl; visual mesh filename=package://ur_description/meshes/ur3/visual/base.dae
- link forearm_link: geometry collision mesh filename=package://ur_description/meshes/ur3/collision/forearm.stl; visual mesh filename=package://ur_description/meshes/ur3/visual/forearm.dae
- link shoulder_link: geometry collision mesh filename=package://ur_description/meshes/ur3/collision/shoulder.stl; visual mesh filename=package://ur_description/meshes/ur3/visual/shoulder.dae
- link upper_arm_link: geometry collision mesh filename=package://ur_description/meshes/ur3/collision/upperarm.stl; visual mesh filename=package://ur_description/meshes/ur3/visual/upperarm.dae
- link wrist_1_link: geometry collision mesh filename=package://ur_description/meshes/ur3/collision/wrist1.stl; visual mesh filename=package://ur_description/meshes/ur3/visual/wrist1.dae
- link wrist_2_link: geometry collision mesh filename=package://ur_description/meshes/ur3/collision/wrist2.stl; visual mesh filename=package://ur_description/meshes/ur3/visual/wrist2.dae
- link wrist_3_link: geometry collision mesh filename=package://ur_description/meshes/ur3/collision/wrist3.stl; visual mesh filename=package://ur_description/meshes/ur3/visual/wrist3.dae

File: robots/ur_description/urdf/ur3_joint_limited_robot.urdf (robot description, URDF)
Before this commit: robot ur3, 11 links, 10 joints
Links:
- link base_link: geometry collision mesh filename=package://ur_description/meshes/ur3/collision/base.stl; visual mesh filename=package://ur_description/meshes/ur3/visual/base.dae
- link forearm_link: geometry collision mesh filename=package://ur_description/meshes/ur3/collision/forearm.stl; visual mesh filename=package://ur_description/meshes/ur3/visual/forearm.dae
- link shoulder_link: geometry collision mesh filename=package://ur_description/meshes/ur3/collision/shoulder.stl; visual mesh filename=package://ur_description/meshes/ur3/visual/shoulder.dae
- link upper_arm_link: geometry collision mesh filename=package://ur_description/meshes/ur3/collision/upperarm.stl; visual mesh filename=package://ur_description/meshes/ur3/visual/upperarm.dae
- link wrist_1_link: geometry collision mesh filename=package://ur_description/meshes/ur3/collision/wrist1.stl; visual mesh filename=package://ur_description/meshes/ur3/visual/wrist1.dae
- link wrist_2_link: geometry collision mesh filename=package://ur_description/meshes/ur3/collision/wrist2.stl; visual mesh filename=package://ur_description/meshes/ur3/visual/wrist2.dae
- link wrist_3_link: geometry collision mesh filename=package://ur_description/meshes/ur3/collision/wrist3.stl; visual mesh filename=package://ur_description/meshes/ur3/visual/wrist3.dae

File: robots/ur_description/urdf/ur3_robot.urdf (robot description, URDF)
Before this commit: robot ur3, 11 links, 10 joints
Links:
- link base_link: geometry collision mesh filename=package://ur_description/meshes/ur3/collision/base.stl; visual mesh filename=package://ur_description/meshes/ur3/visual/base.dae
- link forearm_link: geometry collision mesh filename=package://ur_description/meshes/ur3/collision/forearm.stl; visual mesh filename=package://ur_description/meshes/ur3/visual/forearm.dae
- link shoulder_link: geometry collision mesh filename=package://ur_description/meshes/ur3/collision/shoulder.stl; visual mesh filename=package://ur_description/meshes/ur3/visual/shoulder.dae
- link upper_arm_link: geometry collision mesh filename=package://ur_description/meshes/ur3/collision/upperarm.stl; visual mesh filename=package://ur_description/meshes/ur3/visual/upperarm.dae
- link wrist_1_link: geometry collision mesh filename=package://ur_description/meshes/ur3/collision/wrist1.stl; visual mesh filename=package://ur_description/meshes/ur3/visual/wrist1.dae
- link wrist_2_link: geometry collision mesh filename=package://ur_description/meshes/ur3/collision/wrist2.stl; visual mesh filename=package://ur_description/meshes/ur3/visual/wrist2.dae
- link wrist_3_link: geometry collision mesh filename=package://ur_description/meshes/ur3/collision/wrist3.stl; visual mesh filename=package://ur_description/meshes/ur3/visual/wrist3.dae

File: robots/ur_description/urdf/ur5_gripper.urdf (robot description, URDF)
Before this commit: robot ur5, 11 links, 10 joints
Links:
- link base_link: geometry collision mesh filename=package://ur_description/meshes/ur5/collision/base.stl; visual mesh filename=package://ur_description/meshes/ur5/visual/base.dae
- link forearm_link: geometry collision mesh filename=package://ur_description/meshes/ur5/collision/forearm.stl; visual mesh filename=package://ur_description/meshes/ur5/visual/forearm.dae
- link shoulder_link: geometry collision mesh filename=package://ur_description/meshes/ur5/collision/shoulder.stl; visual mesh filename=package://ur_description/meshes/ur5/visual/shoulder.dae
- link upper_arm_link: geometry collision mesh filename=package://ur_description/meshes/ur5/collision/upperarm.stl; visual mesh filename=package://ur_description/meshes/ur5/visual/upperarm.dae
- link wrist_1_link: geometry collision mesh filename=package://ur_description/meshes/ur5/collision/wrist1.stl; visual mesh filename=package://ur_description/meshes/ur5/visual/wrist1.dae
- link wrist_2_link: geometry collision mesh filename=package://ur_description/meshes/ur5/collision/wrist2.stl; visual mesh filename=package://ur_description/meshes/ur5/visual/wrist2.dae
- link wrist_3_link: geometry collision mesh filename=package://ur_description/meshes/ur5/collision/wrist3.stl; visual mesh filename=package://ur_description/meshes/ur5/visual/wrist3.dae

File: robots/ur_description/urdf/ur5_joint_limited_robot.urdf (robot description, URDF)
Before this commit: robot ur5, 11 links, 10 joints
Links:
- link base_link: geometry collision mesh filename=package://ur_description/meshes/ur5/collision/base.stl; visual mesh filename=package://ur_description/meshes/ur5/visual/base.dae
- link forearm_link: geometry collision mesh filename=package://ur_description/meshes/ur5/collision/forearm.stl; visual mesh filename=package://ur_description/meshes/ur5/visual/forearm.dae
- link shoulder_link: geometry collision mesh filename=package://ur_description/meshes/ur5/collision/shoulder.stl; visual mesh filename=package://ur_description/meshes/ur5/visual/shoulder.dae
- link upper_arm_link: geometry collision mesh filename=package://ur_description/meshes/ur5/collision/upperarm.stl; visual mesh filename=package://ur_description/meshes/ur5/visual/upperarm.dae
- link wrist_1_link: geometry collision mesh filename=package://ur_description/meshes/ur5/collision/wrist1.stl; visual mesh filename=package://ur_description/meshes/ur5/visual/wrist1.dae
- link wrist_2_link: geometry collision mesh filename=package://ur_description/meshes/ur5/collision/wrist2.stl; visual mesh filename=package://ur_description/meshes/ur5/visual/wrist2.dae
- link wrist_3_link: geometry collision mesh filename=package://ur_description/meshes/ur5/collision/wrist3.stl; visual mesh filename=package://ur_description/meshes/ur5/visual/wrist3.dae

File: robots/ur_description/urdf/ur5_robot.urdf (robot description, URDF)
Before this commit: robot ur5, 11 links, 10 joints
Links:
- link base_link: geometry collision mesh filename=package://ur_description/meshes/ur5/collision/base.stl; visual mesh filename=package://ur_description/meshes/ur5/visual/base.dae
- link forearm_link: geometry collision mesh filename=package://ur_description/meshes/ur5/collision/forearm.stl; visual mesh filename=package://ur_description/meshes/ur5/visual/forearm.dae
- link shoulder_link: geometry collision mesh filename=package://ur_description/meshes/ur5/collision/shoulder.stl; visual mesh filename=package://ur_description/meshes/ur5/visual/shoulder.dae
- link upper_arm_link: geometry collision mesh filename=package://ur_description/meshes/ur5/collision/upperarm.stl; visual mesh filename=package://ur_description/meshes/ur5/visual/upperarm.dae
- link wrist_1_link: geometry collision mesh filename=package://ur_description/meshes/ur5/collision/wrist1.stl; visual mesh filename=package://ur_description/meshes/ur5/visual/wrist1.dae
- link wrist_2_link: geometry collision mesh filename=package://ur_description/meshes/ur5/collision/wrist2.stl; visual mesh filename=package://ur_description/meshes/ur5/visual/wrist2.dae
- link wrist_3_link: geometry collision mesh filename=package://ur_description/meshes/ur5/collision/wrist3.stl; visual mesh filename=package://ur_description/meshes/ur5/visual/wrist3.dae

Commit message: ur_description: fix inertia in ur3 & ur10

File: robots/ur_description/urdf/ur10_joint_limited_robot.urdf (robot description, URDF)
Before this commit: robot ur10, 11 links, 10 joints
Links:
- link base: mass None -> 0.0
- link ee_link: mass None -> 0.0
- link tool0: mass None -> 0.0

File: robots/ur_description/urdf/ur3_gripper.urdf (robot description, URDF)
Before this commit: robot ur3, 11 links, 10 joints
Links:
- link base: mass None -> 0.0
- link ee_link: mass None -> 0.0
- link tool0: mass None -> 0.0
