Commit message: [tiago_description] Update paths - cf. #19

File: robots/tiago_description/robots/tiago.urdf (robot description, URDF)
Before this commit: robot tiago, 78 links, 77 joints
Links:
- link arm_1_link: geometry collision mesh filename=package://example-robot-data/robots/tiago_description/meshe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 scale=1 1 1; visual mesh filename=package://example-robot-data/robots/tiago_description/meshe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 scale=1 1 1
- link arm_2_link: geometry collision mesh filename=package://example-robot-data/robots/tiago_description/meshe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 scale=1 1 1; visual mesh filename=package://example-robot-data/robots/tiago_description/meshe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 scale=1 1 1
- link arm_3_link: geometry collision mesh filename=package://example-robot-data/robots/tiago_description/meshe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 scale=1 1 1; visual mesh filename=package://example-robot-data/robots/tiago_description/meshe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 scale=1 1 1
- link arm_4_link: geometry collision mesh filename=package://example-robot-data/robots/tiago_description/meshe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 scale=1 1 1; visual mesh filename=package://example-robot-data/robots/tiago_description/meshe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 scale=1 1 1
- link arm_5_link: geometry collision mesh filename=package://example-robot-data/robots/tiago_description/meshe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 scale=1 1 1; visual mesh filename=package://example-robot-data/robots/tiago_description/meshe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 scale=1 1 1
- link arm_6_link: geometry collision mesh filename=package://example-robot-data/robots/tiago_description/meshe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 scale=1 1 1; visual mesh filename=package://example-robot-data/robots/tiago_description/meshe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 scale=1 1 1
- link base_antenna_left_link: geometry collision cylinder length=0.17 radius=0.005; visual mesh filename=package://example-robot-data/robots/tiago_description/meshe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
- link base_antenna_right_link: geometry collision cylinder length=0.17 radius=0.005; visual mesh filename=package://example-robot-data/robots/tiago_description/meshe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
- link base_cover_link: geometry visual mesh filename=package://example-robot-data/robots/tiago_description/meshe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
- link base_link: geometry collision mesh filename=package://example-robot-data/robots/tiago_description/meshe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; visual mesh filename=package://example-robot-data/robots/tiago_description/meshe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
- link caster_back_left_1_link: geometry visual mesh filename=package://example-robot-data/robots/tiago_description/meshe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
- link caster_back_left_2_link: geometry collision sphere radius=0.025; visual mesh filename=package://example-robot-data/robots/tiago_description/meshe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
- link caster_back_right_1_link: geometry visual mesh filename=package://example-robot-data/robots/tiago_description/meshe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
- link caster_back_right_2_link: geometry collision sphere radius=0.025; visual mesh filename=package://example-robot-data/robots/tiago_description/meshe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
- link caster_front_left_1_link: geometry visual mesh filename=package://example-robot-data/robots/tiago_description/meshe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
- link caster_front_left_2_link: geometry collision sphere radius=0.025; visual mesh filename=package://example-robot-data/robots/tiago_description/meshe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
- link caster_front_right_1_link: geometry visual mesh filename=package://example-robot-data/robots/tiago_description/meshe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
- link caster_front_right_2_link: geometry collision sphere radius=0.025; visual mesh filename=package://example-robot-data/robots/tiago_description/meshe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
- link hand_index_abd_link: geometry collision mesh filename=package://example-robot-data/robots/tiago_description/meshe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 scale=1 1 1; visual mesh filename=package://example-robot-data/robots/tiago_description/meshe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 scale=1 1 1
- link hand_index_flex_1_link: geometry collision mesh filename=package://example-robot-data/robots/tiago_description/meshe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; visual mesh filename=package://example-robot-data/robots/tiago_description/meshe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
- link hand_index_flex_2_link: geometry collision mesh filename=package://example-robot-data/robots/tiago_description/meshe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; visual mesh filename=package://example-robot-data/robots/tiago_description/meshe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
- link hand_index_flex_3_link: geometry collision mesh filename=package://example-robot-data/robots/tiago_description/meshe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; visual mesh filename=package://example-robot-data/robots/tiago_description/meshe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
- link hand_little_abd_link: geometry collision mesh filename=package://example-robot-data/robots/tiago_description/meshe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 scale=1 1 1; visual mesh filename=package://example-robot-data/robots/tiago_description/meshe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 scale=1 1 1
- link hand_little_flex_1_link: geometry collision mesh filename=package://example-robot-data/robots/tiago_description/meshe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; visual mesh filename=package://example-robot-data/robots/tiago_description/meshe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
- link hand_little_flex_2_link: geometry collision mesh filename=package://example-robot-data/robots/tiago_description/meshe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; visual mesh filename=package://example-robot-data/robots/tiago_description/meshe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
- link hand_little_flex_3_link: geometry collision mesh filename=package://example-robot-data/robots/tiago_description/meshe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; visual mesh filename=package://example-robot-data/robots/tiago_description/meshe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
- link hand_middle_abd_link: geometry collision mesh filename=package://example-robot-data/robots/tiago_description/meshe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 scale=1 1 1; visual mesh filename=package://example-robot-data/robots/tiago_description/meshe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 scale=1 1 1
- link hand_middle_flex_1_link: geometry collision mesh filename=package://example-robot-data/robots/tiago_description/meshe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; visual mesh filename=package://example-robot-data/robots/tiago_description/meshe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
- link hand_middle_flex_2_link: geometry collision mesh filename=package://example-robot-data/robots/tiago_description/meshe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; visual mesh filename=package://example-robot-data/robots/tiago_description/meshe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
- link hand_middle_flex_3_link: geometry collision mesh filename=package://example-robot-data/robots/tiago_description/meshe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; visual mesh filename=package://example-robot-data/robots/tiago_description/meshe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
- link hand_palm_link: geometry collision mesh filename=package://example-robot-data/robots/tiago_description/meshe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 scale=1 1 1; visual mesh filename=package://example-robot-data/robots/tiago_description/meshe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 scale=1 1 1
- link hand_ring_abd_link: geometry collision mesh filename=package://example-robot-data/robots/tiago_description/meshe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 scale=1 1 1; visual mesh filename=package://example-robot-data/robots/tiago_description/meshe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 scale=1 1 1
- link hand_ring_flex_1_link: geometry collision mesh filename=package://example-robot-data/robots/tiago_description/meshe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; visual mesh filename=package://example-robot-data/robots/tiago_description/meshe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
- link hand_ring_flex_2_link: geometry collision mesh filename=package://example-robot-data/robots/tiago_description/meshe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; visual mesh filename=package://example-robot-data/robots/tiago_description/meshe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
- link hand_ring_flex_3_link: geometry collision mesh filename=package://example-robot-data/robots/tiago_description/meshe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; visual mesh filename=package://example-robot-data/robots/tiago_description/meshe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
- link hand_thumb_abd_link: geometry collision mesh filename=package://example-robot-data/robots/tiago_description/meshe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 scale=1 1 1; visual mesh filename=package://example-robot-data/robots/tiago_description/meshe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 scale=1 1 1
- link hand_thumb_flex_1_link: geometry collision mesh filename=package://example-robot-data/robots/tiago_description/meshe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; visual mesh filename=package://example-robot-data/robots/tiago_description/meshe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
- link hand_thumb_flex_2_link: geometry collision mesh filename=package://example-robot-data/robots/tiago_description/meshe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; visual mesh filename=package://example-robot-data/robots/tiago_description/meshe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
- link head_1_link: geometry collision mesh filename=package://example-robot-data/robots/tiago_description/meshe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 scale=1 1 1; visual mesh filename=package://example-robot-data/robots/tiago_description/meshe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 scale=1 1 1
- link head_2_link: geometry collision mesh filename=package://example-robot-data/robots/tiago_description/meshe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 scale=1 1 1; visual mesh filename=package://example-robot-data/robots/tiago_description/meshe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 scale=1 1 1
- link torso_fixed_link: geometry collision box size=0.25 0.25 0.1; collision box size=0.4 0.25 0.04
- link torso_lift_link: geometry collision mesh filename=package://example-robot-data/robots/tiago_description/meshe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 scale=1 1 1; collision mesh filename=package://example-robot-data/robots/tiago_description/meshe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 scale=1 1 1
- link wheel_left_link: geometry collision cylinder length=0.04 radius=0.0985; visual mesh filename=package://example-robot-data/robots/tiago_description/meshe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
- link wheel_right_link: geometry collision cylinder length=0.04 radius=0.0985; visual mesh filename=package://example-robot-data/robots/tiago_description/meshe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

File: robots/tiago_description/robots/tiago_no_hand.urdf (robot description, URDF)
Before this commit: robot tiago, 38 links, 37 joints
Links:
- link arm_1_link: geometry collision mesh filename=package://example-robot-data/robots/tiago_description/meshe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 scale=1 1 1; visual mesh filename=package://example-robot-data/robots/tiago_description/meshe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 scale=1 1 1
- link arm_2_link: geometry collision mesh filename=package://example-robot-data/robots/tiago_description/meshe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 scale=1 1 1; visual mesh filename=package://example-robot-data/robots/tiago_description/meshe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 scale=1 1 1
- link arm_3_link: geometry collision mesh filename=package://example-robot-data/robots/tiago_description/meshe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 scale=1 1 1; visual mesh filename=package://example-robot-data/robots/tiago_description/meshe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 scale=1 1 1
- link arm_4_link: geometry collision mesh filename=package://example-robot-data/robots/tiago_description/meshe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 scale=1 1 1; visual mesh filename=package://example-robot-data/robots/tiago_description/meshe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 scale=1 1 1
- link arm_5_link: geometry collision mesh filename=package://example-robot-data/robots/tiago_description/meshe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 scale=1 1 1; visual mesh filename=package://example-robot-data/robots/tiago_description/meshe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 scale=1 1 1
- link arm_6_link: geometry collision mesh filename=package://example-robot-data/robots/tiago_description/meshe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 scale=1 1 1; visual mesh filename=package://example-robot-data/robots/tiago_description/meshe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 scale=1 1 1
- link base_antenna_left_link: geometry collision cylinder length=0.17 radius=0.005; visual mesh filename=package://example-robot-data/robots/tiago_description/meshe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
- link base_antenna_right_link: geometry collision cylinder length=0.17 radius=0.005; visual mesh filename=package://example-robot-data/robots/tiago_description/meshe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
- link base_cover_link: geometry visual mesh filename=package://example-robot-data/robots/tiago_description/meshe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
- link base_link: geometry collision mesh filename=package://example-robot-data/robots/tiago_description/meshe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; visual mesh filename=package://example-robot-data/robots/tiago_description/meshe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
- link caster_back_left_1_link: geometry visual mesh filename=package://example-robot-data/robots/tiago_description/meshe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
- link caster_back_left_2_link: geometry collision sphere radius=0.025; visual mesh filename=package://example-robot-data/robots/tiago_description/meshe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
- link caster_back_right_1_link: geometry visual mesh filename=package://example-robot-data/robots/tiago_description/meshe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
- link caster_back_right_2_link: geometry collision sphere radius=0.025; visual mesh filename=package://example-robot-data/robots/tiago_description/meshe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
- link caster_front_left_1_link: geometry visual mesh filename=package://example-robot-data/robots/tiago_description/meshe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
- link caster_front_left_2_link: geometry collision sphere radius=0.025; visual mesh filename=package://example-robot-data/robots/tiago_description/meshe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
- link caster_front_right_1_link: geometry visual mesh filename=package://example-robot-data/robots/tiago_description/meshe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
- link caster_front_right_2_link: geometry collision sphere radius=0.025; visual mesh filename=package://example-robot-data/robots/tiago_description/meshe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
- link head_1_link: geometry collision mesh filename=package://example-robot-data/robots/tiago_description/meshe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 scale=1 1 1; visual mesh filename=package://example-robot-data/robots/tiago_description/meshe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 scale=1 1 1
- link head_2_link: geometry collision mesh filename=package://example-robot-data/robots/tiago_description/meshe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 scale=1 1 1; visual mesh filename=package://example-robot-data/robots/tiago_description/meshe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 scale=1 1 1
- link torso_fixed_link: geometry collision box size=0.25 0.25 0.1; collision box size=0.4 0.25 0.04
- link torso_lift_link: geometry collision mesh filename=package://example-robot-data/robots/tiago_description/meshe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 scale=1 1 1; collision mesh filename=package://example-robot-data/robots/tiago_description/meshe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 scale=1 1 1
- link wheel_left_link: geometry collision cylinder length=0.04 radius=0.0985; visual mesh filename=package://example-robot-data/robots/tiago_description/meshe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
- link wheel_right_link: geometry collision cylinder length=0.04 radius=0.0985; visual mesh filename=package://example-robot-data/robots/tiago_description/meshe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

Commit message: Fix tiago robot

File: robots/tiago_description/robots/tiago.urdf (robot description, URDF)
Before this commit: robot tiago, 78 links, 77 joints
Links:
- link base_footprint: mass None -> 0.0
- link hand_grasping_frame: mass None -> 0.0

File: robots/tiago_description/robots/tiago_no_hand.urdf (robot description, URDF)
Before this commit: robot tiago, 38 links, 37 joints
Links:
- link base_footprint: mass None -> 0.0
