Commit message: tiago_dual: manually tweak robot description
By comparison to tiago.

This was pure pain. Please don't make me do it again.

File: robots/tiago_description/robots/tiago_dual.urdf (robot description, URDF)
Before this commit: robot tiago_dual, 132 links, 131 joints
Links:
- removed link base_laser_link
- removed link base_mic_back_left_link
- removed link base_mic_back_right_link
- removed link base_mic_front_left_link
- removed link base_mic_front_right_link
- removed link base_sonar_01_link
- removed link base_sonar_02_link
- removed link base_sonar_03_link
- added link xtion_depth_frame, mass 0.001
- added link xtion_depth_optical_frame, mass 0.001
- added link xtion_link, mass 0.21970000000
- added link xtion_optical_frame, mass 0.001
- added link xtion_rgb_frame, mass 0.001
- added link xtion_rgb_optical_frame, mass 0.001
- link arm_left_1_link: geometry collision mesh filename=package://example-robot-data/robots/tiago_description/meshe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 scale=1 -1 -1; visual mesh filename=package://example-robot-data/robots/tiago_description/meshe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 scale=1 -1 -1
- link arm_left_2_link: geometry collision mesh filename=package://example-robot-data/robots/tiago_description/meshe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 scale=1 1 -1; visual mesh filename=package://example-robot-data/robots/tiago_description/meshe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 scale=1 1 -1
- link arm_left_3_link: geometry collision mesh filename=package://example-robot-data/robots/tiago_description/meshe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 scale=1 1 -1; visual mesh filename=package://example-robot-data/robots/tiago_description/meshe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 scale=1 1 -1
- link arm_left_4_link: geometry collision mesh filename=package://example-robot-data/robots/tiago_description/meshe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 scale=-1 -1 -1; visual mesh filename=package://example-robot-data/robots/tiago_description/meshe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 scale=-1 -1 -1
- link arm_left_5_link: geometry collision mesh filename=package://example-robot-data/robots/tiago_description/meshe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 scale=-1 -1 -1; visual mesh filename=package://example-robot-data/robots/tiago_description/meshe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 scale=-1 -1 -1
- link arm_left_6_link: geometry collision mesh filename=package://example-robot-data/robots/tiago_description/meshe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 scale=-1 1 1; visual mesh filename=package://example-robot-data/robots/tiago_description/meshe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 scale=-1 1 1
- link arm_right_1_link: geometry collision mesh filename=package://example-robot-data/robots/tiago_description/meshe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 scale=1 -1 1; visual mesh filename=package://example-robot-data/robots/tiago_description/meshe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 scale=1 -1 1
- link arm_right_2_link: geometry collision mesh filename=package://example-robot-data/robots/tiago_description/meshe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 scale=1 1 1; visual mesh filename=package://example-robot-data/robots/tiago_description/meshe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 scale=1 1 1
- link arm_right_3_link: geometry collision mesh filename=package://example-robot-data/robots/tiago_description/meshe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 scale=1 1 1; visual mesh filename=package://example-robot-data/robots/tiago_description/meshe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 scale=1 1 1
- link arm_right_4_link: geometry collision mesh filename=package://example-robot-data/robots/tiago_description/meshe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 scale=1 1 1; visual mesh filename=package://example-robot-data/robots/tiago_description/meshe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 scale=1 1 1
- link arm_right_5_link: geometry collision mesh filename=package://example-robot-data/robots/tiago_description/meshe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 scale=1 1 1; visual mesh filename=package://example-robot-data/robots/tiago_description/meshe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 scale=1 1 1
- link arm_right_6_link: geometry collision mesh filename=package://example-robot-data/robots/tiago_description/meshe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 scale=1 1 1; visual mesh filename=package://example-robot-data/robots/tiago_description/meshe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 scale=1 1 1
- link base_antenna_left_link: geometry collision cylinder length=0.17 radius=0.005; visual mesh filename=package://example-robot-data/robots/tiago_description/meshe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
- link base_antenna_right_link: geometry collision cylinder length=0.17 radius=0.005; visual mesh filename=package://example-robot-data/robots/tiago_description/meshe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
- link base_cover_link: geometry visual mesh filename=package://example-robot-data/robots/tiago_description/meshe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
- link base_footprint: mass None -> 0.0
- link base_link: geometry collision mesh filename=package://example-robot-data/robots/tiago_description/meshe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; visual mesh filename=package://example-robot-data/robots/tiago_description/meshe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
- link caster_back_left_1_link: geometry visual mesh filename=package://example-robot-data/robots/tiago_description/meshe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
- link caster_back_left_2_link: geometry collision sphere radius=0.025; visual mesh filename=package://example-robot-data/robots/tiago_description/meshe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
- link caster_back_right_1_link: geometry visual mesh filename=package://example-robot-data/robots/tiago_description/meshe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
- link caster_back_right_2_link: geometry collision sphere radius=0.025; visual mesh filename=package://example-robot-data/robots/tiago_description/meshe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
- link caster_front_left_1_link: geometry visual mesh filename=package://example-robot-data/robots/tiago_description/meshe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
- link caster_front_left_2_link: geometry collision sphere radius=0.025; visual mesh filename=package://example-robot-data/robots/tiago_description/meshe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
- link caster_front_right_1_link: geometry visual mesh filename=package://example-robot-data/robots/tiago_description/meshe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
- link caster_front_right_2_link: geometry collision sphere radius=0.025; visual mesh filename=package://example-robot-data/robots/tiago_description/meshe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
- link hand_left_index_abd_link: geometry collision mesh filename=package://example-robot-data/robots/tiago_description/meshe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 scale=1 1 -1; visual mesh filename=package://example-robot-data/robots/tiago_description/meshe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 scale=1 1 -1
- link hand_left_index_flex_1_link: geometry collision mesh filename=package://example-robot-data/robots/tiago_description/meshe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; visual mesh filename=package://example-robot-data/robots/tiago_description/meshe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
- link hand_left_index_flex_2_link: geometry collision mesh filename=package://example-robot-data/robots/tiago_description/meshe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; visual mesh filename=package://example-robot-data/robots/tiago_description/meshe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
- link hand_left_index_flex_3_link: geometry collision mesh filename=package://example-robot-data/robots/tiago_description/meshe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; visual mesh filename=package://example-robot-data/robots/tiago_description/meshe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
- link hand_left_little_abd_link: geometry collision mesh filename=package://example-robot-data/robots/tiago_description/meshe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 scale=1 1 -1; visual mesh filename=package://example-robot-data/robots/tiago_description/meshe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 scale=1 1 -1
- link hand_left_little_flex_1_link: geometry collision mesh filename=package://example-robot-data/robots/tiago_description/meshe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; visual mesh filename=package://example-robot-data/robots/tiago_description/meshe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
- link hand_left_little_flex_2_link: geometry collision mesh filename=package://example-robot-data/robots/tiago_description/meshe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; visual mesh filename=package://example-robot-data/robots/tiago_description/meshe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
- link hand_left_little_flex_3_link: geometry collision mesh filename=package://example-robot-data/robots/tiago_description/meshe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; visual mesh filename=package://example-robot-data/robots/tiago_description/meshe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
- link hand_left_middle_abd_link: geometry collision mesh filename=package://example-robot-data/robots/tiago_description/meshe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 scale=1 1 -1; visual mesh filename=package://example-robot-data/robots/tiago_description/meshe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 scale=1 1 -1
- link hand_left_middle_flex_1_link: geometry collision mesh filename=package://example-robot-data/robots/tiago_description/meshe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; visual mesh filename=package://example-robot-data/robots/tiago_description/meshe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
- link hand_left_middle_flex_2_link: geometry collision mesh filename=package://example-robot-data/robots/tiago_description/meshe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; visual mesh filename=package://example-robot-data/robots/tiago_description/meshe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
- link hand_left_middle_flex_3_link: geometry collision mesh filename=package://example-robot-data/robots/tiago_description/meshe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; visual mesh filename=package://example-robot-data/robots/tiago_description/meshe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
- link hand_left_palm_link: geometry collision mesh filename=package://example-robot-data/robots/tiago_description/meshe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 scale=1 1 -1; visual mesh filename=package://example-robot-data/robots/tiago_description/meshe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 scale=1 1 -1
- link hand_left_ring_abd_link: geometry collision mesh filename=package://example-robot-data/robots/tiago_description/meshe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 scale=1 1 -1; visual mesh filename=package://example-robot-data/robots/tiago_description/meshe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 scale=1 1 -1
- link hand_left_ring_flex_1_link: geometry collision mesh filename=package://example-robot-data/robots/tiago_description/meshe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; visual mesh filename=package://example-robot-data/robots/tiago_description/meshe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
- link hand_left_ring_flex_2_link: geometry collision mesh filename=package://example-robot-data/robots/tiago_description/meshe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; visual mesh filename=package://example-robot-data/robots/tiago_description/meshe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
- link hand_left_ring_flex_3_link: geometry collision mesh filename=package://example-robot-data/robots/tiago_description/meshe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; visual mesh filename=package://example-robot-data/robots/tiago_description/meshe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
- link hand_left_thumb_abd_link: geometry collision mesh filename=package://example-robot-data/robots/tiago_description/meshe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 scale=1 -1 1; visual mesh filename=package://example-robot-data/robots/tiago_description/meshe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 scale=1 1 -1
- link hand_left_thumb_flex_1_link: geometry collision mesh filename=package://example-robot-data/robots/tiago_description/meshe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; visual mesh filename=package://example-robot-data/robots/tiago_description/meshe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
- link hand_left_thumb_flex_2_link: geometry collision mesh filename=package://example-robot-data/robots/tiago_description/meshe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; visual mesh filename=package://example-robot-data/robots/tiago_description/meshe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
- link hand_right_index_abd_link: geometry collision mesh filename=package://example-robot-data/robots/tiago_description/meshe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 scale=1 1 1; visual mesh filename=package://example-robot-data/robots/tiago_description/meshe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 scale=1 1 1
- link hand_right_index_flex_1_link: geometry collision mesh filename=package://example-robot-data/robots/tiago_description/meshe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; visual mesh filename=package://example-robot-data/robots/tiago_description/meshe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
- link hand_right_index_flex_2_link: geometry collision mesh filename=package://example-robot-data/robots/tiago_description/meshe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; visual mesh filename=package://example-robot-data/robots/tiago_description/meshe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
- link hand_right_index_flex_3_link: geometry collision mesh filename=package://example-robot-data/robots/tiago_description/meshe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; visual mesh filename=package://example-robot-data/robots/tiago_description/meshe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
- link hand_right_little_abd_link: geometry collision mesh filename=package://example-robot-data/robots/tiago_description/meshe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 scale=1 1 1; visual mesh filename=package://example-robot-data/robots/tiago_description/meshe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 scale=1 1 1
- link hand_right_little_flex_1_link: geometry collision mesh filename=package://example-robot-data/robots/tiago_description/meshe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; visual mesh filename=package://example-robot-data/robots/tiago_description/meshe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
- link hand_right_little_flex_2_link: geometry collision mesh filename=package://example-robot-data/robots/tiago_description/meshe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; visual mesh filename=package://example-robot-data/robots/tiago_description/meshe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
- link hand_right_little_flex_3_link: geometry collision mesh filename=package://example-robot-data/robots/tiago_description/meshe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; visual mesh filename=package://example-robot-data/robots/tiago_description/meshe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
- link hand_right_middle_abd_link: geometry collision mesh filename=package://example-robot-data/robots/tiago_description/meshe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 scale=1 1 1; visual mesh filename=package://example-robot-data/robots/tiago_description/meshe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 scale=1 1 1
- link hand_right_middle_flex_1_link: geometry collision mesh filename=package://example-robot-data/robots/tiago_description/meshe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; visual mesh filename=package://example-robot-data/robots/tiago_description/meshe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
- link hand_right_middle_flex_2_link: geometry collision mesh filename=package://example-robot-data/robots/tiago_description/meshe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; visual mesh filename=package://example-robot-data/robots/tiago_description/meshe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
- link hand_right_middle_flex_3_link: geometry collision mesh filename=package://example-robot-data/robots/tiago_description/meshe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; visual mesh filename=package://example-robot-data/robots/tiago_description/meshe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
- link hand_right_palm_link: geometry collision mesh filename=package://example-robot-data/robots/tiago_description/meshe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 scale=1 1 1; visual mesh filename=package://example-robot-data/robots/tiago_description/meshe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 scale=1 1 1
- link hand_right_ring_abd_link: geometry collision mesh filename=package://example-robot-data/robots/tiago_description/meshe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 scale=1 1 1; visual mesh filename=package://example-robot-data/robots/tiago_description/meshe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 scale=1 1 1
- link hand_right_ring_flex_1_link: geometry collision mesh filename=package://example-robot-data/robots/tiago_description/meshe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; visual mesh filename=package://example-robot-data/robots/tiago_description/meshe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
- link hand_right_ring_flex_2_link: geometry collision mesh filename=package://example-robot-data/robots/tiago_description/meshe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; visual mesh filename=package://example-robot-data/robots/tiago_description/meshe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
- link hand_right_ring_flex_3_link: geometry collision mesh filename=package://example-robot-data/robots/tiago_description/meshe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; visual mesh filename=package://example-robot-data/robots/tiago_description/meshe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
- link hand_right_thumb_abd_link: geometry collision mesh filename=package://example-robot-data/robots/tiago_description/meshe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 scale=1 1 1; visual mesh filename=package://example-robot-data/robots/tiago_description/meshe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 scale=1 1 1
- link hand_right_thumb_flex_1_link: geometry collision mesh filename=package://example-robot-data/robots/tiago_description/meshe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; visual mesh filename=package://example-robot-data/robots/tiago_description/meshe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
- link hand_right_thumb_flex_2_link: geometry collision mesh filename=package://example-robot-data/robots/tiago_description/meshe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; visual mesh filename=package://example-robot-data/robots/tiago_description/meshe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
- link head_1_link: geometry collision mesh filename=package://example-robot-data/robots/tiago_description/meshe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 scale=1 1 1; visual mesh filename=package://example-robot-data/robots/tiago_description/meshe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 scale=1 1 1
- link head_2_link: geometry collision mesh filename=package://example-robot-data/robots/tiago_description/meshe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 scale=1 1 1; visual mesh filename=package://example-robot-data/robots/tiago_description/meshe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 scale=1 1 1
- link torso_fixed_link: geometry collision box size=0.25 0.25 0.1; collision box size=0.4 0.25 0.04
- link torso_lift_link: geometry collision mesh filename=package://example-robot-data/robots/tiago_description/meshe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 scale=1 1 1; collision mesh filename=package://example-robot-data/robots/tiago_description/meshe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 scale=1 1 1
- link wheel_left_link: geometry collision sphere radius=0.0985; visual mesh filename=package://example-robot-data/robots/tiago_description/meshe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
- link wheel_right_link: geometry collision sphere radius=0.0985; visual mesh filename=package://example-robot-data/robots/tiago_description/meshe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
Joints:
- removed joint base_laser_joint
- removed joint base_mic_back_left_joint
- removed joint base_mic_back_right_joint
- removed joint base_mic_front_left_joint
- removed joint base_mic_front_right_joint
- removed joint base_sonar_01_joint
- removed joint base_sonar_02_joint
- removed joint base_sonar_03_joint
- added joint xtion_depth_joint: type fixed, parent xtion_link, child xtion_depth_frame, origin xyz=0.0 0.047 0.0 rpy=0 0 0
- added joint xtion_depth_optical_joint: type fixed, parent xtion_depth_frame, child xtion_depth_optical_frame, origin xyz=0 0 0 rpy=-1.57079632679 0.0 -1.57079632679
- added joint xtion_joint: type fixed, parent head_2_link, child xtion_link, origin xyz=0.0908 0.08 0.0 rpy=-1.57079632679 0.0 0.0
- added joint xtion_optical_joint: type fixed, parent xtion_link, child xtion_optical_frame, origin xyz=0 0 0 rpy=-1.57079632679 0.0 -1.57079632679
- added joint xtion_rgb_joint: type fixed, parent xtion_link, child xtion_rgb_frame, origin xyz=0.0 0.022 0.0 rpy=0 0 0
- added joint xtion_rgb_optical_joint: type fixed, parent xtion_rgb_frame, child xtion_rgb_optical_frame, origin xyz=0 0 0 rpy=-1.57079632679 0.0 -1.57079632679

Commit message: tiago_dual: fix frame "link" inertia

File: robots/tiago_description/robots/tiago_dual.urdf (robot description, URDF)
Before this commit: robot tiago_dual, 130 links, 129 joints
Links:
- link hand_left_grasping_frame: mass None -> 0.0
- link hand_right_grasping_frame: mass None -> 0.0
