Commit message: baxter: add grippers

File: robots/baxter_description/urdf/baxter.urdf (robot description, URDF)
Before this commit: robot baxter, 49 links, 48 joints
Links:
- removed link head_camera
- removed link left_gripper_base
- removed link left_hand
- removed link left_hand_accelerometer
- removed link left_hand_camera
- removed link left_hand_camera_axis
- removed link left_hand_range
- removed link right_gripper_base
- removed link right_hand
- removed link right_hand_accelerometer
- removed link right_hand_camera
- removed link right_hand_camera_axis
- removed link right_hand_range
- added link head_camera_link, mass 0.0001
- added link l_gripper_l_finger, mass 0.02; collision box size=0.01 0.0135 0.1127; collision box size=0.01 0.05 0.017
- added link l_gripper_l_finger_tip, mass 0.01; collision box size=0.042 0.0065 0.037; visual mesh filename=package://example-robot-data/robots/baxter_description/mesh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
- added link l_gripper_r_finger, mass 0.02; collision box size=0.01 0.0135 0.1127; collision box size=0.01 0.05 0.017
- added link l_gripper_r_finger_tip, mass 0.01; collision box size=0.042 0.0065 0.037; visual mesh filename=package://example-robot-data/robots/baxter_description/mesh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
- added link left_gripper_base_link, mass 0.3; collision cylinder length=0.1 radius=0.029; visual mesh filename=package://example-robot-data/robots/baxter_description/mesh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
- added link left_hand_accelerometer_link, mass 0.0001; visual box size=0.01 0.01 0.01
- added link left_hand_camera_axis_link, mass 0.0001
- added link left_hand_camera_link, mass 0.0001; visual cylinder length=0.01 radius=0.02
- added link left_hand_link, mass 0.19125; collision cylinder length=0.0464 radius=0.04
- added link left_hand_range_link, mass 0.0001; visual box size=0.005 .02 .005
- added link r_gripper_l_finger, mass 0.02; collision box size=0.01 0.0135 0.1127; collision box size=0.01 0.05 0.017
- added link r_gripper_l_finger_tip, mass 0.01; collision cylinder length=0.037 radius=0.008; visual mesh filename=package://example-robot-data/robots/baxter_description/mesh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
- added link r_gripper_r_finger, mass 0.02; collision box size=0.01 0.0135 0.1127; collision box size=0.01 0.05 0.017
- added link r_gripper_r_finger_tip, mass 0.01; collision cylinder length=0.037 radius=0.008; visual mesh filename=package://example-robot-data/robots/baxter_description/mesh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
- added link right_gripper_base_link, mass 0.3; collision cylinder length=0.1 radius=0.029; visual mesh filename=package://example-robot-data/robots/baxter_description/mesh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
- added link right_hand_accelerometer_link, mass 0.0001; visual box size=0.01 0.01 0.01
- added link right_hand_camera_axis_link, mass 0.0001
- added link right_hand_camera_link, mass 0.0001; visual cylinder length=0.01 radius=0.02
- added link right_hand_link, mass 0.19125; collision cylinder length=0.0464 radius=0.04
- added link right_hand_range_link, mass 0.0001; visual box size=0.005 .02 .005
- link left_gripper: geometry 
- link right_gripper: geometry 
Joints:
- removed joint head_camera
- removed joint left_gripper_base
- removed joint left_hand
- removed joint left_hand_accelerometer
- removed joint left_hand_camera
- removed joint left_hand_camera_axis
- removed joint left_hand_range
- removed joint right_gripper_base
- removed joint right_hand
- removed joint right_hand_accelerometer
- removed joint right_hand_camera
- removed joint right_hand_camera_axis
- removed joint right_hand_range
- added joint head_camera_joint: type fixed, parent head, child head_camera_link, origin xyz=0.12839 0 0.06368 rpy=1.75057 0 1.57079632679
- added joint l_gripper_l_finger_joint: type prismatic, parent left_gripper_base_link, child l_gripper_l_finger, origin xyz=0.0 -0.0015 0.02 rpy=0 0 0, axis 0 1 0, limit lower=0.0 upper=0.020833 effort=20.0 velocity=5.0
- added joint l_gripper_l_finger_tip_joint: type fixed, parent l_gripper_l_finger, child l_gripper_l_finger_tip, origin xyz=0.0 0.01725 0.1127 rpy=0 0 0
- added joint l_gripper_r_finger_joint: type prismatic, parent left_gripper_base_link, child l_gripper_r_finger, origin xyz=0.0 0.0015 0.02 rpy=0 0 0, axis 0 1 0, limit lower=-0.020833 upper=0.0 effort=20.0 velocity=5.0, mimic joint=l_gripper_l_finger_joint multiplier=-1.0
- added joint l_gripper_r_finger_tip_joint: type fixed, parent l_gripper_r_finger, child l_gripper_r_finger_tip, origin xyz=0.0 -0.01725 0.1127 rpy=0 0 0
- added joint left_gripper_base_joint: type fixed, parent left_hand_link, child left_gripper_base_link, origin xyz=0 0 0.025 rpy=0 0 0
- added joint left_hand_accelerometer_joint: type fixed, parent left_hand_link, child left_hand_accelerometer_link, origin xyz=0.00198 0.000133 -0.0146 rpy=0 0 0
- added joint left_hand_camera_axis_joint: type fixed, parent left_hand_link, child left_hand_camera_axis_link, origin xyz=0.03825 0.012 0.015355 rpy=0 0 0
- added joint left_hand_camera_joint: type fixed, parent left_hand_link, child left_hand_camera_link, origin xyz=0.03825 0.012 0.015355 rpy=0 0 -1.57079633
- added joint left_hand_joint: type fixed, parent left_wrist, child left_hand_link, origin xyz=0 0 0.11355 rpy=0 0 0, axis 0 0 1
- added joint left_hand_range_joint: type fixed, parent left_hand_link, child left_hand_range_link, origin xyz=0.032 -0.020245 0.0288 rpy=0 -1.57079632679 -1.57079632679
- added joint r_gripper_l_finger_joint: type prismatic, parent right_gripper_base_link, child r_gripper_l_finger, origin xyz=0.0 -0.0015 0.02 rpy=0 0 0, axis 0 1 0, limit lower=0.0 upper=0.020833 effort=20.0 velocity=5.0
- added joint r_gripper_l_finger_tip_joint: type fixed, parent r_gripper_l_finger, child r_gripper_l_finger_tip, origin xyz=0.0 0.01725 0.1127 rpy=0 0 0
- added joint r_gripper_r_finger_joint: type prismatic, parent right_gripper_base_link, child r_gripper_r_finger, origin xyz=0.0 0.0015 0.02 rpy=0 0 0, axis 0 1 0, limit lower=-0.020833 upper=0.0 effort=20.0 velocity=5.0, mimic joint=r_gripper_l_finger_joint multiplier=-1.0
- added joint r_gripper_r_finger_tip_joint: type fixed, parent r_gripper_r_finger, child r_gripper_r_finger_tip, origin xyz=0.0 -0.01725 0.1127 rpy=0 0 0
- added joint right_gripper_base_joint: type fixed, parent right_hand_link, child right_gripper_base_link, origin xyz=0 0 0.025 rpy=0 0 0
- added joint right_hand_accelerometer_joint: type fixed, parent right_hand_link, child right_hand_accelerometer_link, origin xyz=0.00198 0.000133 -0.0146 rpy=0 0 0
- added joint right_hand_camera_axis_joint: type fixed, parent right_hand_link, child right_hand_camera_axis_link, origin xyz=0.03825 0.012 0.015355 rpy=0 0 0
- added joint right_hand_camera_joint: type fixed, parent right_hand_link, child right_hand_camera_link, origin xyz=0.03825 0.012 0.015355 rpy=0 0 -1.57079633
- added joint right_hand_joint: type fixed, parent right_wrist, child right_hand_link, origin xyz=0 0 0.11355 rpy=0 0 0, axis 0 0 1
- added joint right_hand_range_joint: type fixed, parent right_hand_link, child right_hand_range_link, origin xyz=0.032 -0.020245 0.0288 rpy=0 -1.57079632679 -1.57079632679
- joint head_pan: limit lower=-1.57079632679 upper=1.57079632679 effort=50000 velocity=10000 -> lower=-1.3963 upper=1.3963 effort=50000 velocity=10000
- joint left_endpoint: origin xyz=0.0 0 0.025 rpy=0 0 0 -> xyz=0 0 0.1327 rpy=0 0 0; parent left_gripper_base -> left_gripper_base_link
- joint left_s1: limit lower=-2.147 upper=1.047 effort=100.0 velocity=1.5 -> lower=-2.147 upper=1.047 effort=50.0 velocity=1.5
- joint right_endpoint: origin xyz=0.0 0 0.025 rpy=0 0 0 -> xyz=0 0 0.1327 rpy=0 0 0; parent right_gripper_base -> right_gripper_base_link
- joint right_s1: limit lower=-2.147 upper=1.047 effort=100.0 velocity=1.5 -> lower=-2.147 upper=1.047 effort=50.0 velocity=1.5
