Commit message: Bolt: Fix URDF path

File: robots/bolt_description/robots/bolt.urdf (robot description, URDF)
Before this commit: robot bolt, 9 links, 8 joints
Links:
- link FL_FOOT: geometry collision mesh filename=package://example-robot-data/robots/bolt_description/meshes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; visual mesh filename=package://example-robot-data/robots/bolt_description/meshes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
- link FL_LOWER_LEG: geometry collision mesh filename=package://example-robot-data/robots/bolt_description/meshes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; visual mesh filename=package://example-robot-data/robots/bolt_description/meshes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
- link FL_SHOULDER: geometry collision mesh filename=package://example-robot-data/robots/bolt_description/meshes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; visual mesh filename=package://example-robot-data/robots/bolt_description/meshes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
- link FL_UPPER_LEG: geometry collision mesh filename=package://example-robot-data/robots/bolt_description/meshes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; visual mesh filename=package://example-robot-data/robots/bolt_description/meshes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
- link FR_FOOT: geometry collision mesh filename=package://example-robot-data/robots/bolt_description/meshes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; visual mesh filename=package://example-robot-data/robots/bolt_description/meshes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
- link FR_LOWER_LEG: geometry collision mesh filename=package://example-robot-data/robots/bolt_description/meshes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; visual mesh filename=package://example-robot-data/robots/bolt_description/meshes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
- link FR_SHOULDER: geometry collision mesh filename=package://example-robot-data/robots/bolt_description/meshes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; visual mesh filename=package://example-robot-data/robots/bolt_description/meshes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
- link FR_UPPER_LEG: geometry collision mesh filename=package://example-robot-data/robots/bolt_description/meshes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; visual mesh filename=package://example-robot-data/robots/bolt_description/meshes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
- link base_link: geometry collision mesh filename=package://example-robot-data/robots/bolt_description/meshes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; visual mesh filename=package://example-robot-data/robots/bolt_description/meshes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
