Commit message: [double_pendulum_description] Update paths - cf. #19

File: robots/double_pendulum_description/urdf/double_pendulum.urdf (robot description, URDF)
Before this commit: robot 2dof_planar, 3 links, 2 joints
Links:
- link base_link: geometry collision mesh filename=package://example-robot-data/robots/double_pendulum_descrip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; visual mesh filename=package://example-robot-data/robots/double_pendulum_descrip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
- link link1: geometry collision mesh filename=package://example-robot-data/robots/double_pendulum_descrip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; visual mesh filename=package://example-robot-data/robots/double_pendulum_descrip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
- link link2: geometry collision mesh filename=package://example-robot-data/robots/double_pendulum_descrip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; visual mesh filename=package://example-robot-data/robots/double_pendulum_descrip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

Commit message: Make double_pendulum's joints unbounded revolute (continuous)

File: robots/double_pendulum_description/urdf/double_pendulum.urdf (robot description, URDF)
Before this commit: robot 2dof_planar, 3 links, 2 joints
Joints:
- joint joint1: type revolute -> continuous
- joint joint2: type revolute -> continuous
