Commit message: fix inertia on finger_edu & a1, ref #68

File: robots/a1_description/urdf/a1.urdf (robot description, URDF)
Before this commit: robot a1, 23 links, 22 joints
Links:
- link FL_thigh_shoulder: mass None -> 0
- link FR_thigh_shoulder: mass None -> 0
- link RL_thigh_shoulder: mass None -> 0
- link RR_thigh_shoulder: mass None -> 0
