Commit message: removed useless folder and plugins from the urdf

File: robots/asr_twodof_description/urdf/TwoDofs.urdf (robot description, URDF)
Before this commit: robot twodofs, 5 links, 4 joints
Links:
- link Link1: geometry visual mesh filename=package://example-robot-data/robots/asr_twodof_description/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; visual mesh filename=package://example-robot-data/robots/asr_twodof_description/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
- link Link2: geometry visual mesh filename=package://example-robot-data/robots/asr_twodof_description/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; visual mesh filename=package://example-robot-data/robots/asr_twodof_description/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
- link ground: geometry visual mesh filename=package://example-robot-data/robots/asr_twodof_description/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; visual mesh filename=package://example-robot-data/robots/asr_twodof_description/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

Commit message: fix pybullet for asr

File: robots/asr_twodof_description/urdf/TwoDofs.urdf (robot description, URDF)
Before this commit: robot twodofs, 5 links, 4 joints
Links:
- link Tip: mass None -> 0
