Commit message: simple_humanoid: add mesh, update srdf with rotor info, urdf with colliison info

File: robots/simple_humanoid_description/urdf/simple_humanoid.urdf (robot description, URDF)
Before this commit: robot simple_humanoid, 31 links, 30 joints
Links:
- link BODY: geometry collision cylinder length=1 radius=1; collision mesh filename=package://simple_humanoid_description/box.stl

Commit message: simple_humanoid: fix mesh path

File: robots/simple_humanoid_description/urdf/simple_humanoid.urdf (robot description, URDF)
Before this commit: robot simple_humanoid, 31 links, 30 joints
Links:
- link BODY: geometry collision cylinder length=1 radius=1; collision mesh filename=package://example-robot-data/robots/simple_humanoid_descrip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
