Commit message: adding the hand to the urdf

File: robots/panda_description/urdf/panda_collision.urdf (robot description, URDF)
Before this commit: robot panda, 13 links, 12 joints
Links:
- link panda_hand: geometry collision box size=40e-3 20e-2 75e-3; visual mesh filename=package://example-robot-data/robots/panda_description/meshe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

Commit message: fingers as capsules

File: robots/panda_description/urdf/panda_collision.urdf (robot description, URDF)
Before this commit: robot panda, 13 links, 12 joints
Links:
- link panda_leftfinger: geometry collision cylinder length=0.07 radius=0.015; visual mesh filename=package://example-robot-data/robots/panda_description/meshe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
- link panda_rightfinger: geometry collision cylinder length=0.07 radius=0.015; visual mesh filename=package://example-robot-data/robots/panda_description/meshe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

Commit message: hand as capsule

File: robots/panda_description/urdf/panda_collision.urdf (robot description, URDF)
Before this commit: robot panda, 13 links, 12 joints
Links:
- link panda_hand: geometry collision cylinder length=0.25 radius=0.04; visual mesh filename=package://example-robot-data/robots/panda_description/meshe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

Commit message: Fix collision model for Panda

File: robots/panda_description/urdf/panda_collision.urdf (robot description, URDF)
Before this commit: robot panda, 13 links, 12 joints
Links:
- link panda_hand: geometry collision cylinder length=0.15 radius=0.05; collision sphere radius=0.05
- link panda_leftfinger: geometry collision cylinder length=0.03 radius=0.015; collision sphere radius=0.015
- link panda_link7: geometry collision cylinder length=0.01 radius=0.045; collision cylinder length=0.14 radius=0.07
- link panda_rightfinger: geometry collision cylinder length=0.03 radius=0.015; collision sphere radius=0.015
