Commit message: anymal: set 0 mass to camera links

File: robots/anymal_c_simple_description/urdf/anymal.urdf (robot description, URDF)
Before this commit: robot anymal, 78 links, 77 joints
Links:
- link depth_camera_front_camera_parent: mass None -> 0
- link depth_camera_front_color_frame: mass None -> 0
- link depth_camera_front_color_optical_frame: mass None -> 0
- link depth_camera_front_depth_optical_frame: mass None -> 0
- link depth_camera_left_camera_parent: mass None -> 0
- link depth_camera_left_color_frame: mass None -> 0
- link depth_camera_left_color_optical_frame: mass None -> 0
- link depth_camera_left_depth_optical_frame: mass None -> 0
- link depth_camera_rear_camera_parent: mass None -> 0
- link depth_camera_rear_color_frame: mass None -> 0
- link depth_camera_rear_color_optical_frame: mass None -> 0
- link depth_camera_rear_depth_optical_frame: mass None -> 0
- link depth_camera_right_camera_parent: mass None -> 0
- link depth_camera_right_color_frame: mass None -> 0
- link depth_camera_right_color_optical_frame: mass None -> 0
- link depth_camera_right_depth_optical_frame: mass None -> 0
- link wide_angle_camera_front_camera_parent: mass None -> 0
- link wide_angle_camera_rear_camera_parent: mass None -> 0
