Commit message: allegro: adding missing inertia

File: robots/allegro_hand_description/urdf/allegro_left_hand.urdf (robot description, URDF)
Before this commit: robot allegro_hand_left, 21 links, 20 joints
Links:
- removed link base_link
- added link palm_link, mass 0.4154; collision box size=0.0408 0.1130 0.095; visual mesh filename=package://example-robot-data/robots/allegro_hand_descriptio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
- link link_0.0: mass None -> 0.0119
- link link_1.0: mass None -> 0.065
- link link_10.0: mass None -> 0.0355
- link link_11.0: mass None -> 0.0096
- link link_11.0_tip: mass None -> 0.0168
- link link_12.0: mass None -> 0.0176
- link link_13.0: mass None -> 0.0119
- link link_14.0: mass None -> 0.038
- link link_15.0: mass None -> 0.0388
- link link_15.0_tip: mass None -> 0.0168
- link link_2.0: mass None -> 0.0355
- link link_3.0: mass None -> 0.0096
- link link_3.0_tip: mass None -> 0.0168
- link link_4.0: mass None -> 0.0119
- link link_5.0: mass None -> 0.065
- link link_6.0: mass None -> 0.0355
- link link_7.0: mass None -> 0.0096
- link link_7.0_tip: mass None -> 0.0168
- link link_8.0: mass None -> 0.0119
- link link_9.0: mass None -> 0.065
Joints:
- joint joint_0.0: limit lower=-0.47 upper=0.47 effort=0 velocity=0 -> lower=-0.47 upper=0.47 effort=15 velocity=7; parent base_link -> palm_link
- joint joint_1.0: limit lower=-0.196 upper=1.61 effort=0 velocity=0 -> lower=-0.196 upper=1.61 effort=15 velocity=7
- joint joint_10.0: limit lower=-0.174 upper=1.709 effort=0 velocity=0 -> lower=-0.174 upper=1.709 effort=15 velocity=7
- joint joint_11.0: limit lower=-0.227 upper=1.618 effort=0 velocity=0 -> lower=-0.227 upper=1.618 effort=15 velocity=7
- joint joint_12.0: limit lower=0.263 upper=1.396 effort=0 velocity=0 -> lower=0.263 upper=1.396 effort=15 velocity=7; parent base_link -> palm_link
- joint joint_13.0: limit lower=-0.105 upper=1.163 effort=0 velocity=0 -> lower=-0.105 upper=1.163 effort=15 velocity=7
- joint joint_14.0: limit lower=-0.189 upper=1.644 effort=0 velocity=0 -> lower=-0.189 upper=1.644 effort=15 velocity=7
- joint joint_15.0: limit lower=-0.162 upper=1.719 effort=0 velocity=0 -> lower=-0.162 upper=1.719 effort=15 velocity=7
- joint joint_2.0: limit lower=-0.174 upper=1.709 effort=0 velocity=0 -> lower=-0.174 upper=1.709 effort=15 velocity=7
- joint joint_3.0: limit lower=-0.227 upper=1.618 effort=0 velocity=0 -> lower=-0.227 upper=1.618 effort=15 velocity=7
- joint joint_4.0: limit lower=-0.47 upper=0.47 effort=0 velocity=0 -> lower=-0.47 upper=0.47 effort=15 velocity=7; parent base_link -> palm_link
- joint joint_5.0: limit lower=-0.196 upper=1.61 effort=0 velocity=0 -> lower=-0.196 upper=1.61 effort=15 velocity=7
- joint joint_6.0: limit lower=-0.174 upper=1.709 effort=0 velocity=0 -> lower=-0.174 upper=1.709 effort=15 velocity=7
- joint joint_7.0: limit lower=-0.227 upper=1.618 effort=0 velocity=0 -> lower=-0.227 upper=1.618 effort=15 velocity=7
- joint joint_8.0: limit lower=-0.47 upper=0.47 effort=0 velocity=0 -> lower=-0.47 upper=0.47 effort=15 velocity=7; parent base_link -> palm_link
- joint joint_9.0: limit lower=-0.196 upper=1.61 effort=0 velocity=0 -> lower=-0.196 upper=1.61 effort=15 velocity=7

File: robots/allegro_hand_description/urdf/allegro_right_hand.urdf (robot description, URDF)
Before this commit: robot allegro_hand_right, 21 links, 20 joints
Links:
- removed link base_link
- added link palm_link, mass 0.4154; collision box size=0.0408 0.1130 0.095; visual mesh filename=package://example-robot-data/robots/allegro_hand_descriptio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
- link link_0.0: mass None -> 0.0119
- link link_1.0: mass None -> 0.065
- link link_10.0: mass None -> 0.0355
- link link_11.0: mass None -> 0.0096
- link link_11.0_tip: mass None -> 0.0168
- link link_12.0: mass None -> 0.0176
- link link_13.0: mass None -> 0.0119
- link link_14.0: mass None -> 0.038
- link link_15.0: mass None -> 0.0388
- link link_15.0_tip: mass None -> 0.0168
- link link_2.0: mass None -> 0.0355
- link link_3.0: mass None -> 0.0096
- link link_3.0_tip: mass None -> 0.0168
- link link_4.0: mass None -> 0.0119
- link link_5.0: mass None -> 0.065
- link link_6.0: mass None -> 0.0355
- link link_7.0: mass None -> 0.0096
- link link_7.0_tip: mass None -> 0.0168
- link link_8.0: mass None -> 0.0119
- link link_9.0: mass None -> 0.065
Joints:
- joint joint_0.0: limit lower=-0.47 upper=0.47 effort=0 velocity=0 -> lower=-0.47 upper=0.47 effort=15 velocity=7; parent base_link -> palm_link
- joint joint_1.0: limit lower=-0.196 upper=1.61 effort=0 velocity=0 -> lower=-0.196 upper=1.61 effort=15 velocity=7
- joint joint_10.0: limit lower=-0.174 upper=1.709 effort=0 velocity=0 -> lower=-0.174 upper=1.709 effort=15 velocity=7
- joint joint_11.0: limit lower=-0.227 upper=1.618 effort=0 velocity=0 -> lower=-0.227 upper=1.618 effort=15 velocity=7
- joint joint_12.0: limit lower=0.263 upper=1.396 effort=0 velocity=0 -> lower=0.263 upper=1.396 effort=15 velocity=7; parent base_link -> palm_link
- joint joint_13.0: limit lower=-0.105 upper=1.163 effort=0 velocity=0 -> lower=-0.105 upper=1.163 effort=15 velocity=7
- joint joint_14.0: limit lower=-0.189 upper=1.644 effort=0 velocity=0 -> lower=-0.189 upper=1.644 effort=15 velocity=7
- joint joint_15.0: limit lower=-0.162 upper=1.719 effort=0 velocity=0 -> lower=-0.162 upper=1.719 effort=15 velocity=7
- joint joint_2.0: limit lower=-0.174 upper=1.709 effort=0 velocity=0 -> lower=-0.174 upper=1.709 effort=15 velocity=7
- joint joint_3.0: limit lower=-0.227 upper=1.618 effort=0 velocity=0 -> lower=-0.227 upper=1.618 effort=15 velocity=7
- joint joint_4.0: limit lower=-0.47 upper=0.47 effort=0 velocity=0 -> lower=-0.47 upper=0.47 effort=15 velocity=7; parent base_link -> palm_link
- joint joint_5.0: limit lower=-0.196 upper=1.61 effort=0 velocity=0 -> lower=-0.196 upper=1.61 effort=15 velocity=7
- joint joint_6.0: limit lower=-0.174 upper=1.709 effort=0 velocity=0 -> lower=-0.174 upper=1.709 effort=15 velocity=7
- joint joint_7.0: limit lower=-0.227 upper=1.618 effort=0 velocity=0 -> lower=-0.227 upper=1.618 effort=15 velocity=7
- joint joint_8.0: limit lower=-0.47 upper=0.47 effort=0 velocity=0 -> lower=-0.47 upper=0.47 effort=15 velocity=7; parent base_link -> palm_link
- joint joint_9.0: limit lower=-0.196 upper=1.61 effort=0 velocity=0 -> lower=-0.196 upper=1.61 effort=15 velocity=7
