Commit message: [go1][b1] Added fake inertia in base for pybullet

File: robots/b1_description/urdf/b1.urdf (robot description, URDF)
Before this commit: robot b1_description, 31 links, 30 joints
Links:
- link base: mass None -> 1e-6

File: robots/go1_description/urdf/go1.urdf (robot description, URDF)
Before this commit: robot go1, 46 links, 45 joints
Links:
- link base: mass None -> 1e-6
