Commit message: Adding Bravo7+gripper to Bluevolta and Falcon ROVs

File: robots/bluevolta_description/urdf/bluevolta_bravo7_gripper.urdf (robot description, URDF)
Before this commit: robot bravo7_gripper, 12 links, 11 joints
Links:
- added link Thruster_BOTTOM_BL; visual mesh filename=package://example-robot-data/robots/bluevolta_description/m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
- added link Thruster_BOTTOM_BR; visual mesh filename=package://example-robot-data/robots/bluevolta_description/m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
- added link Thruster_BOTTOM_FL; visual mesh filename=package://example-robot-data/robots/bluevolta_description/m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
- added link Thruster_BOTTOM_FR; visual mesh filename=package://example-robot-data/robots/bluevolta_description/m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
- added link Thruster_TOP_B; visual mesh filename=package://example-robot-data/robots/bluevolta_description/m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
- added link Thruster_TOP_FL; visual mesh filename=package://example-robot-data/robots/bluevolta_description/m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
- added link Thruster_TOP_FR; visual mesh filename=package://example-robot-data/robots/bluevolta_description/m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
- added link bluevolta, mass 200.0; collision mesh filename=package://example-robot-data/robots/bluevolta_description/m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; visual mesh filename=package://example-robot-data/robots/bluevolta_description/m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
- added link box_base_bravo; visual box size=0.1 0.1 0.1
Joints:
- added joint Thruster_BOTTOM_BL_joint: type fixed, parent bluevolta, child Thruster_BOTTOM_BL, origin xyz=0.27 -0.6 -0.11 rpy=0.0 0.0 -2.24
- added joint Thruster_BOTTOM_BR_joint: type fixed, parent bluevolta, child Thruster_BOTTOM_BR, origin xyz=-0.27 -0.6 -0.11 rpy=0.0 0.0 -0.9
- added joint Thruster_BOTTOM_FL_joint: type fixed, parent bluevolta, child Thruster_BOTTOM_FL, origin xyz=0.31 0.52 -0.1 rpy=0.0 0.0 -0.9
- added joint Thruster_BOTTOM_FR_joint: type fixed, parent bluevolta, child Thruster_BOTTOM_FR, origin xyz=-0.31 0.52 -0.1 rpy=0.0 0.0 -2.24
- added joint Thruster_TOP_B_joint: type fixed, parent bluevolta, child Thruster_TOP_B, origin xyz=0.0 -0.6 -0.3 rpy=0.0 1.8 -1.57
- added joint Thruster_TOP_FL_joint: type fixed, parent bluevolta, child Thruster_TOP_FL, origin xyz=0.34 0.25 -0.28 rpy=0.0 1.8 0.0
- added joint Thruster_TOP_FR_joint: type fixed, parent bluevolta, child Thruster_TOP_FR, origin xyz=-0.34 0.25 -0.28 rpy=0.0 1.34 0.0
- added joint base2arm: type fixed, parent box_base_bravo, child link1, origin xyz=0 -0.05 -0.05 rpy=3.14 0.0 1.57
- added joint box_base_bravo_joint: type fixed, parent bluevolta, child box_base_bravo, origin xyz=-0.25 0.835 0.17 rpy=0 0 0

File: robots/bluevolta_description/urdf/bluevolta_bravo7_no_ee.urdf (robot description, URDF)
Before this commit: robot bravo7_with_sphere_endeffector, 10 links, 9 joints
Links:
- added link Thruster_BOTTOM_BL; visual mesh filename=package://example-robot-data/robots/bluevolta_description/m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
- added link Thruster_BOTTOM_BR; visual mesh filename=package://example-robot-data/robots/bluevolta_description/m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
- added link Thruster_BOTTOM_FL; visual mesh filename=package://example-robot-data/robots/bluevolta_description/m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
- added link Thruster_BOTTOM_FR; visual mesh filename=package://example-robot-data/robots/bluevolta_description/m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
- added link Thruster_TOP_B; visual mesh filename=package://example-robot-data/robots/bluevolta_description/m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
- added link Thruster_TOP_FL; visual mesh filename=package://example-robot-data/robots/bluevolta_description/m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
- added link Thruster_TOP_FR; visual mesh filename=package://example-robot-data/robots/bluevolta_description/m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
- added link bluevolta, mass 200.0; collision mesh filename=package://example-robot-data/robots/bluevolta_description/m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; visual mesh filename=package://example-robot-data/robots/bluevolta_description/m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
- added link box_base_bravo; visual box size=0.1 0.1 0.1
Joints:
- added joint Thruster_BOTTOM_BL_joint: type fixed, parent bluevolta, child Thruster_BOTTOM_BL, origin xyz=0.27 -0.6 -0.11 rpy=0.0 0.0 -2.24
- added joint Thruster_BOTTOM_BR_joint: type fixed, parent bluevolta, child Thruster_BOTTOM_BR, origin xyz=-0.27 -0.6 -0.11 rpy=0.0 0.0 -0.9
- added joint Thruster_BOTTOM_FL_joint: type fixed, parent bluevolta, child Thruster_BOTTOM_FL, origin xyz=0.31 0.52 -0.1 rpy=0.0 0.0 -0.9
- added joint Thruster_BOTTOM_FR_joint: type fixed, parent bluevolta, child Thruster_BOTTOM_FR, origin xyz=-0.31 0.52 -0.1 rpy=0.0 0.0 -2.24
- added joint Thruster_TOP_B_joint: type fixed, parent bluevolta, child Thruster_TOP_B, origin xyz=0.0 -0.6 -0.3 rpy=0.0 1.8 -1.57
- added joint Thruster_TOP_FL_joint: type fixed, parent bluevolta, child Thruster_TOP_FL, origin xyz=0.34 0.25 -0.28 rpy=0.0 1.8 0.0
- added joint Thruster_TOP_FR_joint: type fixed, parent bluevolta, child Thruster_TOP_FR, origin xyz=-0.34 0.25 -0.28 rpy=0.0 1.34 0.0
- added joint base2arm: type fixed, parent box_base_bravo, child link1, origin xyz=0 -0.05 -0.05 rpy=3.14 0.0 1.57
- added joint box_base_bravo_joint: type fixed, parent bluevolta, child box_base_bravo, origin xyz=-0.25 0.835 0.17 rpy=0 0 0

File: robots/bravo7_description/urdf/bravo7_no_ee.urdf (robot description, URDF)
Before this commit: robot falcon, 19 links, 18 joints
Links:
- removed link BL_propeller
- removed link BR_propeller
- removed link FL_propeller
- removed link FR_propeller
- removed link chassis
- removed link falcon
- removed link floaterL
- removed link floaterR
- removed link top_propeller
Joints:
- removed joint BL_propeller_joint
- removed joint BR_propeller_joint
- removed joint FL_propeller_joint
- removed joint FR_propeller_joint
- removed joint base2arm
- removed joint falcon2chassis
- removed joint falcon2floaterL
- removed joint falcon2floaterR
- removed joint top_propeller_joint

File: robots/falcon_description/urdf/falcon_bravo7_gripper.urdf (robot description, URDF)
Before this commit: robot bluevolta, 19 links, 18 joints
Links:
- removed link Thruster_BOTTOM_BL
- removed link Thruster_BOTTOM_BR
- removed link Thruster_BOTTOM_FL
- removed link Thruster_BOTTOM_FR
- removed link Thruster_TOP_B
- removed link Thruster_TOP_FL
- removed link Thruster_TOP_FR
- removed link bluevolta
- removed link box_base_bravo
- removed link contact_point
- removed link end_effector_ball
- added link BL_propeller; visual mesh filename=package://example-robot-data/robots/falcon_description/mesh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
- added link BR_propeller; visual mesh filename=package://example-robot-data/robots/falcon_description/mesh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
- added link FL_propeller; visual mesh filename=package://example-robot-data/robots/falcon_description/mesh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
- added link FR_propeller; visual mesh filename=package://example-robot-data/robots/falcon_description/mesh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
- added link bravo_finger1_link; collision box size=0.14 0.04 0.045; visual mesh filename=package://example-robot-data/robots/bravo7_description/mesh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
- added link bravo_finger2_link; collision box size=0.14 0.04 0.045; visual mesh filename=package://example-robot-data/robots/bravo7_description/mesh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
- added link bravo_finger_jaws_base_link; collision cylinder length=0.02 radius=0.05; visual mesh filename=package://example-robot-data/robots/bravo7_description/mesh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
- added link chassis, mass 200.0; collision mesh filename=package://example-robot-data/robots/falcon_description/mesh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; visual mesh filename=package://example-robot-data/robots/falcon_description/mesh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
- added link falcon, mass 200.0; collision mesh filename=package://example-robot-data/robots/falcon_description/mesh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; visual mesh filename=package://example-robot-data/robots/falcon_description/mesh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
- added link floaterL, mass 2.0; collision mesh filename=package://example-robot-data/robots/falcon_description/mesh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; visual mesh filename=package://example-robot-data/robots/falcon_description/mesh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
- added link floaterR, mass 2.0; collision mesh filename=package://example-robot-data/robots/falcon_description/mesh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; visual mesh filename=package://example-robot-data/robots/falcon_description/mesh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
- added link grasping_poing
- added link top_propeller; visual mesh filename=package://example-robot-data/robots/falcon_description/mesh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
Joints:
- removed joint Thruster_BOTTOM_BL_joint
- removed joint Thruster_BOTTOM_BR_joint
- removed joint Thruster_BOTTOM_FL_joint
- removed joint Thruster_BOTTOM_FR_joint
- removed joint Thruster_TOP_B_joint
- removed joint Thruster_TOP_FL_joint
- removed joint Thruster_TOP_FR_joint
- removed joint box_base_bravo_joint
- removed joint bravo_EE_joint
- removed joint contact_point_joint
- added joint BL_propeller_joint: type fixed, parent falcon, child BL_propeller, origin xyz=0.19 0.31 0.165 rpy=0.0 0.0 -1.0472
- added joint BR_propeller_joint: type fixed, parent falcon, child BR_propeller, origin xyz=-0.19 0.31 0.165 rpy=0.0 0.0 -2.0944
- added joint FL_propeller_joint: type fixed, parent falcon, child FL_propeller, origin xyz=0.165 -0.307 0.165 rpy=0.0 0.0 -1.0472
- added joint FR_propeller_joint: type fixed, parent falcon, child FR_propeller, origin xyz=-0.165 -0.307 0.165 rpy=0.0 0.0 -2.094395327
- added joint bravo_finger1_joint: type revolute, parent bravo_finger_jaws_base_link, child bravo_finger1_link, origin xyz=0.0 -0.033 0 rpy=0 1.57 0, axis 0 0 -1, limit lower=0 upper=1.0 effort=10 velocity=10
- added joint bravo_finger2_joint: type revolute, parent bravo_finger_jaws_base_link, child bravo_finger2_link, origin xyz=0 0.033 0 rpy=0 1.57 0, axis 0 0 1, limit lower=0 upper=1.0 effort=10 velocity=10
- added joint bravo_finger_jaws_joint: type fixed, parent link7, child bravo_finger_jaws_base_link, origin xyz= 0.0 0 0.132 rpy=3.14 0 0
- added joint falcon2chassis: type fixed, parent falcon, child chassis, origin xyz=0.295 -0.73 -0.275 rpy=-1.57 3.14  0
- added joint falcon2floaterL: type fixed, parent falcon, child floaterL, origin xyz=-0.365 0.45 0.45 rpy=-1.57 0 -1.57
- added joint falcon2floaterR: type fixed, parent falcon, child floaterR, origin xyz=0.29 0.45 0.45 rpy=-1.57 0 -1.57
- added joint grasping_point_joint: type fixed, parent link7, child grasping_poing, origin xyz= 0.0 0 0.175 rpy=3.14 0 0
- added joint top_propeller_joint: type fixed, parent falcon, child top_propeller, origin xyz=-0.005 0.015 0.35 rpy=0.0 1.57 0
- joint base2arm: origin xyz=0 -0.05 -0.05 rpy=3.14 0.0 1.57 -> xyz=-0.325 -0.65 -0.09 rpy=0 0 3.14; parent box_base_bravo -> falcon

File: robots/falcon_description/urdf/falcon_bravo7_no_ee.urdf (robot description, URDF)
Before this commit: robot falcon_bravo7, 19 links, 18 joints
Links:
- removed link 1_propeller
- removed link 2_propeller
- removed link 3_propeller
- removed link 4_propeller
- removed link Z_propeller
- added link BL_propeller; visual mesh filename=package://example-robot-data/robots/falcon_description/mesh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
- added link BR_propeller; visual mesh filename=package://example-robot-data/robots/falcon_description/mesh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
- added link FL_propeller; visual mesh filename=package://example-robot-data/robots/falcon_description/mesh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
- added link FR_propeller; visual mesh filename=package://example-robot-data/robots/falcon_description/mesh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
- added link top_propeller; visual mesh filename=package://example-robot-data/robots/falcon_description/mesh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
- link chassis: geometry collision mesh filename=package://example-robot-data/robots/falcon_description/mesh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; visual mesh filename=package://example-robot-data/robots/falcon_description/mesh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
- link end_effector_ball: geometry collision mesh filename=package://example-robot-data/robots/bravo7_description/mesh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; visual mesh filename=package://example-robot-data/robots/bravo7_description/mesh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
- link falcon: geometry collision mesh filename=package://example-robot-data/robots/falcon_description/mesh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; visual mesh filename=package://example-robot-data/robots/falcon_description/mesh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
- link floaterL: geometry collision mesh filename=package://example-robot-data/robots/falcon_description/mesh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; visual mesh filename=package://example-robot-data/robots/falcon_description/mesh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
- link floaterR: geometry collision mesh filename=package://example-robot-data/robots/falcon_description/mesh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; visual mesh filename=package://example-robot-data/robots/falcon_description/mesh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
- link link1: geometry collision mesh filename=package://example-robot-data/robots/bravo7_description/mesh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; visual mesh filename=package://example-robot-data/robots/bravo7_description/mesh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
- link link2: geometry collision mesh filename=package://example-robot-data/robots/bravo7_description/mesh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; visual mesh filename=package://example-robot-data/robots/bravo7_description/mesh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
- link link3: geometry collision mesh filename=package://example-robot-data/robots/bravo7_description/mesh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; visual mesh filename=package://example-robot-data/robots/bravo7_description/mesh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
- link link4: geometry collision mesh filename=package://example-robot-data/robots/bravo7_description/mesh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; visual mesh filename=package://example-robot-data/robots/bravo7_description/mesh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
- link link5: geometry collision mesh filename=package://example-robot-data/robots/bravo7_description/mesh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; visual mesh filename=package://example-robot-data/robots/bravo7_description/mesh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
- link link6: geometry collision mesh filename=package://example-robot-data/robots/bravo7_description/mesh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; visual mesh filename=package://example-robot-data/robots/bravo7_description/mesh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
- link link7: geometry collision mesh filename=package://example-robot-data/robots/bravo7_description/mesh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; visual mesh filename=package://example-robot-data/robots/bravo7_description/mesh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
Joints:
- removed joint 1_propeller_joint
- removed joint 2_propeller_joint
- removed joint 3_propeller_joint
- removed joint 4_propeller_joint
- removed joint base_fixed
- removed joint z_propeller_joint
- added joint BL_propeller_joint: type fixed, parent falcon, child BL_propeller, origin xyz=0.19 0.31 0.165 rpy=0.0 0.0 -1.0472
- added joint BR_propeller_joint: type fixed, parent falcon, child BR_propeller, origin xyz=-0.19 0.31 0.165 rpy=0.0 0.0 -2.0944
- added joint FL_propeller_joint: type fixed, parent falcon, child FL_propeller, origin xyz=0.165 -0.307 0.165 rpy=0.0 0.0 -1.0472
- added joint FR_propeller_joint: type fixed, parent falcon, child FR_propeller, origin xyz=-0.165 -0.307 0.165 rpy=0.0 0.0 -2.094395327
- added joint base2arm: type fixed, parent falcon, child link1, origin xyz=-0.325 -0.65 -0.09 rpy=0 0 3.14
- added joint top_propeller_joint: type fixed, parent falcon, child top_propeller, origin xyz=-0.005 0.015 0.35 rpy=0.0 1.57 0
- joint joint1: limit lower=0.0 upper=6.3 effort=9.0 velocity=0.5 -> (none); type revolute -> continuous
- joint joint4: limit lower=0.0 upper=6.3 effort=9.0 velocity=0.5 -> (none); type revolute -> continuous
- joint joint6: limit lower=0.0 upper=6.3 effort=9.0 velocity=0.5 -> (none); type revolute -> continuous
