Commit message: Setting rotational axis positive for compatibility with pinocchio

File: robots/bluevolta_description/urdf/bluevolta.urdf (robot description, URDF)
Before this commit: robot bluevolta, 9 links, 8 joints
Links:
- removed link bluevolta
- added link bluevolta_base_link
- added link bluevolta_rov, mass 200.0; collision mesh filename=package://example-robot-data/robots/bluevolta_description/m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; visual mesh filename=package://example-robot-data/robots/bluevolta_description/m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
Joints:
- added joint bluevolta_fixed_joint: type fixed, parent bluevolta_base_link, child bluevolta_rov, origin xyz=0 0 0 rpy=-3.141592654 0 3.141592654
- joint Thruster_BOTTOM_BL_joint: parent bluevolta -> bluevolta_rov
- joint Thruster_BOTTOM_BR_joint: parent bluevolta -> bluevolta_rov
- joint Thruster_BOTTOM_FL_joint: parent bluevolta -> bluevolta_rov
- joint Thruster_BOTTOM_FR_joint: parent bluevolta -> bluevolta_rov
- joint Thruster_TOP_B_joint: parent bluevolta -> bluevolta_rov
- joint Thruster_TOP_FL_joint: parent bluevolta -> bluevolta_rov
- joint Thruster_TOP_FR_joint: parent bluevolta -> bluevolta_rov
- joint box_base_bravo_joint: parent bluevolta -> bluevolta_rov

File: robots/bluevolta_description/urdf/bluevolta_bravo7_gripper.urdf (robot description, URDF)
Before this commit: robot bluevolta_bravo7_gripper, 21 links, 20 joints
Links:
- removed link bluevolta
- added link bluevolta_base_link
- added link bluevolta_rov, mass 200.0; collision mesh filename=package://example-robot-data/robots/bluevolta_description/m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; visual mesh filename=package://example-robot-data/robots/bluevolta_description/m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
Joints:
- added joint bluevolta_fixed_joint: type fixed, parent bluevolta_base_link, child bluevolta_rov, origin xyz=0 0 0 rpy=-3.141592654 0 3.141592654
- joint Thruster_BOTTOM_BL_joint: parent bluevolta -> bluevolta_rov
- joint Thruster_BOTTOM_BR_joint: parent bluevolta -> bluevolta_rov
- joint Thruster_BOTTOM_FL_joint: parent bluevolta -> bluevolta_rov
- joint Thruster_BOTTOM_FR_joint: parent bluevolta -> bluevolta_rov
- joint Thruster_TOP_B_joint: parent bluevolta -> bluevolta_rov
- joint Thruster_TOP_FL_joint: parent bluevolta -> bluevolta_rov
- joint Thruster_TOP_FR_joint: parent bluevolta -> bluevolta_rov
- joint box_base_bravo_joint: parent bluevolta -> bluevolta_rov
- joint joint1: axis 0 0 -1 -> 0 0 1; origin xyz=0.0665 0 0.078 rpy=0 0 0 -> xyz=0.0665 0 0.078 rpy=3.141592654 0 0
- joint joint2: origin xyz=-0.046 0 0.0674 rpy=0 0 0 -> xyz=-0.046 0 -0.0674 rpy=3.141592654 0 0
- joint joint4: axis 0 0 -1 -> 0 0 1; origin xyz=0.0408 0 0.09695 rpy=0 0 0 -> xyz=0.0408 0 0.09695 rpy=3.141592654 0 0
- joint joint5: origin xyz=-0.0408 0 0.063 rpy=0 0 0 -> xyz=-0.0408 0 -0.063 rpy=3.141592654 0 0
- joint joint6: axis 0 0 -1 -> 0 0 1

File: robots/bluevolta_description/urdf/bluevolta_bravo7_no_ee.urdf (robot description, URDF)
Before this commit: robot bluevolta_bravo7_no_ee, 19 links, 18 joints
Links:
- removed link bluevolta
- added link bluevolta_base_link
- added link bluevolta_rov, mass 200.0; collision mesh filename=package://example-robot-data/robots/bluevolta_description/m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; visual mesh filename=package://example-robot-data/robots/bluevolta_description/m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
Joints:
- added joint bluevolta_fixed_joint: type fixed, parent bluevolta_base_link, child bluevolta_rov, origin xyz=0 0 0 rpy=-3.141592654 0 3.141592654
- joint Thruster_BOTTOM_BL_joint: parent bluevolta -> bluevolta_rov
- joint Thruster_BOTTOM_BR_joint: parent bluevolta -> bluevolta_rov
- joint Thruster_BOTTOM_FL_joint: parent bluevolta -> bluevolta_rov
- joint Thruster_BOTTOM_FR_joint: parent bluevolta -> bluevolta_rov
- joint Thruster_TOP_B_joint: parent bluevolta -> bluevolta_rov
- joint Thruster_TOP_FL_joint: parent bluevolta -> bluevolta_rov
- joint Thruster_TOP_FR_joint: parent bluevolta -> bluevolta_rov
- joint box_base_bravo_joint: parent bluevolta -> bluevolta_rov
- joint joint1: axis 0 0 -1 -> 0 0 1; origin xyz=0.0665 0 0.078 rpy=0 0 0 -> xyz=0.0665 0 0.078 rpy=3.141592654 0 0
- joint joint2: origin xyz=-0.046 0 0.0674 rpy=0 0 0 -> xyz=-0.046 0 -0.0674 rpy=3.141592654 0 0
- joint joint4: axis 0 0 -1 -> 0 0 1; origin xyz=0.0408 0 0.09695 rpy=0 0 0 -> xyz=0.0408 0 0.09695 rpy=3.141592654 0 0
- joint joint5: origin xyz=-0.0408 0 0.063 rpy=0 0 0 -> xyz=-0.0408 0 -0.063 rpy=3.141592654 0 0
- joint joint6: axis 0 0 -1 -> 0 0 1

File: robots/bravo7_description/urdf/bravo7_gripper.urdf (robot description, URDF)
Before this commit: robot bravo7_gripper, 12 links, 11 joints
Joints:
- joint joint1: axis 0 0 -1 -> 0 0 1; origin xyz=0.0665 0 0.078 rpy=0 0 0 -> xyz=0.0665 0 0.078 rpy=3.141592654 0 0
- joint joint2: origin xyz=-0.046 0 0.0674 rpy=0 0 0 -> xyz=-0.046 0 -0.0674 rpy=3.141592654 0 0
- joint joint4: axis 0 0 -1 -> 0 0 1; origin xyz=0.0408 0 0.09695 rpy=0 0 0 -> xyz=0.0408 0 0.09695 rpy=3.141592654 0 0
- joint joint5: origin xyz=-0.0408 0 0.063 rpy=0 0 0 -> xyz=-0.0408 0 -0.063 rpy=3.141592654 0 0
- joint joint6: axis 0 0 -1 -> 0 0 1

File: robots/bravo7_description/urdf/bravo7_no_ee.urdf (robot description, URDF)
Before this commit: robot bravo7_no_ee, 10 links, 9 joints
Joints:
- joint joint1: axis 0 0 -1 -> 0 0 1; origin xyz=0.0665 0 0.078 rpy=0 0 0 -> xyz=0.0665 0 0.078 rpy=3.141592654 0 0
- joint joint2: origin xyz=-0.046 0 0.0674 rpy=0 0 0 -> xyz=-0.046 0 -0.0674 rpy=3.141592654 0 0
- joint joint4: axis 0 0 -1 -> 0 0 1; origin xyz=0.0408 0 0.09695 rpy=0 0 0 -> xyz=0.0408 0 0.09695 rpy=3.141592654 0 0
- joint joint5: origin xyz=-0.0408 0 0.063 rpy=0 0 0 -> xyz=-0.0408 0 -0.063 rpy=3.141592654 0 0
- joint joint6: axis 0 0 -1 -> 0 0 1

File: robots/falcon_description/urdf/falcon_bravo7_gripper.urdf (robot description, URDF)
Before this commit: robot falcon_bravo7_gripper, 21 links, 20 joints
Joints:
- joint joint1: axis 0 0 -1 -> 0 0 1; origin xyz=0.0665 0 0.078 rpy=0 0 0 -> xyz=0.0665 0 0.078 rpy=3.141592654 0 0
- joint joint2: origin xyz=-0.046 0 0.0674 rpy=0 0 0 -> xyz=-0.046 0 -0.0674 rpy=3.141592654 0 0
- joint joint4: axis 0 0 -1 -> 0 0 1; origin xyz=0.0408 0 0.09695 rpy=0 0 0 -> xyz=0.0408 0 0.09695 rpy=3.141592654 0 0
- joint joint5: origin xyz=-0.0408 0 0.063 rpy=0 0 0 -> xyz=-0.0408 0 -0.063 rpy=3.141592654 0 0
- joint joint6: axis 0 0 -1 -> 0 0 1

File: robots/falcon_description/urdf/falcon_bravo7_no_ee.urdf (robot description, URDF)
Before this commit: robot falcon_bravo7_no_ee, 19 links, 18 joints
Joints:
- joint joint1: axis 0 0 -1 -> 0 0 1; origin xyz=0.0665 0 0.078 rpy=0 0 0 -> xyz=0.0665 0 0.078 rpy=3.141592654 0 0
- joint joint2: origin xyz=-0.046 0 0.0674 rpy=0 0 0 -> xyz=-0.046 0 -0.0674 rpy=3.141592654 0 0
- joint joint4: axis 0 0 -1 -> 0 0 1; origin xyz=0.0408 0 0.09695 rpy=0 0 0 -> xyz=0.0408 0 0.09695 rpy=3.141592654 0 0
- joint joint5: origin xyz=-0.0408 0 0.063 rpy=0 0 0 -> xyz=-0.0408 0 -0.063 rpy=3.141592654 0 0
- joint joint6: axis 0 0 -1 -> 0 0 1
