Commit message: [topic/Go2] Move visual files to dedicated folder

File: robots/go2_description/urdf/go2.urdf (robot description, URDF)
Before this commit: robot go2_description, 41 links, 40 joints
Links:
- link FL_calf: geometry collision cylinder length=0.12 radius=0.012; visual mesh filename=package://example-robot-data/robots/go2_description/visuals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
- link FL_foot: geometry collision sphere radius=0.022; visual mesh filename=package://example-robot-data/robots/go2_description/visuals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
- link FL_hip: geometry collision cylinder length=0.04 radius=0.046; visual mesh filename=package://example-robot-data/robots/go2_description/visuals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
- link FL_thigh: geometry collision box size=0.213 0.0245 0.034; visual mesh filename=package://example-robot-data/robots/go2_description/visuals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
- link FR_calf: geometry collision cylinder length=0.12 radius=0.013; visual mesh filename=package://example-robot-data/robots/go2_description/visuals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
- link FR_foot: geometry collision sphere radius=0.022; visual mesh filename=package://example-robot-data/robots/go2_description/visuals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
- link FR_hip: geometry collision cylinder length=0.04 radius=0.046; visual mesh filename=package://example-robot-data/robots/go2_description/visuals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
- link FR_thigh: geometry collision box size=0.213 0.0245 0.034; visual mesh filename=package://example-robot-data/robots/go2_description/visuals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
- link RL_calf: geometry collision cylinder length=0.12 radius=0.013; visual mesh filename=package://example-robot-data/robots/go2_description/visuals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
- link RL_foot: geometry collision sphere radius=0.022; visual mesh filename=package://example-robot-data/robots/go2_description/visuals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
- link RL_hip: geometry collision cylinder length=0.04 radius=0.046; visual mesh filename=package://example-robot-data/robots/go2_description/visuals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
- link RL_thigh: geometry collision box size=0.213 0.0245 0.034; visual mesh filename=package://example-robot-data/robots/go2_description/visuals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
- link RR_calf: geometry collision cylinder length=0.12 radius=0.013; visual mesh filename=package://example-robot-data/robots/go2_description/visuals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
- link RR_foot: geometry collision sphere radius=0.022; visual mesh filename=package://example-robot-data/robots/go2_description/visuals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
- link RR_hip: geometry collision cylinder length=0.04 radius=0.046; visual mesh filename=package://example-robot-data/robots/go2_description/visuals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
- link RR_thigh: geometry collision box size=0.213 0.0245 0.034; visual mesh filename=package://example-robot-data/robots/go2_description/visuals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
- link base: geometry collision box size=0.3762 0.0935 0.114; visual mesh filename=package://example-robot-data/robots/go2_description/visuals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

Commit message: [topic/Go2] Add convexified mesh of body and calf to urdf and slightly simplify urdf

File: robots/go2_description/urdf/go2.urdf (robot description, URDF)
Before this commit: robot go2_description, 41 links, 40 joints
Links:
- removed link FL_calflower
- removed link FL_calflower1
- removed link FR_calflower
- removed link FR_calflower1
- removed link Head_lower
- removed link Head_upper
- removed link RL_calflower
- removed link RL_calflower1
- removed link RR_calflower
- removed link RR_calflower1
- link FL_calf: geometry collision mesh filename=package://example-robot-data/robots/go2_description/collisi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; collision mesh filename=package://example-robot-data/robots/go2_description/collisi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
- link FR_calf: geometry collision mesh filename=package://example-robot-data/robots/go2_description/collisi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; collision mesh filename=package://example-robot-data/robots/go2_description/collisi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
- link RL_calf: geometry collision mesh filename=package://example-robot-data/robots/go2_description/collisi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; collision mesh filename=package://example-robot-data/robots/go2_description/collisi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
- link RR_calf: geometry collision mesh filename=package://example-robot-data/robots/go2_description/collisi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; collision mesh filename=package://example-robot-data/robots/go2_description/collisi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
- link base: geometry collision mesh filename=package://example-robot-data/robots/go2_description/collisi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; collision mesh filename=package://example-robot-data/robots/go2_description/collisi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
Joints:
- removed joint FL_calflower1_joint
- removed joint FL_calflower_joint
- removed joint FR_calflower1_joint
- removed joint FR_calflower_joint
- removed joint Head_lower_joint
- removed joint Head_upper_joint
- removed joint RL_calflower1_joint
- removed joint RL_calflower_joint
- removed joint RR_calflower1_joint
- removed joint RR_calflower_joint

Commit message: [topic/Go2] Remove foot from calf mesh and convexify/add them to urdf

File: robots/go2_description/urdf/go2.urdf (robot description, URDF)
Before this commit: robot go2_description, 31 links, 30 joints
Links:
- link FL_foot: geometry collision mesh filename=package://example-robot-data/robots/go2_description/collisi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; visual mesh filename=package://example-robot-data/robots/go2_description/visuals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
- link FR_foot: geometry collision mesh filename=package://example-robot-data/robots/go2_description/collisi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; visual mesh filename=package://example-robot-data/robots/go2_description/visuals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
- link RL_foot: geometry collision mesh filename=package://example-robot-data/robots/go2_description/collisi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; visual mesh filename=package://example-robot-data/robots/go2_description/visuals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
- link RR_foot: geometry collision mesh filename=package://example-robot-data/robots/go2_description/collisi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; visual mesh filename=package://example-robot-data/robots/go2_description/visuals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

Commit message: [topic/Go2] Add hip convex collision mesh

File: robots/go2_description/urdf/go2.urdf (robot description, URDF)
Before this commit: robot go2_description, 31 links, 30 joints
Links:
- link FL_hip: geometry collision mesh filename=package://example-robot-data/robots/go2_description/collisi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; visual mesh filename=package://example-robot-data/robots/go2_description/visuals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
- link FR_hip: geometry collision mesh filename=package://example-robot-data/robots/go2_description/collisi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; visual mesh filename=package://example-robot-data/robots/go2_description/visuals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
- link RL_hip: geometry collision mesh filename=package://example-robot-data/robots/go2_description/collisi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; visual mesh filename=package://example-robot-data/robots/go2_description/visuals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
- link RR_hip: geometry collision mesh filename=package://example-robot-data/robots/go2_description/collisi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; visual mesh filename=package://example-robot-data/robots/go2_description/visuals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

Commit message: [topic/Go2] tigh convex collisison mesh

File: robots/go2_description/urdf/go2.urdf (robot description, URDF)
Before this commit: robot go2_description, 31 links, 30 joints
Links:
- link FL_thigh: geometry collision mesh filename=package://example-robot-data/robots/go2_description/collisi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; visual mesh filename=package://example-robot-data/robots/go2_description/visuals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
- link FR_thigh: geometry collision mesh filename=package://example-robot-data/robots/go2_description/collisi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; visual mesh filename=package://example-robot-data/robots/go2_description/visuals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
- link RL_thigh: geometry collision mesh filename=package://example-robot-data/robots/go2_description/collisi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; visual mesh filename=package://example-robot-data/robots/go2_description/visuals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
- link RR_thigh: geometry collision mesh filename=package://example-robot-data/robots/go2_description/collisi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; visual mesh filename=package://example-robot-data/robots/go2_description/visuals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

Commit message: Simplify base collisisons

File: robots/go2_description/urdf/go2.urdf (robot description, URDF)
Before this commit: robot go2_description, 31 links, 30 joints
Links:
- link base: geometry collision mesh filename=package://example-robot-data/robots/go2_description/collisi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; visual mesh filename=package://example-robot-data/robots/go2_description/visuals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

Commit message: [topic/Go2] remove front hip collision mesh as it is in the body

File: robots/go2_description/urdf/go2.urdf (robot description, URDF)
Before this commit: robot go2_description, 31 links, 30 joints
Links:
- link FL_hip: geometry visual mesh filename=package://example-robot-data/robots/go2_description/visuals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
- link FR_hip: geometry visual mesh filename=package://example-robot-data/robots/go2_description/visuals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
