Commit message: typo

File: robots/tiago_pro_description/robots/tiago_pro.urdf (robot description, URDF)
Before this commit: robot tiago_pro, 58 links, 57 joints
Links:
- link suspension_rear_right_link: geometry collision mesh filename=package://example-robot-data/robots/tiago_pro_description/m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 scale=1 1.0 1; visual mesh filename=package://example-robot-data/robots/tiago_pro_description/m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 scale=1 1.0 1
