Commit message: changes in axis of rotation (and bounds values) to match the model definition

File: robots/human_description/robots/human.urdf (robot description, URDF)
Before this commit: robot human_36dof_ISB_model, 37 links, 36 joints
Joints:
- joint left_clavicle_joint_X: limit lower=-1.0472 upper=0.349066 effort=100 velocity=14.0 -> lower=-0.349066 upper=1.0472 effort=100 velocity=14.0
- joint left_elbow_Y: axis 0 1 0 -> 0 -1 0; limit lower=-3.14159 upper=0.349066 effort=15 velocity=6.0 -> lower=-0.349066 upper=3.14159 effort=15 velocity=6.0
- joint left_hip_Y: axis 0 1 0 -> 0 -1 0; limit lower=-1.047196667 upper=1.570795 effort=60 velocity=12.0 -> lower=-1.570795 upper=1.047196667 effort=60 velocity=12.0
- joint left_shoulder_Y: axis 0 1 0 -> 0 -1 0
- joint left_wrist_X: axis -1 0 0 -> 1 0 0
- joint middle_lumbar_Z: limit lower=-3.14159 upper=0.785398 effort=190 velocity=5.2 -> lower=-0.785398 upper=3.14159 effort=190 velocity=5.2
- joint middle_thoracic_Z: limit lower=-1.0472 upper=0.392699 effort=190 velocity=5.2 -> lower=-0.392699 upper=1.0472 effort=190 velocity=5.2
- joint right_hip_X: axis 1 0 0 -> -1 0 0; limit lower=-1.570795 upper=1.047196667 effort=120 velocity=6.0 -> lower=-1.047196667 upper=1.570795 effort=120 velocity=6.0
- joint right_shoulder_Y: axis 0 -1 0 -> 0 1 0
- joint right_wrist_X: axis 1 0 0 -> -1 0 0

Commit message: put visual of torso after thoracic joint

File: robots/human_description/robots/human.urdf (robot description, URDF)
Before this commit: robot human_36dof_ISB_model, 37 links, 36 joints
Links:
- link middle_abdomen: geometry visual mesh filename=package://example-robot-data/robots/human_description/meshe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 scale=0.0074 0.0074 0.0074
- link middle_thorax: geometry visual mesh filename=package://example-robot-data/robots/human_description/meshe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 scale=0.007 0.007 0.007
