Commit message: xarm: fix mesh paths

File: robots/xarm_description/urdf/xarm7.urdf (robot description, URDF)
Before this commit: robot UF_ROBOT, 10 links, 9 joints
Links:
- link link1: geometry collision mesh filename=package://example-robot-data/robots/xarm_description/meshes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; visual mesh filename=package://example-robot-data/robots/xarm_description/meshes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
- link link2: geometry collision mesh filename=package://example-robot-data/robots/xarm_description/meshes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; visual mesh filename=package://example-robot-data/robots/xarm_description/meshes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
- link link3: geometry collision mesh filename=package://example-robot-data/robots/xarm_description/meshes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; visual mesh filename=package://example-robot-data/robots/xarm_description/meshes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
- link link4: geometry collision mesh filename=package://example-robot-data/robots/xarm_description/meshes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; visual mesh filename=package://example-robot-data/robots/xarm_description/meshes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
- link link5: geometry collision mesh filename=package://example-robot-data/robots/xarm_description/meshes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; visual mesh filename=package://example-robot-data/robots/xarm_description/meshes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
- link link6: geometry collision mesh filename=package://example-robot-data/robots/xarm_description/meshes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; visual mesh filename=package://example-robot-data/robots/xarm_description/meshes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
- link link7: geometry collision mesh filename=package://example-robot-data/robots/xarm_description/meshes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; visual mesh filename=package://example-robot-data/robots/xarm_description/meshes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
- link link_base: geometry collision mesh filename=package://example-robot-data/robots/xarm_description/meshes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; visual mesh filename=package://example-robot-data/robots/xarm_description/meshes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
