Commit message: removed absolute mesh paths

File: robots/centauro_description/urdf/centauro.urdf (robot description, URDF)
Before this commit: robot centauro, 56 links, 55 joints
Links:
- link ankle1_1: geometry collision mesh filename=package://example-robot-data/robots/centauro_description/me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 scale=0.001 0.001 -0.001; visual mesh filename=package://example-robot-data/robots/centauro_description/me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 scale=0.001 0.001 -0.001
- link ankle1_2: geometry collision mesh filename=package://example-robot-data/robots/centauro_description/me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 scale=0.001 0.001 0.001; visual mesh filename=package://example-robot-data/robots/centauro_description/me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 scale=0.001 0.001 0.001
- link ankle1_3: geometry collision mesh filename=package://example-robot-data/robots/centauro_description/me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 scale=0.001 0.001 -0.001; visual mesh filename=package://example-robot-data/robots/centauro_description/me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 scale=0.001 0.001 -0.001
- link ankle1_4: geometry collision mesh filename=package://example-robot-data/robots/centauro_description/me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 scale=0.001 0.001 0.001; visual mesh filename=package://example-robot-data/robots/centauro_description/me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 scale=0.001 0.001 0.001
- link ankle2_1: geometry collision mesh filename=package://example-robot-data/robots/centauro_description/me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 scale=0.001 -0.001 0.001; visual mesh filename=package://example-robot-data/robots/centauro_description/me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 scale=0.001 -0.001 0.001
- link ankle2_2: geometry collision mesh filename=package://example-robot-data/robots/centauro_description/me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 scale=0.001 0.001 0.001; visual mesh filename=package://example-robot-data/robots/centauro_description/me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 scale=0.001 0.001 0.001
- link ankle2_3: geometry collision mesh filename=package://example-robot-data/robots/centauro_description/me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 scale=0.001 -0.001 0.001; visual mesh filename=package://example-robot-data/robots/centauro_description/me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 scale=0.001 -0.001 0.001
- link ankle2_4: geometry collision mesh filename=package://example-robot-data/robots/centauro_description/me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 scale=0.001 0.001 0.001; visual mesh filename=package://example-robot-data/robots/centauro_description/me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 scale=0.001 0.001 0.001
- link arm2_1: geometry collision mesh filename=package://example-robot-data/robots/centauro_description/me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 scale=0.001 0.001 0.001; visual mesh filename=package://example-robot-data/robots/centauro_description/me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 scale=0.001 0.001 0.001
- link arm2_2: geometry collision mesh filename=package://example-robot-data/robots/centauro_description/me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 scale=0.001 0.001 0.001; visual mesh filename=package://example-robot-data/robots/centauro_description/me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 scale=0.001 0.001 0.001
- link arm2_3: geometry collision mesh filename=package://example-robot-data/robots/centauro_description/me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 scale=0.001 0.001 0.001; visual mesh filename=package://example-robot-data/robots/centauro_description/me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 scale=0.001 0.001 0.001
- link arm2_4: geometry collision mesh filename=package://example-robot-data/robots/centauro_description/me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 scale=0.001 0.001 0.001; visual mesh filename=package://example-robot-data/robots/centauro_description/me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 scale=0.001 0.001 0.001
- link arm2_5: geometry collision mesh filename=package://example-robot-data/robots/centauro_description/me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 scale=0.001 0.001 0.001; visual mesh filename=package://example-robot-data/robots/centauro_description/me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 scale=0.001 0.001 0.001
- link arm2_6: geometry collision mesh filename=package://example-robot-data/robots/centauro_description/me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 scale=0.001 0.001 0.001; visual mesh filename=package://example-robot-data/robots/centauro_description/me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 scale=0.001 0.001 0.001
- link ball2: geometry collision mesh filename=package://example-robot-data/robots/centauro_description/me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 scale=0.001 0.001 0.001; visual mesh filename=package://example-robot-data/robots/centauro_description/me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 scale=0.001 0.001 0.001
- link hip1_1: geometry collision mesh filename=package://example-robot-data/robots/centauro_description/me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 scale=0.001 -0.001 0.001; visual mesh filename=package://example-robot-data/robots/centauro_description/me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 scale=0.001 -0.001 0.001
- link hip1_2: geometry collision mesh filename=package://example-robot-data/robots/centauro_description/me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 scale=0.001 0.001 0.001; visual mesh filename=package://example-robot-data/robots/centauro_description/me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 scale=0.001 0.001 0.001
- link hip1_3: geometry collision mesh filename=package://example-robot-data/robots/centauro_description/me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 scale=0.001 -0.001 0.001; visual mesh filename=package://example-robot-data/robots/centauro_description/me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 scale=0.001 -0.001 0.001
- link hip1_4: geometry collision mesh filename=package://example-robot-data/robots/centauro_description/me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 scale=0.001 0.001 0.001; visual mesh filename=package://example-robot-data/robots/centauro_description/me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 scale=0.001 0.001 0.001
- link hip2_1: geometry collision mesh filename=package://example-robot-data/robots/centauro_description/me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 scale=0.001 0.001 -0.001; visual mesh filename=package://example-robot-data/robots/centauro_description/me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 scale=0.001 0.001 -0.001
- link hip2_2: geometry collision mesh filename=package://example-robot-data/robots/centauro_description/me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 scale=0.001 0.001 0.001; visual mesh filename=package://example-robot-data/robots/centauro_description/me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 scale=0.001 0.001 0.001
- link hip2_3: geometry collision mesh filename=package://example-robot-data/robots/centauro_description/me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 scale=0.001 0.001 -0.001; visual mesh filename=package://example-robot-data/robots/centauro_description/me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 scale=0.001 0.001 -0.001
- link hip2_4: geometry collision mesh filename=package://example-robot-data/robots/centauro_description/me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 scale=0.001 0.001 0.001; visual mesh filename=package://example-robot-data/robots/centauro_description/me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 scale=0.001 0.001 0.001
- link knee_1: geometry collision mesh filename=package://example-robot-data/robots/centauro_description/me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 scale=0.001 0.001 -0.001; visual mesh filename=package://example-robot-data/robots/centauro_description/me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 scale=0.001 0.001 -0.001
- link knee_2: geometry collision mesh filename=package://example-robot-data/robots/centauro_description/me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 scale=0.001 0.001 0.001; visual mesh filename=package://example-robot-data/robots/centauro_description/me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 scale=0.001 0.001 0.001
- link knee_3: geometry collision mesh filename=package://example-robot-data/robots/centauro_description/me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 scale=0.001 0.001 -0.001; visual mesh filename=package://example-robot-data/robots/centauro_description/me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 scale=0.001 0.001 -0.001
- link knee_4: geometry collision mesh filename=package://example-robot-data/robots/centauro_description/me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 scale=0.001 0.001 0.001; visual mesh filename=package://example-robot-data/robots/centauro_description/me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 scale=0.001 0.001 0.001
- link wheel_1: geometry collision cylinder length=0.03 radius=0.124; visual mesh filename=package://example-robot-data/robots/centauro_description/me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 scale=0.001 0.001 -0.001
- link wheel_2: geometry collision cylinder length=0.03 radius=0.124; visual mesh filename=package://example-robot-data/robots/centauro_description/me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 scale=0.001 0.001 0.001
- link wheel_3: geometry collision cylinder length=0.03 radius=0.124; visual mesh filename=package://example-robot-data/robots/centauro_description/me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 scale=0.001 0.001 -0.001
- link wheel_4: geometry collision cylinder length=0.03 radius=0.124; visual mesh filename=package://example-robot-data/robots/centauro_description/me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 scale=0.001 0.001 0.001
